File: why2025.kicad_pcb (KiCad board)
At the start: 2 copper layers, 85.1 x 50.6 mm, 75 parts

Commit message: Keyboard stuff, experiments
Parts:
- removed U3: ~, badgeteam:keyboard_arturo182
- added D73: LED, badgeteam:LTW-010DCG-SR-G, F.Cu at (-29.2, -26.9)
- added D74: LED, badgeteam:LTW-010DCG-SR-G, F.Cu at (-14.6, -26.9)
- added D75: LED, badgeteam:LTW-010DCG-SR-G, F.Cu at (14.6, -26.9)
- added D76: LED, badgeteam:LTW-010DCG-SR-G, F.Cu at (29.2, -26.9)
- added H1: ~, smd_round_nut:SMTSO20, F.Cu at (-50.0, -87.0)
- added H2: ~, smd_round_nut:SMTSO20, F.Cu at (50.0, -87.0)
- added H3: ~, smd_round_nut:SMTSO20, F.Cu at (-44.0, 30.0)
- added H4: ~, smd_round_nut:SMTSO20, F.Cu at (44.0, 30.0)
- added J1: USB_C_Receptacle_USB2.0_16P, Connector_USB:USB_C_Receptacle_G-Switch_GT-USB-7010ASV, B.Cu at (-53.6, -41.3)
- added J2: USB_A, Connector_USB:USB_A_Receptacle_GCT_USB1046, B.Cu at (-52.0, -75.2)
- added J3: USB_A, Connector_USB:USB_A_Receptacle_GCT_USB1046, B.Cu at (-52.0, -58.2)
- added J4: AudioJack3_SwitchT, Connector_Audio:Jack_3.5mm_CUI_SJ-3524-SMT_Horizontal, B.Cu at (50.2, -75.2)
- added N1: Housing, proto1_kicad:proto1_kicad, F.Cu at (0.00, -21.4)
- added R1: 10k, Resistor_SMD:R_0402_1005Metric, B.Cu at (-63.9, 28.8)
- added R2: 10k, Resistor_SMD:R_0402_1005Metric, B.Cu at (-63.9, 30.7)
- added R3: 10k, Resistor_SMD:R_0402_1005Metric, B.Cu at (-63.9, 32.7)
- added R4: 10k, Resistor_SMD:R_0402_1005Metric, B.Cu at (-63.9, 34.7)
- added R5: 10k, Resistor_SMD:R_0402_1005Metric, B.Cu at (-63.9, 36.7)
- added R6: 10k, Resistor_SMD:R_0402_1005Metric, B.Cu at (-63.9, 38.7)
- added R7: 10k, Resistor_SMD:R_0402_1005Metric, B.Cu at (-63.9, 40.7)
- added R8: 10k, Resistor_SMD:R_0402_1005Metric, B.Cu at (-63.9, 42.7)
- D1, D10, D11, D12, D13, D14, D15, D16, D17, D18, D19, D2, D20, D21, D22, D23, D24, D25, D26, D27, D28, D29, D3, D30, D31, D32, D33, D34, D35, D36, D37, D38, D39, D4, D40, D41, D42, D43, D44, D45, D46, D47, D48, D49, D5, D50, D51, D52, D53, D54, D55, D56, D57, D58, D59, D6, D60, D61, D62, D63, D64, D65, D66, D67, D68, D69, D7, D70, D71, D72, D8, D9: moved to B.Cu
- U1: footprint Package_DFN_QFN:QFN-28-1EP_4x4mm_P0.4mm_EP2.6x2.6mm -> Package_QFP:LQFP-48_7x7mm_P0.5mm; moved to B.Cu
- U2: footprint Package_QFP:LQFP-48_7x7mm_P0.5mm -> badgeteam:keyboard_arturo182
- moved U1 161.4 mm to (0.60, -37.2), turned to 180 degrees
- moved U2 126.6 mm to (0.00, 0.00)
- moved D72 112.2 mm to (48.4, -25.4), turned to -90 degrees
- moved D12 107.6 mm to (-34.2, -25.0), turned to -90 degrees
- moved D11 104.9 mm to (-29.2, -28.5), turned to -90 degrees
- moved D13 102.9 mm to (-20.2, -25.0), turned to -90 degrees
- moved D6 101.7 mm to (-44.2, -28.5), turned to -90 degrees
- moved D10 101.0 mm to (-32.2, -25.0), turned to -90 degrees
- moved D26 99.5 mm to (-6.25, -25.0), turned to -90 degrees
- moved D24 99.4 mm to (-18.2, -25.0), turned to -90 degrees
- moved D8 99.2 mm to (-33.2, -28.5), turned to -90 degrees
- moved D51 98.4 mm to (9.20, -28.4), turned to -90 degrees
- moved D38 98.4 mm to (-4.25, -25.0), turned to -90 degrees
- moved D25 98.2 mm to (-10.2, -25.0), turned to -90 degrees
- moved D52 98.0 mm to (21.6, -29.0), turned to -90 degrees
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Connections:
- D1 pad 1: COL0 -> /Coprocessor/Keyboard/COL0
- D10 pad 1: COL5 -> /Coprocessor/Keyboard/COL5
- D11 pad 1: COL6 -> /Coprocessor/Keyboard/COL1
- D12 pad 1: COL7 -> /Coprocessor/Keyboard/COL5
- D13 pad 1: COL0 -> /Coprocessor/Keyboard/COL2
- D14 pad 1: COL1 -> /Coprocessor/Keyboard/COL6
- D15 pad 1: COL2 -> /Coprocessor/Keyboard/COL2
- D16 pad 1: COL3 -> /Coprocessor/Keyboard/COL6
- D17 pad 1: COL0 -> /Coprocessor/Keyboard/COL2
- D18 pad 1: COL4 -> /Coprocessor/Keyboard/COL6
- D19 pad 1: COL5 -> /Coprocessor/Keyboard/COL3
- D2 pad 1: COL1 -> /Coprocessor/Keyboard/COL4
- D20 pad 1: COL6 -> /Coprocessor/Keyboard/COL7
- D21 pad 1: COL7 -> /Coprocessor/Keyboard/COL3
- D22 pad 1: COL0 -> /Coprocessor/Keyboard/COL7
- D23 pad 1: COL1 -> /Coprocessor/Keyboard/COL3
- D24 pad 1: COL2 -> /Coprocessor/Keyboard/COL7
- D25 pad 1: COL3 -> /Coprocessor/Keyboard/COL0
- D26 pad 1: COL4 -> /Coprocessor/Keyboard/COL4
- D27 pad 1: COL5 -> /Coprocessor/Keyboard/COL0
- D28 pad 1: COL6 -> /Coprocessor/Keyboard/COL4
- D29 pad 1: COL7 -> /Coprocessor/Keyboard/COL1
- D3 pad 1: COL2 -> /Coprocessor/Keyboard/COL0
- D30 pad 1: COL1 -> /Coprocessor/Keyboard/COL5
- D31 pad 1: COL0 -> /Coprocessor/Keyboard/COL1
- D32 pad 1: COL1 -> /Coprocessor/Keyboard/COL5
- D33 pad 1: COL2 -> /Coprocessor/Keyboard/COL4
- D34 pad 1: COL3 -> /Coprocessor/Keyboard/COL2
- D35 pad 1: COL4 -> /Coprocessor/Keyboard/COL6
- D36 pad 1: COL5 -> /Coprocessor/Keyboard/COL2
- D37 pad 1: COL6 -> /Coprocessor/Keyboard/COL6
- D38 pad 1: COL7 -> /Coprocessor/Keyboard/COL5
- D39 pad 1: COL0 -> /Coprocessor/Keyboard/COL3
- D4 pad 1: COL3 -> /Coprocessor/Keyboard/COL4
- D40 pad 1: COL1 -> /Coprocessor/Keyboard/COL7
- D41 pad 1: COL2 -> /Coprocessor/Keyboard/COL3
- D42 pad 1: COL3 -> /Coprocessor/Keyboard/COL7
- D43 pad 1: COL2 -> /Coprocessor/Keyboard/COL6
- D44 pad 1: COL4 -> /Coprocessor/Keyboard/COL0
- D45 pad 1: COL5 -> /Coprocessor/Keyboard/COL1
- D46 pad 1: COL6 -> /Coprocessor/Keyboard/COL2
- D47 pad 1: COL7 -> /Coprocessor/Keyboard/COL3
- D48 pad 1: COL0 -> /Coprocessor/Keyboard/COL7
- D48 pad 2: Net-(D48-A) -> /Coprocessor/Keyboard/EXT
- D49 pad 1: COL1 -> /Coprocessor/Keyboard/COL0
- D5 pad 1: COL0 -> /Coprocessor/Keyboard/COL0
- D50 pad 1: COL2 -> /Coprocessor/Keyboard/COL4
- D51 pad 1: COL3 -> /Coprocessor/Keyboard/COL0
- D52 pad 1: COL4 -> /Coprocessor/Keyboard/COL4
- D53 pad 1: COL5 -> /Coprocessor/Keyboard/COL0
- D54 pad 1: COL6 -> /Coprocessor/Keyboard/COL4
- D55 pad 1: COL7 -> /Coprocessor/Keyboard/COL1
- D56 pad 1: COL3 -> /Coprocessor/Keyboard/COL5
- D57 pad 1: COL0 -> /Coprocessor/Keyboard/COL1
- D58 pad 1: COL1 -> /Coprocessor/Keyboard/COL5
- D59 pad 1: COL2 -> /Coprocessor/Keyboard/COL1
- D6 pad 1: COL1 -> /Coprocessor/Keyboard/COL4
- D60 pad 1: COL3 -> /Coprocessor/Keyboard/COL5
- D61 pad 1: COL4 -> /Coprocessor/Keyboard/COL2
- D62 pad 1: COL5 -> /Coprocessor/Keyboard/COL6
- D63 pad 1: COL6 -> /Coprocessor/Keyboard/COL2
- D64 pad 1: COL7 -> /Coprocessor/Keyboard/COL6
- D65 pad 1: COL4 -> /Coprocessor/Keyboard/COL2
- D66 pad 1: COL5 -> /Coprocessor/Keyboard/COL6
- D67 pad 1: COL6 -> /Coprocessor/Keyboard/COL3
- D68 pad 1: COL4 -> /Coprocessor/Keyboard/COL7
- D69 pad 1: COL5 -> /Coprocessor/Keyboard/COL3
- D7 pad 1: COL2 -> /Coprocessor/Keyboard/COL1
- D70 pad 1: COL6 -> /Coprocessor/Keyboard/COL7
- D71 pad 1: COL7 -> /Coprocessor/Keyboard/COL3
- D72 pad 1: COL7 -> /Coprocessor/Keyboard/COL7
- D72 pad 2: BO -> Net-(D72-A)
- D8 pad 1: COL3 -> /Coprocessor/Keyboard/COL5
- D9 pad 1: COL4 -> /Coprocessor/Keyboard/COL1
- U1 pad 10: COL2 -> INT
- U1 pad 11: COL3 -> /Coprocessor/Keyboard/ROW0
- U1 pad 12: COL4 -> /Coprocessor/Keyboard/ROW1
- U1 pad 13: COL5 -> unconnected-(U1-PA3-Pad13)
- U1 pad 14: COL6 -> SPI1_NSS
- U1 pad 15: COL7 -> SPI1_SCK
- U1 pad 16: GND -> SPI1_MISO
- U1 pad 17: +3.3V -> SPI1_MOSI
- U1 pad 18: ROW0 -> /Coprocessor/Keyboard/ROW2
- U1 pad 19: USB_N -> /Coprocessor/Keyboard/COL0
- U1 pad 2: ROW6 -> unconnected-(U1-PC13-Pad2)
- U1 pad 20: USB_P -> /Coprocessor/Keyboard/COL1
- U1 pad 21: SWDIO -> /Coprocessor/Keyboard/COL2
- U1 pad 22: SWCLK -> /Coprocessor/Keyboard/COL3
- U1 pad 23: ROW1 -> GND
- U1 pad 24: ROW2 -> +3.3V
- U1 pad 25: ROW3 -> /Coprocessor/Keyboard/COL4
- U1 pad 26: ROW4 -> /Coprocessor/Keyboard/COL5
- U1 pad 27: SCL -> /Coprocessor/Keyboard/COL6
- U1 pad 28: SDA -> /Coprocessor/Keyboard/COL7
- U1 pad 29: GND -> /Coprocessor/Keyboard/ROW6
- U1 pad 3: ROW7 -> OSC32IN
- U1 pad 4: BI -> OSC32OUT
- U1 pad 5: +3.3V -> unconnected-(U1-PD0-Pad5)
- U1 pad 6: INT -> unconnected-(U1-PD1-Pad6)
- U1 pad 7: ROW5 -> unconnected-(U1-NRST-Pad7)
- U1 pad 8: COL0 -> GND
- U1 pad 9: COL1 -> +3.3V
- U2 pad 1: unconnected-(U2-VBAT-Pad1) -> /Coprocessor/Keyboard/ROW0
- U2 pad 10: INT -> Net-(D49-A)
- U2 pad 11: ROW0 -> /Coprocessor/Keyboard/ROW5
- U2 pad 12: ROW1 -> Net-(D55-A)
- U2 pad 13: unconnected-(U2-PA3-Pad13) -> /Coprocessor/Keyboard/ROW5
- U2 pad 14: SPI1_NSS -> Net-(D61-A)
- U2 pad 15: SPI1_SCK -> /Coprocessor/Keyboard/ROW5
- U2 pad 16: SPI1_MISO -> Net-(D67-A)
- U2 pad 17: SPI1_MOSI -> /Coprocessor/Keyboard/ROW0
- U2 pad 18: ROW2 -> Net-(D2-A)
- U2 pad 19: COL0 -> /Coprocessor/Keyboard/ROW0
- U2 pad 2: unconnected-(U2-PC13-Pad2) -> Net-(D1-A)
- U2 pad 20: COL1 -> Net-(D8-A)
- U2 pad 21: COL2 -> /Coprocessor/Keyboard/ROW0
- U2 pad 22: COL3 -> Net-(D14-A)
- U2 pad 23: GND -> /Coprocessor/Keyboard/ROW0
- U2 pad 24: +3.3V -> Net-(D20-A)
- U2 pad 25: COL4 -> /Coprocessor/Keyboard/ROW3
- U2 pad 26: COL5 -> Net-(D25-A)
- U2 pad 27: COL6 -> /Coprocessor/Keyboard/ROW3
- U2 pad 28: COL7 -> Net-(D29-A)
- U2 pad 29: ROW6 -> /Coprocessor/Keyboard/ROW3
- U2 pad 3: OSC32IN -> /Coprocessor/Keyboard/ROW0
- U2 pad 30: ROW7 -> Net-(D34-A)
- U2 pad 31: BI -> /Coprocessor/Keyboard/ROW3
- U2 pad 32: USB1_N -> Net-(D39-A)
- U2 pad 33: USB1_P -> /Coprocessor/Keyboard/ROW8
- U2 pad 34: SWDIO -> Net-(D44-A)
- U2 pad 35: GND -> /Coprocessor/Keyboard/ROW5
- U2 pad 36: +3.3V -> Net-(D50-A)
- U2 pad 37: SWCLK -> /Coprocessor/Keyboard/ROW5
- U2 pad 38: ROW3 -> Net-(D56-A)
- U2 pad 39: ROW4 -> /Coprocessor/Keyboard/ROW5
- U2 pad 4: OSC32OUT -> Net-(D7-A)
- U2 pad 40: ROW5 -> Net-(D62-A)
- U2 pad 41: SMBA -> /Coprocessor/Keyboard/ROW5
- U2 pad 42: USB2_N -> Net-(D68-A)
- U2 pad 43: USB2_P -> /Coprocessor/Keyboard/ROW1
- U2 pad 44: unconnected-(U2-BOOT0-Pad44) -> Net-(D3-A)
- U2 pad 45: SCL -> /Coprocessor/Keyboard/ROW1
- U2 pad 46: SDA -> Net-(D9-A)
- U2 pad 47: GND -> /Coprocessor/Keyboard/ROW1
- U2 pad 48: +3.3V -> Net-(D15-A)
- U2 pad 5: unconnected-(U2-PD0-Pad5) -> /Coprocessor/Keyboard/ROW0
- U2 pad 6: unconnected-(U2-PD1-Pad6) -> Net-(D13-A)
- U2 pad 7: unconnected-(U2-NRST-Pad7) -> /Coprocessor/Keyboard/ROW0
- U2 pad 8: GND -> Net-(D19-A)
- U2 pad 9: +3.3V -> /Coprocessor/Keyboard/ROW5
Routing:
- net Net-(D43-A): track 0.00 -> 58.1 mm
- net Net-(D38-A): track 0.00 -> 56.2 mm
- net /Coprocessor/Keyboard/ROW2: track 0.00 -> 56.0 mm
- net Net-(D33-A): track 0.00 -> 50.6 mm
- net Net-(D24-A): track 0.00 -> 49.3 mm
- net Net-(D6-A): track 0.00 -> 48.8 mm
- net /Coprocessor/Keyboard/ROW7: track 0.00 -> 47.7 mm
- net Net-(D18-A): track 0.00 -> 45.2 mm
- net Net-(D32-A): track 0.00 -> 44.7 mm
- net Net-(D28-A): track 0.00 -> 44.2 mm
- net Net-(D37-A): track 0.00 -> 44.0 mm
- net Net-(D12-A): track 0.00 -> 43.9 mm
- net Net-(D17-A): track 0.00 -> 41.1 mm
- net Net-(D11-A): track 0.00 -> 40.5 mm
- net Net-(D23-A): track 0.00 -> 40.3 mm
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- added copper zone on F.Cu, net /Coprocessor/Keyboard/ROW0
- added copper zone on F.Cu, net /Coprocessor/Keyboard/ROW1
- added copper zone on F.Cu, net /Coprocessor/Keyboard/ROW2
- added copper zone on F.Cu, net /Coprocessor/Keyboard/ROW3
- added copper zone on F.Cu, net /Coprocessor/Keyboard/ROW4
- added copper zone on F.Cu, net /Coprocessor/Keyboard/ROW5
- added copper zone on F.Cu, net /Coprocessor/Keyboard/ROW6
- added copper zone on F.Cu, net /Coprocessor/Keyboard/ROW7
- added copper zone on F.Cu, net /Coprocessor/Keyboard/ROW8
- removed copper zone on F.Cu, net ROW7
Other:
- board size 85.1 x 50.6 mm -> 114.9 x 125.5 mm
- copper layers 2 -> 4

Commit message: Add radio, wire up more stuff
Parts:
- added C1: 100n, Capacitor_SMD:C_0402_1005Metric, B.Cu at (-17.5, -77.0)
- added C10: 100n, Capacitor_SMD:C_0402_1005Metric, B.Cu at (12.4, -83.2)
- added C2: 22u, Capacitor_SMD:C_0805_2012Metric, B.Cu at (-19.0, -76.5)
- added C3: 22p, Capacitor_SMD:C_0402_1005Metric, B.Cu at (-13.7, -80.5)
- added C4: 22u, Capacitor_SMD:C_0805_2012Metric, B.Cu at (-21.0, -80.0)
- added C5: 22u, Capacitor_SMD:C_0805_2012Metric, B.Cu at (-19.0, -80.0)
- added C6: 100n, Capacitor_SMD:C_0402_1005Metric, B.Cu at (-37.4, -78.0)
- added C7: 10u, Capacitor_SMD:C_0402_1005Metric, B.Cu at (-36.4, -78.0)
- added C8: 1u, Capacitor_SMD:C_0402_1005Metric, B.Cu at (-37.0, -76.5)
- added C9: 1u, Capacitor_SMD:C_0402_1005Metric, B.Cu at (13.5, -81.0)
- added F1: 1A, Fuse:Fuse_0805_2012Metric, B.Cu at (-32.2, -84.5)
- added J5: External Add-On, Connector_PinSocket_2.54mm:PinSocket_2x08_P2.54mm_Horizontal, B.Cu at (-45.8, -32.0)
- added J6: Internal Add-On, Connector_PinSocket_2.54mm:PinSocket_2x15_P2.54mm_Vertical_SMD, B.Cu at (0.00, -37.0)
- added L1: 2.2u, inductors:Inductor_MSC20FC, B.Cu at (-15.4, -80.2)
- added R10: 5.1k, Resistor_SMD:R_0402_1005Metric, B.Cu at (-36.5, -82.0)
- added R11: 10k, Resistor_SMD:R_0402_1005Metric, B.Cu at (-11.7, -80.5)
- added R12: 45.3k, Resistor_SMD:R_0402_1005Metric, B.Cu at (-12.7, -80.5)
- added R13: 10k, Resistor_SMD:R_0402_1005Metric, B.Cu at (12.5, -82.2)
- added R14: 10k, Resistor_SMD:R_0402_1005Metric, B.Cu at (12.5, -74.7)
- added R15: 10k, Resistor_SMD:R_0402_1005Metric, B.Cu at (12.5, -72.0)
- added R16: 10k, Resistor_SMD:R_0402_1005Metric, B.Cu at (-9.70, -67.0)
- added R17: 27, Resistor_SMD:R_0402_1005Metric, B.Cu at (13.1, -67.0)
- added R18: 27, Resistor_SMD:R_0402_1005Metric, B.Cu at (13.1, -68.2)
- added R9: 5.1k, Resistor_SMD:R_0402_1005Metric, B.Cu at (-40.5, -82.0)
- added U3: SY8079AAC, Package_TO_SOT_SMD:SOT-23-5, B.Cu at (-14.8, -77.6)
- added U4: CH334R, Package_SO:QSOP-16_3.9x4.9mm_P0.635mm, B.Cu at (-32.2, -76.0)
- added U5: ESP32-C6-WROOM-1, microcontrollers:ESP32-C6-WROOM-1, B.Cu at (1.25, -75.2)
- added Y1: 12MHz, Crystal:Crystal_SMD_3225-4Pin_3.2x2.5mm, B.Cu at (-33.0, -80.5)
- J1: value USB_C_Receptacle_USB2.0_16P -> USB device; footprint Connector_USB:USB_C_Receptacle_G-Switch_GT-USB-7010ASV -> Connector_USB:USB_C_Receptacle_HRO_TYPE-C-31-M-12
- moved R8 83.8 mm to (-24.0, -31.0)
- moved R7 80.2 mm to (-28.0, -31.0)
- moved R4 77.9 mm to (-22.0, -31.0)
- moved R6 75.1 mm to (-36.0, -31.0)
- moved R3 74.1 mm to (-26.0, -31.0)
- moved R5 71.8 mm to (-40.0, -31.0)
- moved R2 68.6 mm to (-34.0, -31.0)
- moved R1 65.1 mm to (-38.0, -31.0)
- moved J1 49.2 mm to (-38.8, -88.1), turned to 0 degrees
- moved D53 38.3 mm to (30.0, -28.5), turned to -90 degrees
- moved U1 30.7 mm to (-30.0, -40.0)
- moved D68 22.7 mm to (25.0, -25.0)
- moved D72 22.6 mm to (26.0, -28.5)
- moved D48 21.6 mm to (28.0, -28.5)
- moved D69 21.4 mm to (22.0, -28.5)
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Connections:
- net /Coprocessor/Keyboard/COL2 renamed KB_COL2
- net /Coprocessor/Keyboard/COL5 renamed KB_COL5
- net /Coprocessor/Keyboard/ROW5 renamed KB_ROW5
- net Net-(J1-VBUS-PadA4) renamed /USB_VBUS
- net SCL renamed /Coprocessor/SCL
- net SDA renamed /Coprocessor/SDA
- net SWCLK renamed /Coprocessor/SWCLK
- net SWDIO renamed /Coprocessor/SWDIO
- D1 pad 1: /Coprocessor/Keyboard/COL0 -> KB_COL0
- D11 pad 1: /Coprocessor/Keyboard/COL1 -> KB_COL1
- D14 pad 1: /Coprocessor/Keyboard/COL6 -> KB_COL6
- D16 pad 1: /Coprocessor/Keyboard/COL6 -> KB_COL6
- D18 pad 1: /Coprocessor/Keyboard/COL6 -> KB_COL6
- D19 pad 1: /Coprocessor/Keyboard/COL3 -> KB_COL3
- D2 pad 1: /Coprocessor/Keyboard/COL4 -> KB_COL4
- D20 pad 1: /Coprocessor/Keyboard/COL7 -> KB_COL7
- D21 pad 1: /Coprocessor/Keyboard/COL3 -> KB_COL3
- D22 pad 1: /Coprocessor/Keyboard/COL7 -> KB_COL7
- D23 pad 1: /Coprocessor/Keyboard/COL3 -> KB_COL3
- D24 pad 1: /Coprocessor/Keyboard/COL7 -> KB_COL7
- D25 pad 1: /Coprocessor/Keyboard/COL0 -> KB_COL0
- D26 pad 1: /Coprocessor/Keyboard/COL4 -> KB_COL4
- D27 pad 1: /Coprocessor/Keyboard/COL0 -> KB_COL0
- D28 pad 1: /Coprocessor/Keyboard/COL4 -> KB_COL4
- D29 pad 1: /Coprocessor/Keyboard/COL1 -> KB_COL1
- D3 pad 1: /Coprocessor/Keyboard/COL0 -> KB_COL0
- D31 pad 1: /Coprocessor/Keyboard/COL1 -> KB_COL1
- D33 pad 1: /Coprocessor/Keyboard/COL4 -> KB_COL4
- D35 pad 1: /Coprocessor/Keyboard/COL6 -> KB_COL6
- D37 pad 1: /Coprocessor/Keyboard/COL6 -> KB_COL6
- D39 pad 1: /Coprocessor/Keyboard/COL3 -> KB_COL3
- D4 pad 1: /Coprocessor/Keyboard/COL4 -> KB_COL4
- D40 pad 1: /Coprocessor/Keyboard/COL7 -> KB_COL7
- D41 pad 1: /Coprocessor/Keyboard/COL3 -> KB_COL3
- D42 pad 1: /Coprocessor/Keyboard/COL7 -> KB_COL7
- D43 pad 1: /Coprocessor/Keyboard/COL6 -> KB_COL6
- D44 pad 1: /Coprocessor/Keyboard/COL0 -> KB_COL0
- D45 pad 1: /Coprocessor/Keyboard/COL1 -> KB_COL1
- D47 pad 1: /Coprocessor/Keyboard/COL3 -> KB_COL3
- D48 pad 1: /Coprocessor/Keyboard/COL7 -> KB_COL7
- D49 pad 1: /Coprocessor/Keyboard/COL0 -> KB_COL0
- D5 pad 1: /Coprocessor/Keyboard/COL0 -> KB_COL0
- D50 pad 1: /Coprocessor/Keyboard/COL4 -> KB_COL4
- D51 pad 1: /Coprocessor/Keyboard/COL0 -> KB_COL0
- D52 pad 1: /Coprocessor/Keyboard/COL4 -> KB_COL4
- D53 pad 1: /Coprocessor/Keyboard/COL0 -> KB_COL0
- D54 pad 1: /Coprocessor/Keyboard/COL4 -> KB_COL4
- D55 pad 1: /Coprocessor/Keyboard/COL1 -> KB_COL1
- D57 pad 1: /Coprocessor/Keyboard/COL1 -> KB_COL1
- D59 pad 1: /Coprocessor/Keyboard/COL1 -> KB_COL1
- D6 pad 1: /Coprocessor/Keyboard/COL4 -> KB_COL4
- D62 pad 1: /Coprocessor/Keyboard/COL6 -> KB_COL6
- D64 pad 1: /Coprocessor/Keyboard/COL6 -> KB_COL6
- D66 pad 1: /Coprocessor/Keyboard/COL6 -> KB_COL6
- D67 pad 1: /Coprocessor/Keyboard/COL3 -> KB_COL3
- D68 pad 1: /Coprocessor/Keyboard/COL7 -> KB_COL7
- D69 pad 1: /Coprocessor/Keyboard/COL3 -> KB_COL3
- D7 pad 1: /Coprocessor/Keyboard/COL1 -> KB_COL1
- D70 pad 1: /Coprocessor/Keyboard/COL7 -> KB_COL7
- D71 pad 1: /Coprocessor/Keyboard/COL3 -> KB_COL3
- D72 pad 1: /Coprocessor/Keyboard/COL7 -> KB_COL7
- D9 pad 1: /Coprocessor/Keyboard/COL1 -> KB_COL1
- J1 pad A1: Net-(J1-GND-PadA1) -> GND
- J1 pad A12: Net-(J1-GND-PadA1) -> GND
- J1 pad A5: unconnected-(J1-CC1-PadA5) -> /CC1
- J1 pad A6: unconnected-(J1-D+-PadA6) -> /USB_DEVICE_P
- J1 pad A7: unconnected-(J1-D--PadA7) -> /USB_DEVICE_N
- J1 pad B1: Net-(J1-GND-PadA1) -> GND
- J1 pad B12: Net-(J1-GND-PadA1) -> GND
- J1 pad B5: unconnected-(J1-CC2-PadB5) -> /CC2
- J1 pad B6: unconnected-(J1-D+-PadB6) -> /USB_DEVICE_P
- J1 pad B7: unconnected-(J1-D--PadB7) -> /USB_DEVICE_N
- J1 pad S1: unconnected-(J1-SHIELD-PadS1) -> GND
- J3 pad 1: unconnected-(J3-VBUS-Pad1) -> VBUS
- J3 pad 2: unconnected-(J3-D--Pad2) -> /Coprocessor/USB_2_N
- J3 pad 3: unconnected-(J3-D+-Pad3) -> /Coprocessor/USB_2_P
- J3 pad 4: unconnected-(J3-GND-Pad4) -> GND
- J3 pad 5: unconnected-(J3-Shield-Pad5) -> GND
- R1 pad 1: /Coprocessor/Keyboard/COL0 -> KB_COL0
- R2 pad 1: /Coprocessor/Keyboard/COL1 -> KB_COL1
- R4 pad 1: /Coprocessor/Keyboard/COL3 -> KB_COL3
- R5 pad 1: /Coprocessor/Keyboard/COL4 -> KB_COL4
- R7 pad 1: /Coprocessor/Keyboard/COL6 -> KB_COL6
- R8 pad 1: /Coprocessor/Keyboard/COL7 -> KB_COL7
- U1 pad 11: /Coprocessor/Keyboard/ROW0 -> KB_ROW7
- U1 pad 12: /Coprocessor/Keyboard/ROW1 -> KB_ROW6
- U1 pad 18: /Coprocessor/Keyboard/ROW2 -> KB_ROW3
- U1 pad 19: /Coprocessor/Keyboard/COL0 -> KB_COL3
- U1 pad 20: /Coprocessor/Keyboard/COL1 -> KB_COL7
- U1 pad 22: /Coprocessor/Keyboard/COL3 -> KB_COL6
- U1 pad 25: /Coprocessor/Keyboard/COL4 -> KB_COL1
- U1 pad 27: /Coprocessor/Keyboard/COL6 -> KB_COL0
- U1 pad 28: /Coprocessor/Keyboard/COL7 -> KB_COL4
- U1 pad 29: /Coprocessor/Keyboard/ROW6 -> KB_ROW0
- U1 pad 30: /Coprocessor/Keyboard/ROW7 -> KB_ROW1
- U1 pad 31: /Coprocessor/Keyboard/ROW8 -> KB_ROW2
- U1 pad 32: USB1_N -> /Coprocessor/USB_1_N
- U1 pad 33: USB1_P -> /Coprocessor/USB_1_P
- U1 pad 38: /Coprocessor/Keyboard/ROW3 -> KB_ROW4
- U1 pad 39: /Coprocessor/Keyboard/ROW4 -> KB_ROW8
- U1 pad 42: USB2_N -> /Coprocessor/USB_2_N
- U1 pad 43: USB2_P -> /Coprocessor/USB_2_P
- U2 pad 1: /Coprocessor/Keyboard/ROW0 -> KB_ROW0
- U2 pad 101: /Coprocessor/Keyboard/ROW2 -> KB_ROW2
- U2 pad 103: /Coprocessor/Keyboard/ROW4 -> KB_ROW4
- U2 pad 105: /Coprocessor/Keyboard/ROW4 -> KB_ROW4
- U2 pad 107: /Coprocessor/Keyboard/ROW4 -> KB_ROW4
- U2 pad 109: /Coprocessor/Keyboard/ROW4 -> KB_ROW4
- U2 pad 111: /Coprocessor/Keyboard/ROW8 -> KB_ROW8
- U2 pad 113: /Coprocessor/Keyboard/ROW7 -> KB_ROW7
- U2 pad 115: /Coprocessor/Keyboard/ROW7 -> KB_ROW7
- U2 pad 117: /Coprocessor/Keyboard/ROW7 -> KB_ROW7
- U2 pad 119: /Coprocessor/Keyboard/ROW7 -> KB_ROW7
- U2 pad 121: /Coprocessor/Keyboard/ROW2 -> KB_ROW2
- U2 pad 123: /Coprocessor/Keyboard/ROW2 -> KB_ROW2
- U2 pad 125: /Coprocessor/Keyboard/ROW2 -> KB_ROW2
- U2 pad 127: /Coprocessor/Keyboard/ROW2 -> KB_ROW2
- U2 pad 129: /Coprocessor/Keyboard/ROW8 -> KB_ROW8
- U2 pad 131: /Coprocessor/Keyboard/ROW8 -> KB_ROW8
- U2 pad 133: /Coprocessor/Keyboard/ROW8 -> KB_ROW8
- U2 pad 135: /Coprocessor/Keyboard/ROW7 -> KB_ROW7
- U2 pad 137: /Coprocessor/Keyboard/ROW7 -> KB_ROW7
- U2 pad 139: /Coprocessor/Keyboard/ROW7 -> KB_ROW7
- U2 pad 141: /Coprocessor/Keyboard/ROW7 -> KB_ROW7
- U2 pad 17: /Coprocessor/Keyboard/ROW0 -> KB_ROW0
- U2 pad 19: /Coprocessor/Keyboard/ROW0 -> KB_ROW0
- U2 pad 21: /Coprocessor/Keyboard/ROW0 -> KB_ROW0
- U2 pad 23: /Coprocessor/Keyboard/ROW0 -> KB_ROW0
- U2 pad 25: /Coprocessor/Keyboard/ROW3 -> KB_ROW3
- U2 pad 27: /Coprocessor/Keyboard/ROW3 -> KB_ROW3
- U2 pad 29: /Coprocessor/Keyboard/ROW3 -> KB_ROW3
- U2 pad 3: /Coprocessor/Keyboard/ROW0 -> KB_ROW0
- U2 pad 31: /Coprocessor/Keyboard/ROW3 -> KB_ROW3
- U2 pad 33: /Coprocessor/Keyboard/ROW8 -> KB_ROW8
- U2 pad 43: /Coprocessor/Keyboard/ROW1 -> KB_ROW1
- U2 pad 45: /Coprocessor/Keyboard/ROW1 -> KB_ROW1
- U2 pad 47: /Coprocessor/Keyboard/ROW1 -> KB_ROW1
- U2 pad 49: /Coprocessor/Keyboard/ROW1 -> KB_ROW1
- U2 pad 5: /Coprocessor/Keyboard/ROW0 -> KB_ROW0
- U2 pad 51: /Coprocessor/Keyboard/ROW3 -> KB_ROW3
- U2 pad 53: /Coprocessor/Keyboard/ROW3 -> KB_ROW3
- U2 pad 55: /Coprocessor/Keyboard/ROW3 -> KB_ROW3
- U2 pad 57: /Coprocessor/Keyboard/ROW3 -> KB_ROW3
- U2 pad 59: /Coprocessor/Keyboard/ROW8 -> KB_ROW8
- U2 pad 61: /Coprocessor/Keyboard/ROW6 -> KB_ROW6
- U2 pad 63: /Coprocessor/Keyboard/ROW6 -> KB_ROW6
- U2 pad 65: /Coprocessor/Keyboard/ROW6 -> KB_ROW6
- U2 pad 67: /Coprocessor/Keyboard/ROW6 -> KB_ROW6
- U2 pad 69: /Coprocessor/Keyboard/ROW1 -> KB_ROW1
- U2 pad 7: /Coprocessor/Keyboard/ROW0 -> KB_ROW0
- U2 pad 71: /Coprocessor/Keyboard/ROW1 -> KB_ROW1
- U2 pad 73: /Coprocessor/Keyboard/ROW1 -> KB_ROW1
- U2 pad 75: /Coprocessor/Keyboard/ROW1 -> KB_ROW1
- U2 pad 77: /Coprocessor/Keyboard/ROW4 -> KB_ROW4
- U2 pad 79: /Coprocessor/Keyboard/ROW4 -> KB_ROW4
- U2 pad 81: /Coprocessor/Keyboard/ROW4 -> KB_ROW4
- U2 pad 83: /Coprocessor/Keyboard/ROW4 -> KB_ROW4
- U2 pad 85: /Coprocessor/Keyboard/ROW8 -> KB_ROW8
- U2 pad 87: /Coprocessor/Keyboard/ROW6 -> KB_ROW6
- U2 pad 89: /Coprocessor/Keyboard/ROW6 -> KB_ROW6
- U2 pad 91: /Coprocessor/Keyboard/ROW6 -> KB_ROW6
- U2 pad 93: /Coprocessor/Keyboard/ROW6 -> KB_ROW6
- U2 pad 95: /Coprocessor/Keyboard/ROW2 -> KB_ROW2
- U2 pad 97: /Coprocessor/Keyboard/ROW2 -> KB_ROW2
- U2 pad 99: /Coprocessor/Keyboard/ROW2 -> KB_ROW2
Routing:
- net KB_ROW7: track 0.00 -> 141.1 mm, vias 0 -> 1
- net KB_ROW6: track 0.00 -> 129.7 mm, vias 0 -> 1
- net KB_COL0: track 0.00 -> 117.0 mm, vias 0 -> 3
- net VBUS: track 0.00 -> 112.9 mm, vias 0 -> 2
- net KB_ROW4: track 0.00 -> 106.7 mm, vias 0 -> 1
- net Net-(D53-A): track 0.00 -> 85.4 mm
- net KB_COL7: track 0.00 -> 84.1 mm, vias 0 -> 3
- net KB_COL6: track 0.00 -> 83.1 mm, vias 0 -> 3
- net KB_COL4: track 0.00 -> 82.7 mm, vias 0 -> 3
- net KB_COL3: track 0.00 -> 81.7 mm, vias 0 -> 4
- net KB_COL1: track 0.00 -> 80.1 mm, vias 0 -> 3
- net KB_COL5: track 15.7 -> 94.0 mm, vias 0 -> 4
- net Net-(D44-A): track 0.00 -> 76.0 mm
- net Net-(D51-A): track 0.00 -> 72.2 mm
- net KB_ROW8: track 0.00 -> 71.7 mm, vias 0 -> 1
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- added copper zone on In2.Cu, net +3.3V
- added copper zone on B.Cu, net GND
- added copper zone on In1.Cu, net GND
- added copper zone on F.Cu, net KB_ROW0
- added copper zone on F.Cu, net KB_ROW1
- added copper zone on F.Cu, net KB_ROW2
- added copper zone on F.Cu, net KB_ROW3
- added copper zone on F.Cu, net KB_ROW4
- added copper zone on F.Cu, net KB_ROW6
- added copper zone on F.Cu, net KB_ROW7
- added copper zone on F.Cu, net KB_ROW8
- removed copper zone on F.Cu, net /Coprocessor/Keyboard/ROW0
- removed copper zone on F.Cu, net /Coprocessor/Keyboard/ROW1
- removed copper zone on F.Cu, net /Coprocessor/Keyboard/ROW2
- removed copper zone on F.Cu, net /Coprocessor/Keyboard/ROW3
- removed copper zone on F.Cu, net /Coprocessor/Keyboard/ROW4
- removed copper zone on F.Cu, net /Coprocessor/Keyboard/ROW6
- removed copper zone on F.Cu, net /Coprocessor/Keyboard/ROW7
- removed copper zone on F.Cu, net /Coprocessor/Keyboard/ROW8

Commit message: Relabeling of ESP32-C6 GPIO, route signals to expansion header for testing
Parts:
- removed C9: 1u, Capacitor_SMD:C_0402_1005Metric
- removed R14: 10k, Resistor_SMD:R_0402_1005Metric
- added D77: LED, badgeteam:LTW-010DCG-SR-G, F.Cu at (-27.9, 26.9)
- added D78: LED, badgeteam:LTW-010DCG-SR-G, F.Cu at (-13.9, 26.9)
- added D79: LED, badgeteam:LTW-010DCG-SR-G, F.Cu at (0.05, 26.9)
- added D80: LED, badgeteam:LTW-010DCG-SR-G, F.Cu at (14.1, 26.9)
- added D81: LED, badgeteam:LTW-010DCG-SR-G, F.Cu at (28.1, 26.9)
- added H5: ~, MountingHole:MountingHole_2.2mm_M2_Pad_Via, F.Cu at (-53.0, 3.00)
- added H6: ~, MountingHole:MountingHole_2.2mm_M2_Pad_Via, F.Cu at (53.0, 3.00)
- H1, H2, H3, H4: footprint smd_round_nut:SMTSO20 -> MountingHole:MountingHole_2.2mm_M2_Pad_Via
- moved H4 2.00 mm to (36.0, 30.0)
- moved H1 1.25 mm to (-50.0, -88.2)
- moved H2 0.90 mm to (50.0, -88.2), turned to 90 degrees
Connections:
- D73 pad 1: unconnected-(D73-K-Pad1) -> Net-(D73-K)
- D73 pad 2: unconnected-(D73-A-Pad2) -> Net-(D73-A)
- D74 pad 1: unconnected-(D74-K-Pad1) -> Net-(D73-A)
- D74 pad 2: unconnected-(D74-A-Pad2) -> Net-(D74-A)
- D75 pad 1: unconnected-(D75-K-Pad1) -> Net-(D74-A)
- D75 pad 2: unconnected-(D75-A-Pad2) -> Net-(D75-A)
- D76 pad 1: unconnected-(D76-K-Pad1) -> Net-(D75-A)
- D76 pad 2: unconnected-(D76-A-Pad2) -> Net-(D76-A)
- R13 pad 1: Net-(U5-EN/CHIP_PU) -> P4_MDI
- R15 pad 1: /Radio/DISPLAY CS -> RMII_CLK
- R16 pad 2: /Radio/BUTTON A -> RMII_TXEN
- U1 pad 10: INT -> EXT_IO8
- U1 pad 14: SPI1_NSS -> RMII_CLK
- U1 pad 15: SPI1_SCK -> REFCLK
- U1 pad 16: SPI1_MISO -> P4_USB_1B_P
- U1 pad 17: SPI1_MOSI -> P4_USB_1B_N
- U1 pad 34: /Coprocessor/SWDIO -> EXT_MTCK
- U1 pad 37: /Coprocessor/SWCLK -> EXT_MTDI
- U1 pad 41: SMBA -> unconnected-(U1-PB5-Pad41)
- U1 pad 45: /Coprocessor/SCL -> INT_SCL
- U1 pad 46: /Coprocessor/SDA -> INT_SDA
- U5 pad 10: /Radio/DISPLAY CS -> RMII_CLK
- U5 pad 11: /Radio/DISPLAY BUSY -> P4_USB_1B_N
- U5 pad 15: /Radio/BUTTON A -> RMII_TXEN
- U5 pad 16: /Radio/SDCARD CS -> RMII_RXDV
- U5 pad 17: /Radio/SPI MOSI -> RMII_TXER
- U5 pad 18: /Radio/SPI MISO -> RMII_RXER
- U5 pad 19: /Radio/SPI SCK -> RMII_TXD1
- U5 pad 20: /Radio/I2S DATA -> RMII_RXD1
- U5 pad 21: /Radio/I2S CLOCK -> RMII_TXD0
- U5 pad 23: /Radio/BUTTON C -> RMII_RXD0
- U5 pad 24: /Radio/I2S_LRCK -> P4_UART_RX
- U5 pad 25: /Radio/DISPLAY_RST -> P4_UART_TX
- U5 pad 26: /Radio/BATT CHRG -> P4_I3C_SDA
- U5 pad 27: /Radio/BATT ADC -> P4_I3C_SCL
- U5 pad 3: Net-(U5-EN/CHIP_PU) -> P4_MDI
- U5 pad 4: /Radio/BUTTON B -> EXT_IRQ
- U5 pad 5: /Radio/DISPLAY DC -> P4_MDC
- U5 pad 6: /Radio/I2C SDA -> INT_SDA
- U5 pad 7: /Radio/I2C SCL -> INT_SCL
- U5 pad 8: /Radio/INT -> REFCLK
- U5 pad 9: /Radio/AMP_ENABLE -> P4_USB_1B_P
Routing:
- net Net-(D73-K): track 0.00 -> 148.6 mm, vias 0 -> 2
- net Net-(D76-A): track 0.00 -> 140.2 mm
- net P4_USB_1B_P: track 0.00 -> 54.6 mm
- net P4_I3C_SDA: track 0.00 -> 53.0 mm
- net P4_USB_1B_N: track 0.00 -> 52.6 mm
- net INT_SCL: track 0.00 -> 52.5 mm
- net P4_MDC: track 0.00 -> 52.3 mm
- net P4_UART_TX: track 0.00 -> 52.1 mm
- net RMII_RXD0: track 0.00 -> 49.9 mm
- net P4_MDI: track 0.00 -> 49.7 mm
- net P4_I3C_SCL: track 0.00 -> 49.7 mm
- net RMII_CLK: track 0.00 -> 49.2 mm
- net INT_SDA: track 0.00 -> 47.3 mm
- net RMII_RXD1: track 0.00 -> 47.0 mm
- net REFCLK: track 0.00 -> 46.8 mm
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- added copper zone on F.Cu, net GND

Commit message: Boot pin, bit more routing
Parts:
- added R14: 10k, Resistor_SMD:R_0402_1005Metric, B.Cu at (-28.0, -49.1)
Connections:
- R13 pad 1: P4_MDI -> REFCLK
- U1 pad 10: EXT_IO8 -> EXT_MTMS
- U1 pad 13: unconnected-(U1-PA3-Pad13) -> P4_MDO
- U1 pad 15: REFCLK -> P4_MDI
- U1 pad 44: unconnected-(U1-BOOT0-Pad44) -> EXT_IO1
- U5 pad 3: P4_MDI -> REFCLK
- U5 pad 8: REFCLK -> P4_MDI
Routing:
- net INT_SDA: track 47.3 -> 114.4 mm, vias 0 -> 3
- net INT_SCL: track 52.5 -> 115.2 mm, vias 0 -> 3
- net P4_MDO: track 0.00 -> 43.7 mm, vias 0 -> 2
- net P4_MDI: track 49.7 -> 92.2 mm, vias 0 -> 2
- net RMII_CLK: track 49.2 -> 89.8 mm, vias 0 -> 2
- net P4_USB_1B_P: track 54.6 -> 93.7 mm, vias 0 -> 2
- net P4_USB_1B_N: track 52.6 -> 91.1 mm, vias 0 -> 2
- net /Coprocessor/USB_1_N: track 39.2 -> 55.7 mm, vias 0 -> 2
- net /Coprocessor/USB_1_P: track 37.5 -> 52.4 mm, vias 0 -> 2
- net unconnected-(U1-VBAT-Pad1): track 0.00 -> 10.9 mm
- net EXT_IRQ: track 46.6 -> 55.3 mm
- net EXT_MTCK: track 27.6 -> 19.7 mm, vias 1 -> 0
- net REFCLK: track 46.8 -> 53.1 mm
- net EXT_IO1: track 0.00 -> 6.27 mm, vias 0 -> 1
- net P4_MDC: track 52.3 -> 57.2 mm
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
Commit message: A bit of progress
Parts:
- added J7: Speaker, Connector_Molex:Molex_PicoBlade_53261-0271_1x02-1MP_P1.25mm_Horizontal, B.Cu at (39.0, -30.3)
- added J8: Micro_SD_Card, library:SD_Card-micro_socket_A, B.Cu at (36.8, -82.4)
- J2, J3: footprint Connector_USB:USB_A_Receptacle_GCT_USB1046 -> library:USB-A-TH_JTJ-USB-A-F-10.0-010
- J4: value AudioJack3_SwitchT -> Headphones; footprint Connector_Audio:Jack_3.5mm_CUI_SJ-3524-SMT_Horizontal -> adamgreig:PJ-327C-4A
- moved J4 42.5 mm to (50.3, -32.7)
- moved J2 4.85 mm to (-47.5, -77.0)
- moved J3 4.61 mm to (-47.5, -60.5)
Connections:
- J2 pad 1: unconnected-(J2-VBUS-Pad1) -> VBUS
- J2 pad 4: unconnected-(J2-GND-Pad4) -> GND
- J2 pad 5: unconnected-(J2-Shield-Pad5) -> GND
- J4 pad R: unconnected-(J4-PadR) -> /Audio/HP_R
- J4 pad S: unconnected-(J4-PadS) -> GND
- J4 pad T: unconnected-(J4-PadT) -> /Audio/HP_L
Routing:
- net VBUS: track 112.9 -> 143.8 mm, vias 2 -> 0
- net EXT_IO1: track 6.27 -> 35.2 mm
- net GND: track 2.36 -> 28.7 mm, vias 22 -> 25
- net EXT_MTMS: track 3.54 -> 28.3 mm
- net unconnected-(J2-Shield-Pad5): track 12.8 -> 0.00 mm
- net /Coprocessor/USB_1_N: track 55.7 -> 44.4 mm
- net /Coprocessor/USB_1_P: track 52.4 -> 41.1 mm
- net Net-(J7-Pin_2): track 0.00 -> 10.6 mm
- net /Coprocessor/USB_2_P: track 33.4 -> 36.0 mm, vias 2 -> 0
- net /Coprocessor/USB_2_N: track 33.3 -> 35.0 mm, vias 2 -> 0
