File: why2025.kicad_pcb (KiCad board)
At the start: 4 copper layers, 114.9 x 125.5 mm, 131 parts, among them J1 USB device, J2 USB_A, J3 USB_A, J4 Headphones, J5 External Add-On, J6 Internal Add-On, J7 Speaker, J8 Micro_SD_Card, U3 SY8079AAC, U4 CH334R, U5 ESP32-C6-WROOM-1, Y1 12MHz

Commit message: Work in progress
Parts:
- removed J3: USB_A, library:USB-A-TH_JTJ-USB-A-F-10.0-010
- removed L1: 2.2u, inductors:Inductor_MSC20FC
- removed R15: 10k, Resistor_SMD:R_0402_1005Metric
- removed U3: SY8079AAC, Package_TO_SOT_SMD:SOT-23-5
- added C11: 47nF, Capacitor_SMD:C_0402_1005Metric, F.Cu at (39.9, -55.1)
- added C12: 4.7uF, Capacitor_SMD:C_0603_1608Metric, F.Cu at (37.5, -64.2)
- added C13: 10uF, Capacitor_SMD:C_1206_3216Metric, F.Cu at (29.8, -66.3)
- added C14: 10uF, Capacitor_SMD:C_1206_3216Metric, F.Cu at (29.8, -63.0)
- added C15: 10uF, Capacitor_SMD:C_1206_3216Metric, F.Cu at (29.8, -59.6)
- added C16: 120pF, Capacitor_SMD:C_0402_1005Metric, F.Cu at (39.9, -53.1)
- added C17: 10uF, Capacitor_SMD:C_1206_3216Metric, F.Cu at (29.8, -56.3)
- added C18: 10uF, Capacitor_SMD:C_1206_3216Metric, F.Cu at (29.8, -52.9)
- added C19: 10uF, Capacitor_SMD:C_1206_3216Metric, F.Cu at (29.8, -49.6)
- added C20: 1uF, Capacitor_SMD:C_0603_1608Metric, F.Cu at (37.5, -61.7)
- added C23: 100n, Capacitor_SMD:C_0402_1005Metric, F.Cu at (20.6, -55.1)
- added C9: 1uF, Capacitor_SMD:C_0603_1608Metric, F.Cu at (37.5, -66.8)
- added JP1: BOOT, Jumper:SolderJumper-2_P1.3mm_Open_RoundedPad1.0x1.5mm, F.Cu at (21.4, -57.9)
- added L2: YHNR4020-2R2M, Inductor_SMD_Wurth:L_Wurth_WE-LQSH-4020, F.Cu at (35.5, -53.3)
- added L3: FTC252010SR47MBCA, Inductor_SMD_Wurth:L_Wurth_WE-LQSH-2512, F.Cu at (37.6, -58.7)
- added R19: 2.2k, Resistor_SMD:R_0402_1005Metric, F.Cu at (34.0, -67.0)
- added R20: 261, Resistor_SMD:R_0402_1005Metric, F.Cu at (34.0, -65.0)
- added R21: 5.23k, Resistor_SMD:R_0402_1005Metric, F.Cu at (34.0, -63.0)
- added R22: 30.1k, Resistor_SMD:R_0402_1005Metric, F.Cu at (34.0, -61.0)
- added R23: 45k3, Resistor_SMD:R_0402_1005Metric, F.Cu at (34.0, -59.1)
- added R24: 10k, Resistor_SMD:R_0402_1005Metric, F.Cu at (34.0, -57.1)
- added R25: 4.7k, Resistor_SMD:R_0402_1005Metric, F.Cu at (31.3, -43.5)
- added R26: 4.7k, Resistor_SMD:R_0402_1005Metric, F.Cu at (41.2, -45.5)
- added R27: 4.7k, Resistor_SMD:R_0402_1005Metric, F.Cu at (41.2, -43.5)
- added R28: 10k, Resistor_SMD:R_0402_1005Metric, F.Cu at (31.3, -41.5)
- added R29: 10k, Resistor_SMD:R_0402_1005Metric, F.Cu at (31.3, -39.5)
- added R30: 51k, Resistor_SMD:R_0402_1005Metric, F.Cu at (15.8, -58.7)
- added R33: 51k, Resistor_SMD:R_0402_1005Metric, F.Cu at (15.8, -56.7)
- added R34: 51k, Resistor_SMD:R_0402_1005Metric, F.Cu at (15.8, -54.7)
- added R35: 51k, Resistor_SMD:R_0402_1005Metric, F.Cu at (15.8, -52.7)
- added R36: 51k, Resistor_SMD:R_0402_1005Metric, F.Cu at (15.8, -50.7)
- added R37: 51k, Resistor_SMD:R_0402_1005Metric, F.Cu at (15.8, -48.7)
- added R38: 10k, Resistor_SMD:R_0402_1005Metric, F.Cu at (15.8, -46.7)
- added Y2: 32.768KHz, Crystal:Crystal_SMD_3215-2Pin_3.2x1.5mm, B.Cu at (-22.3, -41.8)
- C1, R11: moved to F.Cu
- C2, C4, C5: value 22u -> 100n; footprint Capacitor_SMD:C_0805_2012Metric -> Capacitor_SMD:C_0402_1005Metric; moved to F.Cu
- C3: value 22p -> 100n; moved to F.Cu
- J2: value USB_A -> ESP32USB
- R12: value 45.3k -> 4.7k; moved to F.Cu
- R16: value 10k -> 100k
- moved C4 63.8 mm to (28.4, -39.6), turned to 0 degrees
- moved C5 63.5 mm to (28.4, -37.6), turned to 0 degrees
- moved R11 58.0 mm to (44.8, -67.0), turned to 0 degrees
- moved C2 57.7 mm to (28.4, -43.5), turned to 0 degrees
- moved C3 57.3 mm to (28.4, -41.6), turned to 0 degrees
- moved R12 56.1 mm to (31.3, -45.5), turned to 0 degrees
- moved C1 55.6 mm to (28.4, -45.5), turned to 0 degrees
- moved J5 16.0 mm to (-45.5, -48.0)
Connections:
- C1 pad 1: VBUS -> +3.3V
- C2 pad 1: VBUS -> +3.3vsb
- C3 pad 2: /Power/FB33 -> GND
- C8 pad 1: VBUS -> VOTG
- J2 pad 1: VBUS -> VOTG
- J6 pad 10: P4_UART_RX -> unconnected-(J6-Pin_10-Pad10)
- J6 pad 11: RMII_RXD0 -> unconnected-(J6-Pin_11-Pad11)
- J6 pad 12: RMII_TXD0 -> unconnected-(J6-Pin_12-Pad12)
- J6 pad 13: RMII_RXD1 -> unconnected-(J6-Pin_13-Pad13)
- J6 pad 14: RMII_TXD1 -> unconnected-(J6-Pin_14-Pad14)
- J6 pad 15: RMII_RXER -> unconnected-(J6-Pin_15-Pad15)
- J6 pad 16: RMII_TXER -> unconnected-(J6-Pin_16-Pad16)
- J6 pad 17: RMII_RXDV -> unconnected-(J6-Pin_17-Pad17)
- J6 pad 18: RMII_TXEN -> unconnected-(J6-Pin_18-Pad18)
- J6 pad 19: P4_USB_1B_N -> unconnected-(J6-Pin_19-Pad19)
- J6 pad 20: RMII_CLK -> unconnected-(J6-Pin_20-Pad20)
- J6 pad 21: P4_USB_1B_P -> unconnected-(J6-Pin_21-Pad21)
- J6 pad 22: P4_MDI -> unconnected-(J6-Pin_22-Pad22)
- J6 pad 23: P4_MDC -> unconnected-(J6-Pin_23-Pad23)
- J6 pad 24: P4_MDO -> unconnected-(J6-Pin_24-Pad24)
- J6 pad 25: EXT_IRQ -> unconnected-(J6-Pin_25-Pad25)
- J6 pad 26: REFCLK -> unconnected-(J6-Pin_26-Pad26)
- J6 pad 7: P4_I3C_SDA -> unconnected-(J6-Pin_7-Pad7)
- J6 pad 8: P4_I3C_SCL -> unconnected-(J6-Pin_8-Pad8)
- J6 pad 9: P4_UART_TX -> unconnected-(J6-Pin_9-Pad9)
- R11 pad 1: /Power/FB33 -> VOTG
- R11 pad 2: GND -> /Power/~{DSEL}
- R12 pad 2: /Power/FB33 -> /Coprocessor/PM_SDA
- R13 pad 1: REFCLK -> /Coprocessor/C6_EN
- R14 pad 1: EXT_IO1 -> Net-(JP1-A)
- R16 pad 2: RMII_TXEN -> /Radio/WAKEUP
- U1 pad 1: unconnected-(U1-VBAT-Pad1) -> +3.3vsb
- U1 pad 10: EXT_MTMS -> /Coprocessor/INT
- U1 pad 11: KB_ROW7 -> KB_ROW5
- U1 pad 12: KB_ROW6 -> KB_ROW8
- U1 pad 13: P4_MDO -> KB_ROW4
- U1 pad 14: RMII_CLK -> KB_ROW3
- U1 pad 15: P4_MDI -> KB_ROW7
- U1 pad 16: P4_USB_1B_P -> KB_ROW6
- U1 pad 17: P4_USB_1B_N -> KB_COL3
- U1 pad 18: KB_ROW3 -> KB_COL7
- U1 pad 19: KB_COL3 -> KB_COL2
- U1 pad 2: unconnected-(U1-PC13-Pad2) -> /Coprocessor/ALARM
- U1 pad 20: KB_COL7 -> KB_COL6
- U1 pad 21: KB_COL2 -> /Coprocessor/PM_SCL
- U1 pad 22: KB_COL6 -> /Coprocessor/PM_SDA
- U1 pad 3: OSC32IN -> Net-(U1-PC14)
- U1 pad 34: EXT_MTCK -> /Coprocessor/SWDIO
- U1 pad 37: EXT_MTDI -> /Coprocessor/SWCLK
- U1 pad 38: KB_ROW4 -> unconnected-(U1-PA15-Pad38)
- U1 pad 39: KB_ROW8 -> unconnected-(U1-PB3-Pad39)
- U1 pad 4: OSC32OUT -> Net-(U1-PC15)
- U1 pad 40: KB_ROW5 -> unconnected-(U1-PB4-Pad40)
- U1 pad 42: /Coprocessor/USB_2_N -> INT_SCL
- U1 pad 43: /Coprocessor/USB_2_P -> INT_SDA
- U1 pad 44: EXT_IO1 -> Net-(JP1-A)
- U1 pad 45: INT_SCL -> /Coprocessor/C6_BOOT
- U1 pad 46: INT_SDA -> /Coprocessor/C6_EN
- U1 pad 7: unconnected-(U1-NRST-Pad7) -> Net-(U1-NRST)
- U4 pad 12: VBUS -> VOTG
- U4 pad 9: unconnected-(U4-~{RESET}/CDP-Pad9) -> /Power/~{DSEL}
- U5 pad 10: RMII_CLK -> /Radio/WAKEUP
- U5 pad 11: P4_USB_1B_N -> unconnected-(U5-GPIO10-Pad11)
- U5 pad 15: RMII_TXEN -> /Coprocessor/C6_BOOT
- U5 pad 16: RMII_RXDV -> /Radio/SDIO_CMD
- U5 pad 17: RMII_TXER -> /Radio/SDIO_CLK
- U5 pad 18: RMII_RXER -> /Radio/SDIO_DATA0
- U5 pad 19: RMII_TXD1 -> /Radio/SDIO_DATA1
- U5 pad 20: RMII_RXD1 -> /Radio/SDIO_DATA2
- U5 pad 21: RMII_TXD0 -> /Radio/SDIO_DATA3
- U5 pad 23: RMII_RXD0 -> unconnected-(U5-GPIO15-Pad23)
- U5 pad 24: P4_UART_RX -> /Radio/RX
- U5 pad 25: P4_UART_TX -> /Radio/TX
- U5 pad 26: P4_I3C_SDA -> unconnected-(U5-GPIO3/ADC1_CH3-Pad26)
- U5 pad 27: P4_I3C_SCL -> unconnected-(U5-GPIO2/ADC1_CH2-Pad27)
- U5 pad 3: REFCLK -> /Coprocessor/C6_EN
- U5 pad 4: EXT_IRQ -> unconnected-(U5-MTMS/GPIO4/ADC1_CH4-Pad4)
- U5 pad 5: P4_MDC -> unconnected-(U5-MTDI/GPIO5/ADC1_CH5-Pad5)
- U5 pad 8: P4_MDI -> unconnected-(U5-GPIO0/ADC1_CH0/XTAL_32K_P-Pad8)
- U5 pad 9: P4_USB_1B_P -> unconnected-(U5-GPIO1/ADC1_CH1/XTAL_32K_N-Pad9)
Routing:
- net P4_USB_1B_P: track 93.7 -> 0.00 mm, vias 2 -> 0
- net P4_MDI: track 92.2 -> 0.00 mm, vias 2 -> 0
- net P4_USB_1B_N: track 91.1 -> 0.00 mm, vias 2 -> 0
- net RMII_CLK: track 89.8 -> 0.00 mm, vias 2 -> 0
- net VBUS: track 143.8 -> 59.6 mm
- net INT_SCL: track 115.2 -> 40.1 mm, vias 3 -> 2
- net INT_SDA: track 114.4 -> 47.3 mm, vias 3 -> 2
- net P4_MDC: track 57.2 -> 0.00 mm
- net EXT_IRQ: track 55.3 -> 0.00 mm
- net REFCLK: track 53.1 -> 0.00 mm
- net P4_I3C_SDA: track 53.0 -> 0.00 mm
- net P4_UART_TX: track 52.1 -> 0.00 mm
- net RMII_RXD0: track 49.9 -> 0.00 mm
- net P4_I3C_SCL: track 49.7 -> 0.00 mm
- net RMII_RXD1: track 47.0 -> 0.00 mm
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
Commit message: Stuff.
Parts:
- added C24: 10uF, Capacitor_SMD:C_1206_3216Metric, F.Cu at (126.1, -141.6)
- added C25: 22p, Capacitor_SMD:C_0402_1005Metric, F.Cu at (130.3, -142.3)
- added C26: 10uF, Capacitor_SMD:C_1206_3216Metric, F.Cu at (126.1, -138.3)
- added C27: 22p, Capacitor_SMD:C_0402_1005Metric, F.Cu at (130.3, -140.3)
- added C28: 22p, Capacitor_SMD:C_0402_1005Metric, F.Cu at (130.3, -138.4)
- added C29: 10uF, Capacitor_SMD:C_1206_3216Metric, F.Cu at (126.1, -134.9)
- added C30: 10uF, Capacitor_SMD:C_1206_3216Metric, F.Cu at (126.1, -131.6)
- added R15: 10k, Resistor_SMD:R_0402_1005Metric, F.Cu at (116.7, -124.4)
- added R39: 499k, Resistor_SMD:R_0402_1005Metric, F.Cu at (116.7, -142.3)
- added R40: 499k, Resistor_SMD:R_0402_1005Metric, F.Cu at (116.7, -140.3)
- added R41: 100k, Resistor_SMD:R_0402_1005Metric, F.Cu at (116.7, -138.3)
- added R42: 365k, Resistor_SMD:R_0402_1005Metric, F.Cu at (116.7, -136.3)
- added R43: 316k, Resistor_SMD:R_0402_1005Metric, F.Cu at (116.7, -134.3)
- added R44: 100k, Resistor_SMD:R_0402_1005Metric, F.Cu at (116.7, -132.4)
- added R45: 100k, Resistor_SMD:R_0402_1005Metric, F.Cu at (116.7, -130.4)
- added R46: 100k, Resistor_SMD:R_0402_1005Metric, F.Cu at (116.7, -128.4)
- added U3: TLV62569DBV, Package_TO_SOT_SMD:SOT-23-5, F.Cu at (120.7, -140.9)
- added U8: TLV62569DBV, Package_TO_SOT_SMD:SOT-23-5, F.Cu at (120.7, -136.3)
- added U9: TLV62569DBV, Package_TO_SOT_SMD:SOT-23-5, F.Cu at (120.7, -131.7)
- moved R12 109.9 mm to (113.3, -118.7)
- moved R26 109.9 mm to (123.3, -118.7)
- moved R29 109.9 mm to (113.3, -112.7)
- moved C1 109.9 mm to (110.4, -118.7)
- moved C2 109.9 mm to (110.4, -116.7)
- moved C3 109.9 mm to (110.4, -114.7)
- moved C4 109.9 mm to (110.4, -112.8)
- moved C5 109.9 mm to (110.4, -110.8)
- moved R25 109.9 mm to (113.3, -116.7)
- moved R27 109.9 mm to (123.3, -116.7)
- moved R28 109.9 mm to (113.3, -114.7)
- moved C13 97.4 mm to (94.6, -139.0)
- moved C16 97.4 mm to (104.7, -125.8)
- moved C17 97.4 mm to (94.6, -129.0)
- moved C18 97.4 mm to (94.6, -125.6)
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Connections:
- U1 pad 38: unconnected-(U1-PA15-Pad38) -> /Coprocessor/PM_INT
- U1 pad 39: unconnected-(U1-PB3-Pad39) -> /Coprocessor/B3
- U1 pad 40: unconnected-(U1-PB4-Pad40) -> /Coprocessor/B4
- U1 pad 41: unconnected-(U1-PB5-Pad41) -> /Coprocessor/STAT_LED
- U1 pad 5: unconnected-(U1-PD0-Pad5) -> /Coprocessor/D0
- U1 pad 6: unconnected-(U1-PD1-Pad6) -> /Coprocessor/D1
- U5 pad 11: unconnected-(U5-GPIO10-Pad11) -> /Radio/10
- U5 pad 23: unconnected-(U5-GPIO15-Pad23) -> /Radio/15
- U5 pad 26: unconnected-(U5-GPIO3/ADC1_CH3-Pad26) -> /Radio/3
- U5 pad 27: unconnected-(U5-GPIO2/ADC1_CH2-Pad27) -> /Radio/2
- U5 pad 4: unconnected-(U5-MTMS/GPIO4/ADC1_CH4-Pad4) -> /Radio/4
- U5 pad 5: unconnected-(U5-MTDI/GPIO5/ADC1_CH5-Pad5) -> /Radio/5
- U5 pad 8: unconnected-(U5-GPIO0/ADC1_CH0/XTAL_32K_P-Pad8) -> /Radio/0
- U5 pad 9: unconnected-(U5-GPIO1/ADC1_CH1/XTAL_32K_N-Pad9) -> /Radio/1
Routing:
- net unconnected-(U1-PB5-Pad41): track 3.61 -> 0.00 mm
- net /Coprocessor/STAT_LED: track 0.00 -> 3.61 mm
Other:
- outline, holes or cut-outs redrawn

Commit message: More schematics
Parts:
- removed U8: TLV62569DBV, Package_TO_SOT_SMD:SOT-23-5
- added C31: 10uF, Capacitor_SMD:C_0603_1608Metric, F.Cu at (148.1, -102.0)
- added C32: 1uF, Capacitor_SMD:C_0603_1608Metric, F.Cu at (148.1, -99.5)
- added C33: 10uF, Capacitor_SMD:C_0603_1608Metric, F.Cu at (148.1, -97.0)
- added C34: 1uF, Capacitor_SMD:C_0603_1608Metric, F.Cu at (148.1, -94.5)
- added C35: 100n, Capacitor_SMD:C_0402_1005Metric, F.Cu at (147.6, -116.8)
- added C36: 100n, Capacitor_SMD:C_0402_1005Metric, F.Cu at (147.6, -114.8)
- added C37: 100n, Capacitor_SMD:C_0402_1005Metric, F.Cu at (147.6, -112.8)
- added C38: 100n, Capacitor_SMD:C_0402_1005Metric, F.Cu at (147.6, -110.9)
- added C39: 1u, Capacitor_SMD:C_0402_1005Metric, F.Cu at (150.4, -122.7)
- added C40: 100n, Capacitor_SMD:C_0402_1005Metric, F.Cu at (150.4, -120.7)
- added C41: 100n, Capacitor_SMD:C_0402_1005Metric, F.Cu at (150.4, -118.7)
- added C42: 100n, Capacitor_SMD:C_0402_1005Metric, F.Cu at (150.4, -116.8)
- added C43: 100n, Capacitor_SMD:C_0402_1005Metric, F.Cu at (150.4, -114.8)
- added C44: 100n, Capacitor_SMD:C_0402_1005Metric, F.Cu at (150.4, -112.8)
- added C45: 100n, Capacitor_SMD:C_0402_1005Metric, F.Cu at (150.4, -110.9)
- added C46: 100n, Capacitor_SMD:C_0402_1005Metric, F.Cu at (153.3, -122.7)
- added C47: 22p, Capacitor_SMD:C_0402_1005Metric, F.Cu at (153.3, -120.7)
- added C48: 22p, Capacitor_SMD:C_0402_1005Metric, F.Cu at (153.3, -118.7)
- added C49: 1u, Capacitor_SMD:C_0402_1005Metric, F.Cu at (153.3, -116.8)
- added C50: 100n, Capacitor_SMD:C_0402_1005Metric, F.Cu at (153.3, -114.8)
- added C51: 100n, Capacitor_SMD:C_0402_1005Metric, F.Cu at (153.3, -112.8)
- added C52: 100n, Capacitor_SMD:C_0402_1005Metric, F.Cu at (153.3, -110.9)
- added C53: 100n, Capacitor_SMD:C_0402_1005Metric, F.Cu at (156.2, -122.7)
- added C54: 100n, Capacitor_SMD:C_0402_1005Metric, F.Cu at (156.2, -120.7)
- added C55: 100n, Capacitor_SMD:C_0402_1005Metric, F.Cu at (156.2, -118.7)
- added C56: 100n, Capacitor_SMD:C_0402_1005Metric, F.Cu at (156.2, -116.8)
- added C57: 100n, Capacitor_SMD:C_0402_1005Metric, F.Cu at (156.2, -114.8)
- added D83: 1N5819, Diode_SMD:D_SOD-323_HandSoldering, F.Cu at (157.7, -92.5)
- added D84: 1N5819, Diode_SMD:D_SOD-323_HandSoldering, F.Cu at (157.7, -89.6)
- added L6: 6.8uH, Inductor_SMD:L_1008_2520Metric, F.Cu at (152.6, -92.1)
- added L7: 6.8uH, Inductor_SMD:L_1008_2520Metric, F.Cu at (152.6, -88.4)
- added R47: 4.7K, Resistor_SMD:R_0603_1608Metric, F.Cu at (148.1, -92.0)
- added R48: 4.7, Resistor_SMD:R_0603_1608Metric, F.Cu at (148.1, -89.5)
- added R50: 4.7K, Resistor_SMD:R_0603_1608Metric, F.Cu at (148.1, -86.9)
- added R51: 10, Resistor_SMD:R_0603_1608Metric, F.Cu at (148.1, -84.4)
- added R52: 4k02, Resistor_SMD:R_0402_1005Metric, F.Cu at (162.0, -122.7)
- added R53: 4k7, Resistor_SMD:R_0402_1005Metric, F.Cu at (162.0, -120.7)
- added R54: 51k, Resistor_SMD:R_0402_1005Metric, F.Cu at (162.0, -118.7)
- added R55: 51k, Resistor_SMD:R_0402_1005Metric, F.Cu at (162.0, -116.7)
- added R56: 51k, Resistor_SMD:R_0402_1005Metric, F.Cu at (162.0, -114.7)
- added R57: 51k, Resistor_SMD:R_0402_1005Metric, F.Cu at (164.9, -122.7)
- added R58: 51k, Resistor_SMD:R_0402_1005Metric, F.Cu at (164.9, -120.7)
- added R59: 51k, Resistor_SMD:R_0402_1005Metric, F.Cu at (164.9, -118.7)
- added R60: 4k7, Resistor_SMD:R_0402_1005Metric, F.Cu at (164.9, -116.7)
- added R61: 4k7, Resistor_SMD:R_0402_1005Metric, F.Cu at (164.9, -114.7)
- added R62: 4k7, Resistor_SMD:R_0402_1005Metric, F.Cu at (167.8, -122.7)
- added R63: 4k7, Resistor_SMD:R_0402_1005Metric, F.Cu at (167.8, -120.7)
- added R64: 4k7, Resistor_SMD:R_0402_1005Metric, F.Cu at (167.8, -118.7)
- added R65: 4k7, Resistor_SMD:R_0402_1005Metric, F.Cu at (167.8, -116.7)
- added R66: 4k7, Resistor_SMD:R_0402_1005Metric, F.Cu at (167.8, -114.7)
- added TP1: TP_BL_CTRL, TestPoint:TestPoint_Pad_D1.5mm, F.Cu at (157.1, -101.5)
- added TP2: TP_BL_CTRL, TestPoint:TestPoint_Pad_D1.5mm, F.Cu at (157.1, -97.9)
- added U11: AP3032KTR, Package_TO_SOT_SMD:SOT-23-6, F.Cu at (152.7, -100.9)
- added U12: AP3032KTR, Package_TO_SOT_SMD:SOT-23-6, F.Cu at (152.7, -96.2)
- added U13: W25Q128JVS, Package_SO:SOIC-8_5.23x5.23mm_P1.27mm, F.Cu at (162.8, -110.3)
- C24: value 10uF -> 22p; footprint Capacitor_SMD:C_1206_3216Metric -> Capacitor_SMD:C_0402_1005Metric
- C25: value 22p -> 10uF; footprint Capacitor_SMD:C_0402_1005Metric -> Capacitor_SMD:C_1206_3216Metric
- C26: value 10uF -> 100n; footprint Capacitor_SMD:C_1206_3216Metric -> Capacitor_SMD:C_0402_1005Metric
- C27: value 22p -> 100n
- R39: value 499k -> 100k
- R41: value 100k -> 499k
- R43: value 316k -> 10k
- R44: value 100k -> 4k02
- moved U3 47.4 mm to (154.3, -107.5)
- moved R39 46.7 mm to (159.1, -122.7)
- moved R41 46.7 mm to (159.1, -118.7)
- moved R40 46.7 mm to (159.1, -120.7)
- moved R44 45.9 mm to (159.1, -114.7)
- moved R43 45.9 mm to (159.1, -116.7)
- moved C25 38.9 mm to (148.9, -108.2)
- moved C24 28.6 mm to (147.6, -122.7)
- moved C26 27.7 mm to (147.6, -120.7)
- moved C27 27.6 mm to (147.6, -118.7)
- moved J8 0.05 mm to (-49.8, -60.1)
Connections:
- net /Coprocessor/SWCLK renamed /Application processor/CH32_SWCLK
- net /Coprocessor/SWDIO renamed /Application processor/CH32_SWDIO
- net /Radio/10 renamed LED_DATA
- net /Radio/15 renamed CAM_GPIO
- net /Radio/RX renamed /Application processor/UART_TX
- net /Radio/SDIO_CLK renamed /Application processor/C6_CLK
- net /Radio/SDIO_CMD renamed /Application processor/C6_CMD
- net /Radio/SDIO_DATA0 renamed /Application processor/C6_D0
- net /Radio/SDIO_DATA1 renamed /Application processor/C6_D1
- net /Radio/SDIO_DATA2 renamed /Application processor/C6_D2
- net /Radio/SDIO_DATA3 renamed /Application processor/C6_D3
- net /Radio/TX renamed /Application processor/UART_RX
- net EXT_IO1 renamed SAO_IO1
- net EXT_IO2 renamed SAO_IO2
- net EXT_MTCK renamed MTDO
- net EXT_MTDI renamed MTDI
- net EXT_MTDO renamed MTCK
- net EXT_MTMS renamed MTMS
- net Net-(J7-Pin_2) renamed /Audio/HP_NC
- C24 pad 2: GND -> Net-(U3-FB)
- C25 pad 1: +2.5v -> VESPHP
- C25 pad 2: Net-(U8-FB) -> GND
- C26 pad 1: +2.5v -> VESPHP
- C27 pad 2: /Power/P4HP_FB -> GND
- J2 pad 2: unconnected-(J2-D--Pad2) -> /Application processor/USB_DM
- J2 pad 3: unconnected-(J2-D+-Pad3) -> /Application processor/USB_DP
- J5 pad 10: EXT_IO4 -> E18
- J5 pad 13: EXT_SDA -> SAO_SDA
- J5 pad 14: EXT_SCL -> SAO_SCL
- J5 pad 5: EXT_IO7 -> E13
- J5 pad 6: EXT_IO8 -> E14
- J5 pad 7: EXT_IO5 -> E15
- J5 pad 8: EXT_IO6 -> E16
- J5 pad 9: EXT_IO3 -> E17
- J6 pad 10: unconnected-(J6-Pin_10-Pad10) -> INT_SDA
- J6 pad 11: unconnected-(J6-Pin_11-Pad11) -> I3C_SCL
- J6 pad 12: unconnected-(J6-Pin_12-Pad12) -> I3C_SDA
- J6 pad 13: unconnected-(J6-Pin_13-Pad13) -> EXT_USB_P
- J6 pad 14: unconnected-(J6-Pin_14-Pad14) -> EXT_USB_N
- J6 pad 15: unconnected-(J6-Pin_15-Pad15) -> E0
- J6 pad 16: unconnected-(J6-Pin_16-Pad16) -> E1
- J6 pad 17: unconnected-(J6-Pin_17-Pad17) -> E2
- J6 pad 18: unconnected-(J6-Pin_18-Pad18) -> E3
- J6 pad 19: unconnected-(J6-Pin_19-Pad19) -> E4
- J6 pad 2: VIN -> VBATT
- J6 pad 20: unconnected-(J6-Pin_20-Pad20) -> E5
- J6 pad 21: unconnected-(J6-Pin_21-Pad21) -> E6
- J6 pad 22: unconnected-(J6-Pin_22-Pad22) -> E7
- J6 pad 23: unconnected-(J6-Pin_23-Pad23) -> E8
- J6 pad 24: unconnected-(J6-Pin_24-Pad24) -> E9
- J6 pad 25: unconnected-(J6-Pin_25-Pad25) -> INT_SDA
- J6 pad 26: unconnected-(J6-Pin_26-Pad26) -> INT_SCL
- J6 pad 27: INT_SDA -> E12
- J6 pad 28: INT_SCL -> E9
- J6 pad 3: GND -> VOTG
- J6 pad 5: +3.3V -> VSYS
- J6 pad 6: VBAT -> +3.3V
- J6 pad 7: unconnected-(J6-Pin_7-Pad7) -> VSDCARD
- J6 pad 8: unconnected-(J6-Pin_8-Pad8) -> +3.3vsb
- J6 pad 9: unconnected-(J6-Pin_9-Pad9) -> INT_SCL
- J8 pad 1: unconnected-(J8-DAT2-Pad1) -> /Application processor/SD_D2
- J8 pad 2: unconnected-(J8-DAT3/CD-Pad2) -> /Application processor/SD_D3
- J8 pad 3: unconnected-(J8-CMD-Pad3) -> /Application processor/SD_CMD
- J8 pad 4: unconnected-(J8-VDD-Pad4) -> VSDCARD
- J8 pad 5: unconnected-(J8-CLK-Pad5) -> /Application processor/SD_CLK
- J8 pad 6: unconnected-(J8-VSS-Pad6) -> GND
- J8 pad 7: unconnected-(J8-DAT0-Pad7) -> /Application processor/SD_D0
- J8 pad 8: unconnected-(J8-DAT1-Pad8) -> /Application processor/SD_D1
- J8 pad 9: unconnected-(J8-SHIELD-Pad9) -> GND
- R16 pad 2: /Radio/WAKEUP -> E8
- R28 pad 2: /Coprocessor/INT -> E7
- R39 pad 2: /Power/P4HP_FB -> Net-(U3-EN)
- R40 pad 1: /Power/P4HP_FB -> Net-(U3-FB)
- R41 pad 2: /Power/P4HP_EN -> Net-(U3-FB)
- R43 pad 1: Net-(U8-FB) -> Net-(U8K-CHIP_PU)
- R43 pad 2: +2.5v -> +3.3V
- R44 pad 1: GND -> Net-(U8H-CSI_REXT)
- R44 pad 2: Net-(U8-FB) -> GND
- R46 pad 2: /Power/VLED_EN -> /Coprocessor/D0
- U1 pad 10: /Coprocessor/INT -> E7
- U3 pad 1: /Power/P4HP_EN -> Net-(U3-EN)
- U3 pad 5: /Power/P4HP_FB -> Net-(U3-FB)
- U4 pad 3: unconnected-(U4-DM3--Pad3) -> /Application processor/USB1_P1_N
- U4 pad 4: unconnected-(U4-DP3+-Pad4) -> /Application processor/USB1_P1_P
- U5 pad 10: /Radio/WAKEUP -> E8
- U5 pad 26: /Radio/3 -> E16
- U5 pad 27: /Radio/2 -> E15
- U5 pad 4: /Radio/4 -> E17
- U5 pad 5: /Radio/5 -> E18
- U5 pad 8: /Radio/0 -> E13
- U5 pad 9: /Radio/1 -> E14
Routing:
- net +3.3V: track 27.7 -> 23.8 mm, vias 7 -> 6
- net VSYS: track 0.00 -> 3.87 mm, vias 0 -> 1
