File: why2025.kicad_pcb (KiCad board)
At the start: 4 copper layers, 114.9 x 125.5 mm, 237 parts, among them J1 USB device, J2 ESP32USB, J4 Headphones, J5 External Add-On, J6 Internal Add-On, J7 Speaker, J8 Micro_SD_Card, SW2 Button, U11 AP3032KTR, U12 AP3127B, U13 W25Q128JVS, U15 DS8561-25S3, U3 TLV62569DBV, U4 CH334R, U5 ESP32-C6-WROOM-1, U9 TLV62569DBV, Y1 12MHz, Y2 32.768KHz, Y4 32.768KHz

Commit message: More work on the schematic, add protection circuit, fix display pinout
Parts:
- removed J4: Headphones, adamgreig:PJ-327C-4A
- removed L7: 22uH, Inductor_SMD:L_Changjiang_FNR252010S
- removed R42: 365k, Resistor_SMD:R_0402_1005Metric
- removed R45: 100k, Resistor_SMD:R_0402_1005Metric
- removed U9: TLV62569DBV, Package_TO_SOT_SMD:SOT-23-5
- removed Y4: 32.768KHz, Crystal:Crystal_SMD_3215-2Pin_3.2x1.5mm
- added C21: 22p, Capacitor_SMD:C_0402_1005Metric, F.Cu at (78.4, -141.8)
- added C22: 22p, Capacitor_SMD:C_0402_1005Metric, F.Cu at (78.4, -139.8)
- added C61: 1u, Capacitor_SMD:C_0603_1608Metric, F.Cu at (165.3, -63.0)
- added C62: 1u, Capacitor_SMD:C_0603_1608Metric, F.Cu at (165.3, -60.5)
- added C63: 1u, Capacitor_SMD:C_0603_1608Metric, F.Cu at (165.3, -58.0)
- added C64: 100n, Capacitor_SMD:C_0402_1005Metric, F.Cu at (164.7, -53.2)
- added C65: 22u, Capacitor_SMD:C_1206_3216Metric, F.Cu at (170.1, -62.6)
- added C66: 22u, Capacitor_SMD:C_1206_3216Metric, F.Cu at (170.1, -59.2)
- added C67: 1u, Capacitor_SMD:C_0603_1608Metric, F.Cu at (165.3, -55.5)
- added C71: 22p, Capacitor_SMD:C_0402_1005Metric, F.Cu at (164.7, -51.2)
- added C72: 22p, Capacitor_SMD:C_0402_1005Metric, F.Cu at (164.7, -49.3)
- added C73: 100n, Capacitor_SMD:C_0402_1005Metric, F.Cu at (148.7, -167.4)
- added C74: 100n, Capacitor_SMD:C_0402_1005Metric, F.Cu at (148.7, -165.4)
- added C75: 100n, Capacitor_SMD:C_0402_1005Metric, F.Cu at (148.7, -163.4)
- added F2: 1A, Fuse:Fuse_0805_2012Metric, F.Cu at (143.2, -144.4)
- added J10: Expansion I3C, library:1X04_1MM_RA_GND, B.Cu at (59.5, -41.0)
- added J14: LH397K, library:LH397K-IC01, F.Cu at (38.3, -96.9)
- added J3: Internal I2C, library:1X04_1MM_RA_GND, B.Cu at (59.5, -50.9)
- added JP2: EN, Jumper:SolderJumper-2_P1.3mm_Open_RoundedPad1.0x1.5mm, F.Cu at (136.6, -170.5)
- added JP3: EN, Jumper:SolderJumper-2_P1.3mm_Open_RoundedPad1.0x1.5mm, F.Cu at (136.6, -167.0)
- added JP4: EN, Jumper:SolderJumper-2_P1.3mm_Open_RoundedPad1.0x1.5mm, F.Cu at (136.6, -163.4)
- added JP5: EN, Jumper:SolderJumper-2_P1.3mm_Open_RoundedPad1.0x1.5mm, F.Cu at (136.6, -159.9)
- added L4: 6.8uH, Inductor_SMD:L_1008_2520Metric, F.Cu at (143.0, -148.5)
- added Q4: AP2302B, Package_TO_SOT_SMD:SOT-23, F.Cu at (169.8, -49.9)
- added R31: 100k, Resistor_SMD:R_0402_1005Metric, F.Cu at (87.5, -114.9)
- added R32: 330, Resistor_SMD:R_0402_1005Metric, F.Cu at (149.1, -144.2)
- added R49: 4k7, Resistor_SMD:R_0402_1005Metric, F.Cu at (87.4, -120.2)
- added R67: 33, Resistor_SMD:R_0402_1005Metric, F.Cu at (161.8, -63.2)
- added R68: 33, Resistor_SMD:R_0402_1005Metric, F.Cu at (161.8, -61.3)
- added R69: 0, Resistor_SMD:R_0402_1005Metric, F.Cu at (161.8, -59.3)
- added R70: 100k, Resistor_SMD:R_0402_1005Metric, F.Cu at (161.8, -57.3)
- added R72: 100k, Resistor_SMD:R_0402_1005Metric, F.Cu at (161.8, -55.3)
- added R73: 0, Resistor_SMD:R_0402_1005Metric, F.Cu at (161.8, -53.3)
- added R98: 10k, Resistor_SMD:R_0402_1005Metric, F.Cu at (149.1, -148.2)
- added TP10: TS, TestPoint:TestPoint_Pad_D1.0mm, F.Cu at (135.9, -150.5)
- added TP11: BLL+, TestPoint:TestPoint_Pad_D1.0mm, F.Cu at (135.9, -147.4)
- added TP12: BLL-, TestPoint:TestPoint_Pad_D1.0mm, F.Cu at (139.0, -153.5)
- added TP13: BLK+, TestPoint:TestPoint_Pad_D1.0mm, F.Cu at (139.0, -150.5)
- added TP14: BLK-, TestPoint:TestPoint_Pad_D1.0mm, F.Cu at (139.0, -147.4)
- added TP3: PR1, TestPoint:TestPoint_Pad_D1.0mm, F.Cu at (132.9, -170.8)
- added TP4: PR2, TestPoint:TestPoint_Pad_D1.0mm, F.Cu at (132.9, -167.7)
- added TP5: PR3, TestPoint:TestPoint_Pad_D1.0mm, F.Cu at (132.9, -164.7)
- added TP6: PR4, TestPoint:TestPoint_Pad_D1.0mm, F.Cu at (132.9, -161.6)
- added TP7: PRR, TestPoint:TestPoint_Pad_D1.0mm, F.Cu at (132.9, -158.6)
- added TP8: PA, TestPoint:TestPoint_Pad_D1.0mm, F.Cu at (132.9, -147.4)
- added TP9: ~{QON}, TestPoint:TestPoint_Pad_D1.0mm, F.Cu at (135.9, -153.5)
- added U14: ~, Package_DFN_QFN:VQFN-20-1EP_3x3mm_P0.4mm_EP1.7x1.7mm, F.Cu at (169.9, -54.9)
- added U16: FM8002A, Package_SO:SSOP-8_3.9x5.05mm_P1.27mm, F.Cu at (156.3, -168.9)
- added U20: 74LVC1G125, Package_TO_SOT_SMD:SOT-353_SC-70-5, F.Cu at (154.2, -161.6)
- added U21: LM339, Package_SO:SOIC-14_3.9x8.7mm_P1.27mm, F.Cu at (143.0, -167.0)
- added U6: BQ25895RTW, library:Texas_S-PWQFN-N24_EP2.7x2.7mm_ThermalVias, F.Cu at (92.3, -158.3)
- C11: value 47nF -> 47n; footprint Capacitor_SMD:C_0402_1005Metric -> Capacitor_SMD:C_0603_1608Metric
- C12: value 4.7uF -> 4u7
- C13, C14, C15, C17, C18, C19, C25, C30, C58: value 10uF -> 10u
- C16: value 120pF -> 120p; footprint Capacitor_SMD:C_0402_1005Metric -> Capacitor_SMD:C_0603_1608Metric
- C20, C32, C34, C9: value 1uF -> 1u
- C28: value 22p -> 100n
- C29: value 10uF -> 100n; footprint Capacitor_SMD:C_1206_3216Metric -> Capacitor_SMD:C_0402_1005Metric
- C31, C33: value 10uF -> 10u; footprint Capacitor_SMD:C_0603_1608Metric -> Capacitor_SMD:C_1206_3216Metric
- C39, C49, C8: footprint Capacitor_SMD:C_0402_1005Metric -> Capacitor_SMD:C_0603_1608Metric
- C7: footprint Capacitor_SMD:C_0402_1005Metric -> Capacitor_SMD:C_1206_3216Metric
- J6: footprint Connector_PinSocket_2.54mm:PinSocket_2x15_P2.54mm_Vertical_SMD -> Connector_PinSocket_2.54mm:PinSocket_2x18_P2.54mm_Vertical_SMD
- JP1: moved to B.Cu
- R10, R9: value 5.1k -> 5k1
- R12, R25: value 4.7k -> 4k7
- R19: value 2.2k -> 2k2
- R21: value 5.23k -> 5k23
- R22: value 30.1k -> 30k1
- R48: value 4.7 -> 4R7
- R51: value 14R7 -> 10
- TP1: value TP_BL_CTRL -> BLKC; footprint TestPoint:TestPoint_Pad_D1.5mm -> TestPoint:TestPoint_Pad_D1.0mm
- TP2: value TP_BL_CTRL -> BLLC; footprint TestPoint:TestPoint_Pad_D1.5mm -> TestPoint:TestPoint_Pad_D1.0mm
- U12: value AP3127B -> AP3032KTR
- moved JP1 138.6 mm to (-26.1, -49.2), turned to 90 degrees
- moved R51 59.5 mm to (133.4, -142.1)
- moved TP2 57.8 mm to (132.9, -150.5)
- moved TP1 57.4 mm to (132.9, -153.5)
- moved U12 57.2 mm to (143.1, -152.6)
- moved D84 55.1 mm to (137.9, -141.1)
- moved C34 52.3 mm to (133.4, -144.6)
- moved C33 48.3 mm to (138.2, -144.2)
- moved C29 41.1 mm to (148.7, -169.3)
- moved C28 37.7 mm to (148.7, -171.3)
- moved J6 3.81 mm to (3.81, -37.0)
Connections:
- net /LEDs/DATA renamed /LEDs/DIN
- net EXT_INT renamed E9
- net INT_SDA renamed E10
- net Net-(U8K-CHIP_PU) renamed /Application processor/Protection/~{RESET}
- C28 pad 1: +2.8v -> Net-(U21B-+)
- C28 pad 2: Net-(U9-FB) -> GND
- C29 pad 1: +2.8v -> Net-(U21C-+)
- J5 pad 1: MTDO -> /LEDs/DOUT
- J5 pad 10: E18 -> GND
- J5 pad 3: MTMS -> VLED
- J5 pad 4: MTCK -> MTDO
- J5 pad 5: E13 -> GND
- J5 pad 6: E14 -> MTCK
- J5 pad 7: E15 -> SAO_IO3
- J5 pad 8: E16 -> MTMS
- J5 pad 9: E17 -> VSYS
- J7 pad 1: GND -> /Audio/SPK+
- J7 pad 2: /Audio/HP_NC -> /Audio/SPK-
- J7 pad MP: GND -> GNDA
- R46 pad 2: /Coprocessor/VLED_EN -> /Power/VLED_EN
- U1 pad 41: /Coprocessor/STAT_LED -> HP_DET
- U1 pad 5: /Coprocessor/VLED_EN -> AMP_EN
- U4 pad 1: unconnected-(U4-DM4--Pad1) -> HUB_USB_N
- U4 pad 2: unconnected-(U4-DP4+-Pad2) -> HUB_USB_P
- U5 pad 26: E16 -> /Radio/GPIO3
- U5 pad 27: E15 -> /Radio/GPIO2
- U5 pad 4: E17 -> Net-(U5-MTMS/GPIO4/ADC1_CH4)
- U5 pad 5: E18 -> /Power/VLED_EN
- U5 pad 8: E13 -> /Radio/GPIO0
- U5 pad 9: E14 -> /Radio/GPIO1
Routing:
- net E12: track 47.3 -> 0.00 mm, vias 2 -> 0
- net E10: track 0.00 -> 47.3 mm, vias 0 -> 2
- net INT_SCL: track 0.00 -> 40.1 mm, vias 0 -> 2
- net E9: track 40.1 -> 0.00 mm, vias 2 -> 0
- net /Audio/SPK-: track 0.00 -> 10.6 mm
- net /Audio/HP_NC: track 10.6 -> 0.00 mm
- net HP_DET: track 0.00 -> 3.61 mm
- net /Coprocessor/STAT_LED: track 3.61 -> 0.00 mm

Commit message: Assign footprints, create P4 footprint
Parts:
- added U8: ESP32P4-REV0, library:esp32p4rev0, B.Cu at (0.00, -55.0)
Connections:
- net E10 renamed INT_SDA
- net E9 renamed EXT_INT
- net INT_SCL renamed E11
Routing:
- net INT_SDA: track 47.3 -> 0.00 mm, vias 2 -> 0
- net E12: track 0.00 -> 47.3 mm, vias 0 -> 2
- net E11: track 40.1 -> 0.00 mm, vias 2 -> 0
- net (no net): track 0.00 -> 40.1 mm, vias 0 -> 2
