File: coprocessor.kicad_sch (KiCad schematic)
At the start: 1 part

Commit message: Add radio, wire up more stuff
Connections:
- net Keyboard/COL0 renamed KB_COL3
- net Keyboard/COL1 renamed KB_COL7
- net Keyboard/COL2 renamed KB_COL2
- net Keyboard/COL3 renamed KB_COL6
- net Keyboard/COL4 renamed KB_COL1
- net Keyboard/COL5 renamed KB_COL5
- net Keyboard/COL6 renamed KB_COL0
- net Keyboard/COL7 renamed KB_COL4
- net Keyboard/ROW0 renamed KB_ROW7
- net Keyboard/ROW1 renamed KB_ROW6
- net Keyboard/ROW2 renamed KB_ROW3
- net Keyboard/ROW3 renamed KB_ROW4
- net Keyboard/ROW4 renamed KB_ROW8
- net Keyboard/ROW5 renamed KB_ROW5
- net Keyboard/ROW6 renamed KB_ROW0
- net Keyboard/ROW7 renamed KB_ROW1
- net Keyboard/ROW8 renamed KB_ROW2
- net USB1_N renamed USB_1_N
- net USB1_P renamed USB_1_P
- net USB2_N renamed USB_2_N
- net USB2_P renamed USB_2_P

Commit message: Relabeling of ESP32-C6 GPIO, route signals to expansion header for testing
Connections:
- net SMBA: no longer names the net of U1.41 (PB5)
- net SPI1_MISO renamed SPI_MISO
- net SPI1_MOSI renamed SPI_MOSI
- net SPI1_NSS renamed SPI_NSS
- net SPI1_SCK renamed SPI_SCK
Changed lines of the file:
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@@
-		)
-	)
-	(global_label "SPI1_NSS"
-		(shape input)
-		(at 109.22 105.41 270)
-		(fields_autoplaced yes)
-		(effects
-			(font
-				(size 1.27 1.27)
-			)
-			(justify right)
-		)
-		(property "Intersheetrefs" "${INTERSHEET_REFS}"
-			(at 109.22 117.4061 90)
-			(effects
-				(font
-					(size 1.27 1.27)
-				)
-				(justify right)
-				(hide yes)
-			)
-		)
-	)
-	(global_label "INT"
-		(shape bidirectional)
-		(at 97.79 91.44 180)
-		(fields_autoplaced yes)
-		(effects
-			(font
-				(size 1.016 1.016)
-			)
-			(justify right)
-		)
-		(property "Intersheetrefs" "${INTERSHEET_REFS}"
-			(at 92.1908 91.44 0)
-			(effects
-				(font
-					(size 1.27 1.27)
-				)
-				(justify right)
-				(hide yes)
-			)
-		)
-	)
-	(global_label "SMBA"
-		(shape bidirectional)
-		(at 124.46 59.69 90)
-		(fields_autoplaced yes)
-		(effects
-			(font
-				(size 1.016 1.016)
-			)
-			(justify left)
-		)
-		(property "Intersheetrefs" "${INTERSHEET_REFS}"
-			(at 124.46 52.3975 90)
-			(effects
-				(font
-					(size 1.27 1.27)
-				)
-				(justify left)
-				(hide yes)
-			)
 		)
 	)
@@
 		)
 	)
-	(global_label "SPI1_SCK"
-		(shape input)
-		(at 111.76 105.41 270)
-		(fields_autoplaced yes)
-		(effects
-			(font
-				(size 1.27 1.27)
-			)
-			(justify right)
-		)
-		(property "Intersheetrefs" "${INTERSHEET_REFS}"
-			(at 111.76 117.4061 90)
-			(effects
-				(font
-					(size 1.27 1.27)
-				)
-				(justify right)
-				(hide yes)
-			)
-		)
-	)
 	(global_label "KB_COL2"
 		(shape output)
@@
 		)
 	)
-	(global_label "SPI1_MOSI"
-		(shape input)
-		(at 116.84 105.41 270)
-		(fields_autoplaced yes)
-		(effects
-			(font
-				(size 1.27 1.27)
-			)
-			(justify right)
-		)
-		(property "Intersheetrefs" "${INTERSHEET_REFS}"
-			(at 116.84 118.2528 90)
-			(effects
-				(font
-					(size 1.27 1.27)
-				)
-				(justify right)
-				(hide yes)
-			)
-		)
-	)
 	(global_label "KB_COL1"
 		(shape output)
@@
 		(property "Intersheetrefs" "${INTERSHEET_REFS}"
 			(at 255.0955 154.94 0)
-			(effects
-				(font
-					(size 1.27 1.27)
-				)
-				(justify right)
-				(hide yes)
-			)
-		)
-	)
-	(global_label "SPI1_MISO"
-		(shape input)
-		(at 114.3 105.41 270)
-		(fields_autoplaced yes)
-		(effects
-			(font
-				(size 1.27 1.27)
-			)
-			(justify right)
-		)
-		(property "Intersheetrefs" "${INTERSHEET_REFS}"
-			(at 114.3 118.2528 90)
 			(effects
 				(font
@@
 		)
 	)
+	(hierarchical_label "INT"
+		(shape bidirectional)
+		(at 97.79 91.44 180)
+		(fields_autoplaced yes)
+		(effects
+			(font
+				(size 1.27 1.27)
+			)
+			(justify right)
+		)
+	)
 	(hierarchical_label "USB_2_P"
 		(shape bidirectional)
@@
 		)
 	)
+	(hierarchical_label "SPI_MISO"
+		(shape output)
+		(at 114.3 105.41 270)
+		(fields_autoplaced yes)
+		(effects
+			(font
+				(size 1.27 1.27)
+			)
+			(justify right)
+		)
+	)
 	(hierarchical_label "USB_2_N"
 		(shape bidirectional)
@@
 		)
 	)
+	(hierarchical_label "SPI_NSS"
+		(shape input)
+		(at 109.22 105.41 270)
+		(fields_autoplaced yes)
+		(effects
+			(font
+				(size 1.27 1.27)
+			)
+			(justify right)
+		)
+	)
 	(hierarchical_label "SWCLK"
 		(shape input)
@@
 			)
 			(justify left)
+		)
+	)
+	(hierarchical_label "SPI_MOSI"
+		(shape input)
+		(at 116.84 105.41 270)
+		(fields_autoplaced yes)
+		(effects
+			(font
+				(size 1.27 1.27)
+			)
+			(justify right)
 		)
 	)
@@
 		)
 	)
+	(hierarchical_label "SPI_SCK"
+		(shape input)
+		(at 111.76 105.41 270)
+		(fields_autoplaced yes)
+		(effects
+			(font
+				(size 1.27 1.27)
+			)
+			(justify right)
+		)
+	)

Commit message: Boot pin, bit more routing
Parts:
- added R14: 10k, Resistor_SMD:R_0402_1005Metric, symbol symbols:R
Connections:
- net GND: now also R14.2
- net PA3: now reaches U1.13 (PA3)
- net BOOT: now reaches U1.44 (BOOT0)
- net BOOT: now also R14.1
Other:
- note added: "Normal boot: BOOT0 low Bootloader: BOOT0 high, BOOT1 low SRAM: BOOT0 high, BOOT1 high"
Changed lines of the file:
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@@
 		(comment 2 "License: CERN-OHL-P")
 	)
+	(junction
+		(at 121.92 25.4)
+		(diameter 0)
+		(color 0 0 0 0)
+	)
 	(wire
 		(pts
@@
 	(wire
 		(pts
+			(xy 121.92 25.4) (xy 124.46 25.4)
+		)
+		(stroke
+			(width 0)
+			(type default)
+		)
+	)
+	(wire
+		(pts
 			(xy 264.16 142.24) (xy 266.7 142.24)
 		)
@@
 	(wire
 		(pts
+			(xy 121.92 27.94) (xy 121.92 25.4)
+		)
+		(stroke
+			(width 0)
+			(type default)
+		)
+	)
+	(wire
+		(pts
 			(xy 264.16 132.08) (xy 266.7 132.08)
 		)
@@
 	(wire
 		(pts
+			(xy 116.84 25.4) (xy 121.92 25.4)
+		)
+		(stroke
+			(width 0)
+			(type default)
+		)
+	)
+	(wire
+		(pts
 			(xy 264.16 129.54) (xy 266.7 129.54)
 		)
@@
 	(wire
 		(pts
+			(xy 116.84 25.4) (xy 116.84 59.69)
+		)
+		(stroke
+			(width 0)
+			(type default)
+		)
+	)
+	(wire
+		(pts
 			(xy 264.16 152.4) (xy 266.7 152.4)
 		)
@@
 			(width 0)
 			(type default)
+		)
+	)
+	(text "Normal boot: BOOT0 low\nBootloader: BOOT0 high, BOOT1 low\nSRAM: BOOT0 high, BOOT1 high"
+		(exclude_from_sim no)
+		(at 129.794 29.718 0)
+		(effects
+			(font
+				(face "KiCad Font")
+				(size 1.27 1.27)
+			)
+			(justify left)
 		)
 	)
@@
 			)
 			(justify right)
+		)
+	)
+	(hierarchical_label "PA3"
+		(shape bidirectional)
+		(at 106.68 105.41 270)
+		(fields_autoplaced yes)
+		(effects
+			(font
+				(size 1.27 1.27)
+			)
+			(justify right)
+		)
+	)
+	(hierarchical_label "BOOT"
+		(shape output)
+		(at 124.46 25.4 0)
+		(fields_autoplaced yes)
+		(effects
+			(font
+				(size 1.27 1.27)
+			)
+			(justify left)
 		)
 	)
@@
 	)
 	(symbol
+		(lib_name "GND_1")
+		(lib_id "power:GND")
+		(at 121.92 35.56 0)
+		(unit 1)
+		(exclude_from_sim no)
+		(in_bom yes)
+		(on_board yes)
+		(dnp no)
+		(fields_autoplaced yes)
+		(property "Reference" "#PWR045"
+			(at 121.92 41.91 0)
+			(effects
+				(font
+					(size 1.27 1.27)
+				)
+				(hide yes)
+			)
+		)
+		(property "Value" "GND"
+			(at 121.92 40.64 0)
+			(effects
+				(font
+					(size 1.27 1.27)
+				)
+			)
+		)
+		(property "Footprint" ""
+			(at 121.92 35.56 0)
+			(effects
+				(font
+					(size 1.27 1.27)
+				)
+				(hide yes)
+			)
+		)
+		(property "Datasheet" ""
+			(at 121.92 35.56 0)
+			(effects
+				(font
+					(size 1.27 1.27)
+				)
+				(hide yes)
+			)
+		)
+		(property "Description" "Power symbol creates a global label with name \"GND\" , ground"
+			(at 121.92 35.56 0)
+			(effects
+				(font
+					(size 1.27 1.27)
+				)
+				(hide yes)
+			)
+		)
+		(pin "1"
+		)
+		(instances
+			(project "why2025"
+				(path "/6a31734e-65de-48f3-8156-2b24b665b183/17d99d7a-f62d-4bb1-94fb-986230f9fa4f"
+					(reference "#PWR045")
+					(unit 1)
+				)
+			)
+		)
+	)
+	(symbol
 		(lib_id "ch32v203:CH32V203CxT6")
 		(at 120.65 82.55 0)
@@
 					(unit 1)
 				)
+			)
+		)
+	)
+	(symbol
+		(lib_id "symbols:R")
+		(at 121.92 31.75 0)
+		(mirror y)
+		(unit 1)
+		(exclude_from_sim no)
+		(in_bom yes)
+		(on_board yes)
+		(dnp no)
+		(property "Reference" "R14"
+			(at 125.73 33.02 0)
+			(effects
+				(font
+					(size 1.27 1.27)
+				)
+			)
+		)
+		(property "Value" "10k"
+			(at 125.73 30.48 0)
+			(effects
+				(font
+					(size 1.27 1.27)
+				)
+			)
+		)
+		(property "Footprint" "Resistor_SMD:R_0402_1005Metric"
+			(at 123.698 31.75 90)
+			(effects
+				(font
+					(size 1.27 1.27)
+				)
+				(hide yes)
+			)
+		)
+		(property "Datasheet" "https://datasheet.lcsc.com/lcsc/2110260030_UNI-ROYAL-Uniroyal-Elec-0402WGF1002TCE_C25744.pdf"
+			(at 121.92 31.75 0)
+			(effects
+				(font
+					(size 1.27 1.27)
+				)
+				(hide yes)
+			)
+		)
+		(property "Description" ""
+			(at 121.92 31.75 0)
+			(effects
+				(font
+					(size 1.27 1.27)
+				)
+				(hide yes)
+			)
+		)
+		(property "LCSC" "C25744"
+			(at 121.92 31.75 0)
+			(effects
+				(font
+					(size 1.27 1.27)
+				)
+				(hide yes)
+			)
+		)
+		(pin "1"
+		)
+		(pin "2"
+		)
+		(instances
+			(project "why2025"
+				(path "/6a31734e-65de-48f3-8156-2b24b665b183/17d99d7a-f62d-4bb1-94fb-986230f9fa4f"
+					(reference "R14")
+					(unit 1)
+				)

Commit message: Work in progress
Parts:
- added C1, C2, C23, C3, C4, C5: 100n, Capacitor_SMD:C_0402_1005Metric, symbol symbols:C
- added C21, C22: tbd, symbol Device:C
- added JP1: BOOT, Jumper:SolderJumper-2_P1.3mm_Open_RoundedPad1.0x1.5mm, symbol Jumper:Jumper_2_Open
- added R12, R25: 4.7k, Resistor_SMD:R_0402_1005Metric, symbol symbols:R
- added R15, R28, R29: 10k, Resistor_SMD:R_0402_1005Metric, symbol symbols:R
- added Y2: 32.768KHz, Crystal:Crystal_SMD_3215-2Pin_3.2x1.5mm, symbol symbols:Crystal_Small
Connections:
- net PA3 is gone; now on net KB_ROW4: U1.13 (PA3)
- net SPI_MISO is gone; now on net KB_ROW6: U1.16 (PA6)
- net SPI_MOSI is gone; now on net KB_COL3: U1.17 (PA7)
- net SPI_NSS is gone; now on net KB_ROW3: U1.14 (PA4)
- net SPI_SCK is gone; now on net KB_ROW7: U1.15 (PA5)
- net USB_2_N is gone; now on net SCL: U1.42 (PB6)
- net USB_2_P is gone; now on net SDA: U1.43 (PB7)
- net +3.3V: now also C1.1, C3.1, C4.1, C5.1, JP1.2 (B), R12.1, R15.1, R25.1, R28.1, R29.1
- net GND: now also C1.2, C2.2, C21.2, C22.2, C23.2, C3.2, C4.2, C5.2
- net INT: now also R28.2
- net KB_COL2: now also U1.19 (PB1); no longer U1.21 (PB10)
- net KB_COL3: no longer U1.19 (PB1)
- net KB_COL6: now also U1.20 (PB2); no longer U1.22 (PB11)
- net KB_COL7: now also U1.18 (PB0); no longer U1.20 (PB2)
- net KB_ROW3: no longer U1.18 (PB0)
- net KB_ROW4: no longer U1.38 (PA15)
- net KB_ROW5: now also U1.11 (PA1); no longer U1.40 (PB4)
- net KB_ROW6: no longer U1.12 (PA2)
- net KB_ROW7: no longer U1.11 (PA1)
- net KB_ROW8: now also U1.12 (PA2); no longer U1.39 (PB3)
- net SCL: no longer U1.45 (PB8)
- net SDA: no longer U1.46 (PB9)
- net +3.3vsb: now reaches U1.1 (VBAT)
- net +3.3vsb: now also C2.1
- net ALARM: now reaches U1.2 (PC13)
- net STAT_LED: now reaches U1.41 (PB5)
- net D0: now reaches U1.5 (PD0)
- net D1: now reaches U1.6 (PD1)
- net at U1.7 (NRST): now also C23.1, R29.2
- net BOOT: no longer names the net of R14.1, U1.44 (BOOT0)
- net BOOT: now also JP1.1 (A)
- net OSC32IN: no longer names the net of U1.3 (PC14)
- net OSC32IN: now also C22.1, Y2.2
- net OSC32OUT: no longer names the net of U1.4 (PC15)
- net OSC32OUT: now also C21.1, Y2.1
- new net B3: U1.39 (PB3)
- new net B4: U1.40 (PB4)
- new net C6_BOOT: U1.45 (PB8)
- new net C6_EN: U1.46 (PB9)
- new net PM_INT: R15.2, U1.38 (PA15)
- new net PM_SCL: R25.2, U1.21 (PB10)
- new net PM_SDA: R12.2, U1.22 (PB11)
Other:
- moved on the sheet: R14, U1

Commit message: More fixes, add display, update display backlight driver circuit, fix some of the footprint associations
Parts:
- added SW2: Button, Button_Switch_SMD:SW_SPST_PTS645, symbol Switch:SW_Push
- C21, C22: footprint (none) -> Capacitor_SMD:C_0402_1005Metric
Connections:
- net +3.3vsb renamed +2.5vsb
- net B3 renamed KEYBOARD_BL
- net B4 renamed DISPLAY_BL
- net D0 renamed VLED_EN
- net D1 renamed LCD_RST
- new net Keyboard/EXT_I: SW2.1
- new net Keyboard/EXT_O: SW2.2
Other:
- sheet Keyboard ports: added EXT_I, EXT_O; removed EXT

Commit message: More work on the schematic, add protection circuit, fix display pinout
Parts:
- C21, C22: value tbd -> 22p
- R12, R25: value 4.7k -> 4k7
Connections:
- net STAT_LED renamed HP_DET
- net VLED_EN renamed AMP_EN
Other:
- note added: "To-do Maybe this could be a jumper instead? Could be used to unlock developer mode for the co-processor."
Changed lines of the file:
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@@
 	(title_block
 		(title "WHY2025 badge")
-		(date "2024-04-02")
-		(rev "0.1")
+		(date "2024-05-05")
+		(rev "Prototype 1")
 		(company "Badge.Team")
 		(comment 1 "Copyright 2024 Nicolai Electronics")
 		(comment 2 "License: CERN-OHL-P")
+		(comment 3 "PROTOYPE DESIGN UNTESTED")
+		(comment 4 "(Work in progress!)")
 	)
 	(junction
@@
 		)
 	)
+	(text "To-do\nMaybe this could be a jumper instead?\nCould be used to unlock developer mode\nfor the co-processor."
+		(exclude_from_sim no)
+		(at 211.836 159.004 0)
+		(effects
+			(font
+				(size 1.27 1.27)
+			)
+		)
+	)
 	(global_label "KB_COL3"
 		(shape input)
@@
 		)
 	)
-	(hierarchical_label "VLED_EN"
+	(hierarchical_label "AMP_EN"
 		(shape output)
 		(at 57.15 80.01 180)
@@
 		)
 	)
-	(hierarchical_label "STAT_LED"
-		(shape output)
+	(hierarchical_label "HP_DET"
+		(shape input)
 		(at 212.09 48.26 0)
 		(fields_autoplaced yes)
@@
 			)
 		)
-		(property "Datasheet" "https://datasheet.lcsc.com/lcsc/2304140030_Samsung-Electro-Mechanics-CL05B104KB54PNC_C307331.pdf"
+		(property "Datasheet" ""
 			(at 191.77 138.43 0)
 			(effects
@@
 			)
 		)
+		(property "Manufacturer" ""
+			(at 191.77 138.43 0)
+			(effects
+				(font
+					(size 1.27 1.27)
+				)
+				(hide yes)
+			)
+		)
 		(pin "1"
 		)
@@
 			)
 		)
-		(property "Value" "4.7k"
+		(property "Value" "4k7"
 			(at 86.36 26.67 0)
 			(effects
@@
 			)
 		)
+		(property "Manufacturer" ""
+			(at 82.55 27.94 0)
+			(effects
+				(font
+					(size 1.27 1.27)
+				)
+				(hide yes)
+			)
+		)
 		(pin "1"
 		)
@@
 			)
 		)
-		(property "Datasheet" "https://datasheet.lcsc.com/lcsc/2304140030_Samsung-Electro-Mechanics-CL05B104KB54PNC_C307331.pdf"
+		(property "Datasheet" ""
 			(at 116.84 138.43 0)
 			(effects
@@
 			)
 		)
+		(property "Manufacturer" ""
+			(at 116.84 138.43 0)
+			(effects
+				(font
+					(size 1.27 1.27)
+				)
+				(hide yes)
+			)
+		)
 		(pin "1"
 		)
@@
 			)
 		)
+		(property "Manufacturer" ""
+			(at 162.56 27.94 0)
+			(effects
+				(font
+					(size 1.27 1.27)
+				)
+				(hide yes)
+			)
+		)
 		(pin "1"
 		)
@@
 			)
 		)
-		(property "Value" "4.7k"
+		(property "Value" "4k7"
 			(at 78.74 26.67 0)
 			(effects
@@
 			)
 		)
+		(property "Manufacturer" ""
+			(at 74.93 27.94 0)
+			(effects
+				(font
+					(size 1.27 1.27)
+				)
+				(hide yes)
+			)
+		)
 		(pin "1"
 		)
@@
 			)
 		)
+		(property "Manufacturer" ""
+			(at 151.13 83.82 0)
+			(effects
+				(font
+					(size 1.27 1.27)
+				)
+				(hide yes)
+			)
+		)
 		(pin "8"
 		)
@@
 			)
 		)
-		(property "Datasheet" "https://datasheet.lcsc.com/lcsc/2304140030_Samsung-Electro-Mechanics-CL05B104KB54PNC_C307331.pdf"
+		(property "Datasheet" ""
 			(at 106.68 138.43 0)
 			(effects
@@
 			)
 		)
+		(property "Manufacturer" ""
+			(at 106.68 138.43 0)
+			(effects
+				(font
+					(size 1.27 1.27)
+				)
+				(hide yes)
+			)
+		)
 		(pin "1"
 		)
@@
 			)
 		)
-		(property "Value" "tbd"
+		(property "Value" "22p"
 			(at 89.408 140.716 0)
 			(effects
@@
 			)
 		)
-		(property "Datasheet" "~"
+		(property "Datasheet" ""
 			(at 88.9 138.43 0)
 			(effects
@@
 			)
 		)
+		(property "Manufacturer" ""
+			(at 88.9 138.43 0)
+			(effects
+				(font
+					(size 1.27 1.27)
+				)
+				(hide yes)
+			)
+		)
 		(pin "2"
 		)
@@
 			)
 		)
-		(property "Value" "tbd"
+		(property "Value" "22p"
 			(at 94.488 140.97 0)
 			(effects
@@
 			)
 		)
-		(property "Datasheet" "~"
+		(property "Datasheet" ""
 			(at 93.98 138.43 0)
 			(effects
@@
 			)
 		)
+		(property "Manufacturer" ""
+			(at 93.98 138.43 0)
+			(effects
+				(font
+					(size 1.27 1.27)
+				)
+				(hide yes)
+			)
+		)
 		(pin "2"
 		)
@@
 			)
 		)
-		(property "Datasheet" "https://datasheet.lcsc.com/lcsc/2304140030_Samsung-Electro-Mechanics-CL05B104KB54PNC_C307331.pdf"
+		(property "Datasheet" ""
 			(at 176.53 138.43 0)
 			(effects
@@
 			)
 		)
+		(property "Manufacturer" ""
+			(at 176.53 138.43 0)
+			(effects
+				(font
+					(size 1.27 1.27)
+				)
+				(hide yes)
+			)
+		)
 		(pin "1"
 		)
@@
 			)
 		)
-		(property "Datasheet" "https://datasheet.lcsc.com/lcsc/2304140030_Samsung-Electro-Mechanics-CL05B104KB54PNC_C307331.pdf"
+		(property "Datasheet" ""
 			(at 99.06 138.43 0)
 			(effects
@@
 			)
 		)
+		(property "Manufacturer" ""
+			(at 99.06 138.43 0)
+			(effects
+				(font
+					(size 1.27 1.27)
+				)
+				(hide yes)
+			)
+		)
 		(pin "1"
 		)
@@
 			)
 		)
+		(property "Manufacturer" ""
+			(at 242.57 160.02 0)
+			(effects
+				(font
+					(size 1.27 1.27)
+				)
+				(hide yes)
+			)
+		)
 		(pin "1"
 		)
@@
 			)
 		)
+		(property "Manufacturer" ""
+			(at 201.93 27.94 0)
+			(effects
+				(font
+					(size 1.27 1.27)
+				)
+				(hide yes)
+			)
+		)
 		(pin "1"
 		)
@@
 			)
 		)
+		(property "Manufacturer" ""
+			(at 59.69 27.94 0)
+			(effects
+				(font
+					(size 1.27 1.27)
+				)
+				(hide yes)
+			)
+		)
 		(pin "1"
 		)
@@
 			)
 		)
+		(property "Manufacturer" ""
+			(at 201.93 138.43 0)
+			(effects
+				(font
+					(size 1.27 1.27)
+				)
+				(hide yes)
+			)
+		)
 		(pin "1"
 		)
@@
 			)
 		)
+		(property "Manufacturer" ""
+			(at 67.31 27.94 0)
+			(effects
+				(font
+					(size 1.27 1.27)
+				)
+				(hide yes)
+			)
+		)
 		(pin "1"
 		)
@@
 			)
 		)
+		(property "Manufacturer" ""
+			(at 91.44 77.47 0)
+			(effects
+				(font
+					(size 1.27 1.27)
+				)
+				(hide yes)
+			)
+		)
 		(pin "1"
 		)
@@
 			)
 		)
-		(property "Datasheet" "https://datasheet.lcsc.com/lcsc/2304140030_Samsung-Electro-Mechanics-CL05B104KB54PNC_C307331.pdf"
+		(property "Datasheet" ""
 			(at 59.69 138.43 0)
 			(effects
@@
 			)
 		)
+		(property "Manufacturer" ""
+			(at 59.69 138.43 0)
+			(effects
+				(font
+					(size 1.27 1.27)
+				)
+				(hide yes)
+			)
+		)
 		(pin "1"
 		)
@@
 			(project "why2025"
 				(path "/6a31734e-65de-48f3-8156-2b24b665b183/17d99d7a-f62d-4bb1-94fb-986230f9fa4f"
-					(page "3")
+					(page "5")
 				)
 			)
