File: coprocessor.kicad_sch (KiCad schematic)
At the start: 18 parts, among them SW2 Button, U1 CH32V203C8T6, Y2 32.768KHz

Commit message: Small tweaks and fixes, update LCSC numbers on some components, change to new key type for power key
Parts:
- SW2: value Button -> User; footprint Button_Switch_SMD:SW_SPST_PTS645 -> library:KEY-TH_TC-1101V-C-A-W
Connections:
- net Keyboard/EXT_I is gone; now on net +3.3V: SW2.1
- net ALARM renamed POWER_ON
- net Keyboard/EXT_O renamed Keyboard/EXT
Other:
- sheet Keyboard ports: added EXT; removed EXT_I, EXT_O
- note removed: "To-do Maybe this could be a jumper instead? Could be used to unlock developer mode for the co-processor."
- moved on the sheet: SW2

Commit message: More routing and fixes
Connections:
- net USB_1_N renamed CH32_USB1_N
- net USB_1_P renamed CH32_USB1_P
Changed lines of the file:
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@@
 		)
 	)
-	(hierarchical_label "USB_1_N"
+	(hierarchical_label "CH32_USB1_N"
 		(shape bidirectional)
 		(at 210.82 80.01 0)
@@
 		)
 	)
-	(hierarchical_label "USB_1_P"
+	(hierarchical_label "CH32_USB1_P"
 		(shape bidirectional)
 		(at 210.82 77.47 0)

Commit message: More routing, move PM I2C to ESP32-C6 instead of CH32
Parts:
- removed R12, R25: 4k7, Resistor_SMD:R_0402_1005Metric, symbol symbols:R
- removed R15: 10k, Resistor_SMD:R_0402_1005Metric, symbol symbols:R
- SW2: symbol Switch:SW_Push -> pushbutton_gnd:pushbutton_gnd
Connections:
- net GND: now also SW2.3, SW2.4
- net PM_INT: no longer names the net of U1.38 (PA15)
- net PM_SCL: no longer names the net of U1.21 (PB10)
- net PM_SDA: no longer names the net of U1.22 (PB11)
Other:
- note added: "To-do"

Commit message: More routing, moved some more signals
Connections:
- net C6_BOOT: now also U1.46 (PB9); no longer U1.45 (PB8)
- net C6_EN: now also U1.45 (PB8); no longer U1.46 (PB9)
- net LCD_RST: no longer names the net of U1.6 (PD1)
Changed lines of the file:
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@@
+	(text "To-do"
+		(exclude_from_sim no)
+		(at 53.34 82.55 0)
+		(effects
+			(font
+				(size 1.27 1.27)
+			)
+		)
+	)
 	(text "To-do"
 		(exclude_from_sim no)
@@
 	(hierarchical_label "C6_EN"
 		(shape output)
-		(at 212.09 35.56 0)
+		(at 212.09 38.1 0)
 		(fields_autoplaced yes)
 		(effects
@@
 	(hierarchical_label "C6_BOOT"
 		(shape output)
-		(at 212.09 38.1 0)
+		(at 212.09 35.56 0)
 		(fields_autoplaced yes)
 		(effects
@@
 		)
 	)
-	(hierarchical_label "LCD_RST"
-		(shape output)
-		(at 57.15 82.55 180)
-		(fields_autoplaced yes)
-		(effects
-			(font
-				(size 1.27 1.27)
-			)
-			(justify right)
-		)
-	)

Commit message: Add more testpoints for CH32, add text, move addressable LEDs further apart
Parts:
- added R32: 100k, Resistor_SMD:R_0402_1005Metric, symbol Device:R
- added TP10: SWDIO, TestPoint:TestPoint_Pad_1.0x1.0mm, symbol Connector:TestPoint
- added TP15: SWCLK, TestPoint:TestPoint_Pad_1.0x1.0mm, symbol Connector:TestPoint
- added TP3, TP5, TP6: PB10, TestPoint:TestPoint_Pad_1.0x1.0mm, symbol Connector:TestPoint
- added TP4: PB11, TestPoint:TestPoint_Pad_1.0x1.0mm, symbol Connector:TestPoint
- added TP8: PD1, TestPoint:TestPoint_Pad_1.0x1.0mm, symbol Connector:TestPoint
Connections:
- net +3.3V: now also R32.2, TP5.1
- net GND: now also TP6.1
- net SWCLK: now also TP15.1
- net SWDIO: now also TP10.1
- net at U1.21 (PB10): now also TP3.1
- net at U1.22 (PB11): now also TP4.1
- net SD_DET: now reaches U1.38 (PA15)
- net SD_DET: now also R32.1
- net at U1.6 (PD1): now also TP8.1
Other:
- note removed: "To-do"

Commit message: Remove some items from BOM, generate fabrication files
Parts:
- TP10, TP15, TP3, TP4, TP5, TP6, TP8: now left out of the parts list
Changed lines of the file:
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@@
 		(unit 1)
 		(exclude_from_sim no)
-		(in_bom yes)
+		(in_bom no)
 		(on_board yes)
 		(dnp no)
@@
 		(unit 1)
 		(exclude_from_sim no)
-		(in_bom yes)
+		(in_bom no)
 		(on_board yes)
 		(dnp no)
@@
 		(unit 1)
 		(exclude_from_sim no)
-		(in_bom yes)
+		(in_bom no)
 		(on_board yes)
 		(dnp no)
@@
 		(unit 1)
 		(exclude_from_sim no)
-		(in_bom yes)
+		(in_bom no)
 		(on_board yes)
 		(dnp no)
@@
 		(unit 1)
 		(exclude_from_sim no)
-		(in_bom yes)
+		(in_bom no)
 		(on_board yes)
 		(dnp no)
@@
 		(unit 1)
 		(exclude_from_sim no)
-		(in_bom yes)
+		(in_bom no)
 		(on_board yes)
 		(dnp no)
@@
 		(unit 1)
 		(exclude_from_sim no)
-		(in_bom yes)
-		(on_board yes)
-		(dnp no)
+		(in_bom no)
+		(on_board yes)
+		(dnp no)

Commit message: More fabrication stuff for prototype 1
Parts:
- JP1: now left out of the parts list
- SW2: LCSC (none) -> C318992
Changed lines of the file:
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@@
 			)
 		)
-		(property "Datasheet" "~"
+		(property "Datasheet" "-"
 			(at 199.39 58.42 0)
 			(effects
@@
 			)
 		)
-		(property "Datasheet" "~"
+		(property "Datasheet" "-"
 			(at 25.4 124.46 0)
 			(effects
@@
 			)
 		)
-		(property "Datasheet" "~"
+		(property "Datasheet" "-"
 			(at 44.45 137.16 0)
 			(effects
@@
 			)
 		)
-		(property "Datasheet" "~"
+		(property "Datasheet" "-"
 			(at 25.4 137.16 0)
 			(effects
@@
 			)
 		)
-		(property "Datasheet" "~"
+		(property "Datasheet" "-"
 			(at 44.45 124.46 0)
 			(effects
@@
 			)
 		)
-		(property "Datasheet" "~"
+		(property "Datasheet" "https://www.lcsc.com/product-detail/Tactile-Switches_XKB-Connection-TC-1101V-C-A-W_C318992.html"
 			(at 245.11 154.94 0)
 			(effects
@@
 			)
 		)
-		(property "Description" "Power switch"
+		(property "Description" "User button"
+			(at 245.11 160.02 0)
+			(effects
+				(font
+					(size 1.27 1.27)
+				)
+				(hide yes)
+			)
+		)
+		(property "LCSC" "C318992"
 			(at 245.11 160.02 0)
 			(effects
@@
 		(unit 1)
 		(exclude_from_sim yes)
-		(in_bom yes)
+		(in_bom no)
 		(on_board yes)
 		(dnp no)
@@
 			)
 		)
-		(property "Datasheet" "~"
+		(property "Datasheet" "-"
 			(at 209.55 74.93 0)
 			(effects
@@
 			)
 		)
-		(property "Datasheet" "~"
+		(property "Datasheet" "-"
 			(at 43.18 87.63 0)
 			(effects
