File: coprocessor.kicad_sch (KiCad schematic)
At the start: 18 parts, among them SW2 User, U1 CH32V203C8T6, Y2 32.768KHz

Commit message: Add latch to power on from the ch32.
Parts:
- added R84: 10k, Resistor_SMD:R_0402_1005Metric, symbol symbols:R
- added U26: 74LVC2G02HD4-7, lcsc:X2-DFN2010-8_L2.0-W1.0-P0.50-BL, symbol lcsc:74LVC2G02HD4-7
Connections:
- net +2.5vsb: now also U26.8 (VCC)
- net +3.3V: now also R84.2
- net GND: now also U26.4 (GND)
- net POWER_ON: now also U26.2 (1B), U26.3 (2Y); no longer U1.2 (PC13)
- new net: U26.5 (2A), U26.7 (1Y)
- new net POWER_ON_PULSE: U1.2 (PC13), U26.6 (2B)
- new net RTC_RESET: R84.1, U26.1 (1A)
Other:
- note added: "Power on latch circuit To keep the power signal low until the 3v3 comes up"

Commit message: Shortened VBATT, rerouted VBUS to a less crowded part of the PCB and it's now 1.2mm. Moved vias tohove ground in between for better EM.
Parts:
- added TP8: PON, TestPoint:TestPoint_Pad_D1.0mm, symbol Connector:TestPoint
Connections:
- net POWER_ON: now also TP8.1
- net POWER_ON_PULSE: now also U26.5 (2A); no longer U26.6 (2B)
- net at U26.7 (1Y): now also U26.6 (2B); no longer U26.5 (2A)
Other:
- moved on the sheet: R84, U26

Commit message: Fix SR latch circuit
Connections:
- net POWER_ON: now also U26.6 (2B), U26.7 (1Y); no longer U26.2 (1B), U26.3 (2Y)
- new net: U26.2 (1B), U26.3 (2Y)
Other:
- moved on the sheet: R84, TP8, U26

Commit message: WIP: change LED, camera, LoRa and C6 pins and add USB-A port 1A current limit
Connections:
- net C6_BOOT renamed USB_ENABLE
- net CAMERA renamed LED_DATA
Changed lines of the file:
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@@
 	)
 	(global_label "POWER_ON_PULSE"
-		(shape input)
+		(shape output)
 		(at 57.15 72.39 180)
 		(fields_autoplaced yes)
 		(effects
 			(font
-				(size 1.27 1.27)
-			)
-			(justify right)
-		)
-		(property "Intersheetrefs" "${INTERSHEET_REFS}"
-			(at 37.1106 72.39 0)
+				(size 1.016 1.016)
+			)
+			(justify right)
+		)
+		(property "Intersheetrefs" "${INTERSHEET_REFS}"
+			(at 41.1187 72.39 0)
 			(effects
 				(font
@@
 		)
 	)
-	(hierarchical_label "CAMERA"
+	(hierarchical_label "LED_DATA"
 		(shape output)
 		(at 210.82 80.01 0)
@@
 		)
 	)
-	(hierarchical_label "C6_BOOT"
+	(hierarchical_label "USB_ENABLE"
 		(shape output)
 		(at 57.15 82.55 180)

Commit message: Change TE resistor to 100k pull-down and export production files
Parts:
- TP10, TP15: LCSC (none) -> -
- U26: LCSC (none) -> C842640; LCSC Part C842640 -> (none)
