File: radio.kicad_sch (KiCad schematic)
At the start: 9 parts, among them U5 ESP32-C6-WROOM-1

Commit message: Relabeling of ESP32-C6 GPIO, route signals to expansion header for testing
Parts:
- removed C9: 1u, Capacitor_SMD:C_0402_1005Metric, symbol symbols:C
- removed R14: 10k, Resistor_SMD:R_0402_1005Metric, symbol symbols:R
Connections:
- net RESET: now reaches R13.1, U5.3 (EN/CHIP_PU)
- net AMP_ENABLE renamed SPI_MISO
- net BATT ADC renamed GPIO2
- net BATT CHRG renamed GPIO3
- net BUTTON A renamed DATA_READY
- net BUTTON B renamed GPIO4
- net BUTTON C renamed HANDSHAKE
- net DISPLAY BUSY renamed SPI_MOSI
- net DISPLAY CS renamed SPI_NSS
- net DISPLAY DC renamed GPIO5
- net DISPLAY_RST renamed TX
- net I2S CLOCK renamed SDIO_DATA3
- net I2S DATA renamed SDIO_DATA2
- net I2S_LRCK renamed RX
- net INT renamed SPI_SCK
- net SDCARD CS renamed SDIO_CMD
- net SPI MISO renamed SDIO_DATA0
- net SPI MOSI renamed SDIO_CLK
- net SPI SCK renamed SDIO_DATA1
Other:
- moved on the sheet: R13

Commit message: Work in progress
Parts:
- removed R15: 10k, Resistor_SMD:R_0402_1005Metric, symbol symbols:R
- added R30, R33, R34, R35, R36, R37: 51k, Resistor_SMD:R_0402_1005Metric, symbol symbols:R
- added R38: 10k, Resistor_SMD:R_0402_1005Metric, symbol symbols:R
- R16: value 10k -> 100k; LCSC C25744 -> (none)
Connections:
- net +3.3V: now also R30.1, R33.1, R34.1, R35.1, R36.1, R37.1, R38.2
- net SDIO_CLK: now also R33.2
- net SDIO_CMD: now also R30.2
- net SDIO_DATA0: now also R34.2
- net SDIO_DATA1: now also R35.2
- net SDIO_DATA2: now also R36.2
- net SDIO_DATA3: now also R37.2
- net DATA_READY renamed BOOT
- net BOOT: now also R38.1; no longer R16.2
- net GPIO2 renamed 2
- net GPIO3 renamed 3
- net GPIO4 renamed 4
- net GPIO5 renamed 5
- net HANDSHAKE renamed 15
- net RESET renamed EN
- net SPI_MISO renamed 1
- net SPI_MOSI renamed 10
- net SPI_NSS renamed WAKEUP
- net WAKEUP: now also R16.2
- net SPI_SCK renamed 0
Other:
- moved on the sheet: C10, R13, R16, R17, R18, U5

Commit message: More schematics
Connections:
- net 0 renamed GPIO0
- net 1 renamed GPIO1
- net 10 renamed GPIO10
- net 15 renamed GPIO15
- net 2 renamed GPIO2
- net 3 renamed GPIO3
- net 4 renamed GPIO4
- net 5 renamed GPIO5
- net RX renamed UART_RX
- net TX renamed UART_TX
- net WAKEUP renamed INT
Changed lines of the file:
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@@
 		)
 	)
-	(hierarchical_label "15"
+	(hierarchical_label "GPIO15"
 		(shape bidirectional)
 		(at 229.87 92.71 0)
@@
 		)
 	)
-	(hierarchical_label "3"
+	(hierarchical_label "GPIO3"
 		(shape bidirectional)
 		(at 69.85 77.47 180)
@@
 		)
 	)
-	(hierarchical_label "RX"
-		(shape bidirectional)
+	(hierarchical_label "UART_RX"
+		(shape input)
 		(at 229.87 67.31 0)
 		(fields_autoplaced yes)
@@
 		)
 	)
-	(hierarchical_label "4"
+	(hierarchical_label "GPIO4"
 		(shape bidirectional)
 		(at 69.85 85.09 180)
@@
 		)
 	)
-	(hierarchical_label "TX"
-		(shape bidirectional)
+	(hierarchical_label "UART_TX"
+		(shape output)
 		(at 229.87 64.77 0)
 		(fields_autoplaced yes)
@@
 		)
 	)
-	(hierarchical_label "2"
+	(hierarchical_label "GPIO2"
 		(shape bidirectional)
 		(at 69.85 74.93 180)
@@
 		)
 	)
-	(hierarchical_label "WAKEUP"
+	(hierarchical_label "INT"
 		(shape output)
 		(at 229.87 85.09 0)
@@
 		)
 	)
-	(hierarchical_label "10"
+	(hierarchical_label "GPIO10"
 		(shape bidirectional)
 		(at 229.87 90.17 0)
@@
 		)
 	)
-	(hierarchical_label "5"
+	(hierarchical_label "GPIO5"
 		(shape bidirectional)
 		(at 69.85 87.63 180)
@@
 		)
 	)
-	(hierarchical_label "1"
+	(hierarchical_label "GPIO1"
 		(shape bidirectional)
 		(at 69.85 72.39 180)
@@
 		)
 	)
-	(hierarchical_label "0"
+	(hierarchical_label "GPIO0"
 		(shape bidirectional)
 		(at 69.85 69.85 180)

Commit message: More fixes, add display, update display backlight driver circuit, fix some of the footprint associations
Parts:
- added R26: 51k, Resistor_SMD:R_0402_1005Metric, symbol symbols:R
Connections:
- net GND: now also R26.2
- net GPIO10 renamed LED_DATA
- net LED_DATA: now also R26.1
- net GPIO15 renamed CAMERA
Changed lines of the file:
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@@
+	)
+	(junction
+		(at 158.75 90.17)
+		(diameter 0)
+		(color 0 0 0 0)
 	)
 	(junction
@@
 	(wire
 		(pts
+			(xy 158.75 90.17) (xy 229.87 90.17)
+		)
+		(stroke
+			(width 0)
+			(type default)
+		)
+	)
+	(wire
+		(pts
 			(xy 146.05 67.31) (xy 229.87 67.31)
 		)
@@
 	(wire
 		(pts
+			(xy 158.75 119.38) (xy 158.75 132.08)
+		)
+		(stroke
+			(width 0)
+			(type default)
+		)
+	)
+	(wire
+		(pts
 			(xy 85.09 64.77) (xy 90.17 64.77)
 		)
@@
 	(wire
 		(pts
+			(xy 158.75 90.17) (xy 158.75 111.76)
+		)
+		(stroke
+			(width 0)
+			(type default)
+		)
+	)
+	(wire
+		(pts
 			(xy 173.99 95.25) (xy 229.87 95.25)
 		)
@@
 	(wire
 		(pts
-			(xy 146.05 90.17) (xy 229.87 90.17)
+			(xy 146.05 90.17) (xy 158.75 90.17)
 		)
 		(stroke
@@
 		)
 	)
-	(hierarchical_label "GPIO15"
-		(shape bidirectional)
+	(hierarchical_label "CAMERA"
+		(shape output)
 		(at 229.87 92.71 0)
 		(fields_autoplaced yes)
@@
 		)
 	)
-	(hierarchical_label "GPIO10"
-		(shape bidirectional)
+	(hierarchical_label "LED_DATA"
+		(shape output)
 		(at 229.87 90.17 0)
 		(fields_autoplaced yes)
@@
 				(path "/6a31734e-65de-48f3-8156-2b24b665b183/44fda57d-f8c9-4d6b-8127-d170c04d09fe"
 					(reference "#PWR047")
+					(unit 1)
+				)
+			)
+		)
+	)
+	(symbol
+		(lib_id "symbols2:GND")
+		(at 158.75 132.08 0)
+		(unit 1)
+		(exclude_from_sim no)
+		(in_bom yes)
+		(on_board yes)
+		(dnp no)
+		(property "Reference" "#PWR027"
+			(at 158.75 138.43 0)
+			(effects
+				(font
+					(size 1.27 1.27)
+				)
+				(hide yes)
+			)
+		)
+		(property "Value" "GND"
+			(at 158.877 136.4742 0)
+			(effects
+				(font
+					(size 1.27 1.27)
+				)
+			)
+		)
+		(property "Footprint" ""
+			(at 158.75 132.08 0)
+			(effects
+				(font
+					(size 1.27 1.27)
+				)
+				(hide yes)
+			)
+		)
+		(property "Datasheet" ""
+			(at 158.75 132.08 0)
+			(effects
+				(font
+					(size 1.27 1.27)
+				)
+				(hide yes)
+			)
+		)
+		(property "Description" "Power symbol creates a global label with name \"GND\" , ground"
+			(at 158.75 132.08 0)
+			(effects
+				(font
+					(size 1.27 1.27)
+				)
+				(hide yes)
+			)
+		)
+		(pin "1"
+		)
+		(instances
+			(project "why2025"
+				(path "/6a31734e-65de-48f3-8156-2b24b665b183/44fda57d-f8c9-4d6b-8127-d170c04d09fe"
+					(reference "#PWR027")
 					(unit 1)
 				)
@@
 					(unit 1)
 				)
+			)
+		)
+	)
+	(symbol
+		(lib_id "symbols:R")
+		(at 158.75 115.57 0)
+		(mirror y)
+		(unit 1)
+		(exclude_from_sim no)
+		(in_bom yes)
+		(on_board yes)
+		(dnp no)
+		(property "Reference" "R26"
+			(at 162.56 116.84 0)
+			(effects
+				(font
+					(size 1.27 1.27)
+				)
+			)
+		)
+		(property "Value" "51k"
+			(at 162.56 114.3 0)
+			(effects
+				(font
+					(size 1.27 1.27)
+				)
+			)
+		)
+		(property "Footprint" "Resistor_SMD:R_0402_1005Metric"
+			(at 160.528 115.57 90)
+			(effects
+				(font
+					(size 1.27 1.27)
+				)
+				(hide yes)
+			)
+		)
+		(property "Datasheet" ""
+			(at 158.75 115.57 0)
+			(effects
+				(font
+					(size 1.27 1.27)
+				)
+				(hide yes)
+			)
+		)
+		(property "Description" ""
+			(at 158.75 115.57 0)
+			(effects
+				(font
+					(size 1.27 1.27)
+				)
+				(hide yes)
+			)
+		)
+		(property "LCSC" ""
+			(at 158.75 115.57 0)
+			(effects
+				(font
+					(size 1.27 1.27)
+				)
+				(hide yes)
+			)
+		)
+		(pin "1"
+		)
+		(pin "2"
+		)
+		(instances
+			(project "why2025"
+				(path "/6a31734e-65de-48f3-8156-2b24b665b183/44fda57d-f8c9-4d6b-8127-d170c04d09fe"
+					(reference "R26")
+					(unit 1)
+				)

Commit message: More work on the schematic, add protection circuit, fix display pinout
Parts:
- added D79: LED, SparkFun-LED:LED_0603_1608Metric, symbol SparkFun-LED:LED
- added R32: 330, Resistor_SMD:R_0402_1005Metric, symbol Device:R
Connections:
- net +3.3V: now also D79.2 (A)
- net GPIO4: no longer names the net of U5.4 (MTMS/GPIO4/ADC1_CH4)
- net GPIO4: now also R32.1
- net GPIO5 renamed VLED_EN
- new net: D79.1 (K), R32.2
Other:
- company: (none) -> Badge.Team
- title: (none) -> WHY2025 badge

Commit message: Assign footprints, create P4 footprint
Parts:
- D79: footprint SparkFun-LED:LED_0603_1608Metric -> LED_SMD:LED_0603_1608Metric

Commit message: Bill of materials part 1
Parts:
- D79: value LED -> Blue LED; LCSC (none) -> C965809
- R13, R38: LCSC C25744 -> C60490
- R16: LCSC (none) -> C25741
- U5: LCSC - -> C5366877
