File: radio.kicad_sch (KiCad schematic)
At the start: 16 parts, among them U5 ESP32-C6-WROOM-1

Commit message: Small tweaks and fixes, update LCSC numbers on some components, change to new key type for power key
Parts:
- R17, R18: LCSC C25156 -> C25100
Connections:
- net GPIO0 is gone; now on an unnamed net: U5.8 (GPIO0/ADC1_CH0/XTAL_32K_P)
- net GPIO1 is gone; now on net VLED_EN: U5.9 (GPIO1/ADC1_CH1/XTAL_32K_N)
- net VLED_EN: no longer U5.5 (MTDI/GPIO5/ADC1_CH5)
- net at R32.1: no longer U5.4 (MTMS/GPIO4/ADC1_CH4)
- net GPIO2 renamed UNUSED0
- net GPIO3 renamed UNUSED1
- new net UNUSED2: U5.4 (MTMS/GPIO4/ADC1_CH4)
- new net UNUSED3: U5.5 (MTDI/GPIO5/ADC1_CH5)
Other:
- moved on the sheet: R32
Changed lines of the file:
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@@
-	(wire
-		(pts
-			(xy 25.4 68.58) (xy 25.4 66.04)
-		)
-		(stroke
-			(width 0)
-			(type default)
-		)
-	)
 	(wire
 		(pts
@@
 	(wire
 		(pts
+			(xy 69.85 85.09) (xy 90.17 85.09)
+		)
+		(stroke
+			(width 0)
+			(type default)
+		)
+	)
+	(wire
+		(pts
 			(xy 204.47 105.41) (xy 229.87 105.41)
 		)
@@
 	(wire
 		(pts
+			(xy 31.75 69.85) (xy 25.4 69.85)
+		)
+		(stroke
+			(width 0)
+			(type default)
+		)
+	)
+	(wire
+		(pts
 			(xy 69.85 64.77) (xy 85.09 64.77)
 		)
@@
 	(wire
 		(pts
+			(xy 25.4 69.85) (xy 25.4 66.04)
+		)
+		(stroke
+			(width 0)
+			(type default)
+		)
+	)
+	(wire
+		(pts
 			(xy 85.09 64.77) (xy 90.17 64.77)
 		)
@@
 	(wire
 		(pts
-			(xy 25.4 76.2) (xy 25.4 85.09)
-		)
-		(stroke
-			(width 0)
-			(type default)
-		)
-	)
-	(wire
-		(pts
 			(xy 72.39 129.54) (xy 72.39 132.08)
 		)
@@
 	(wire
 		(pts
-			(xy 69.85 69.85) (xy 90.17 69.85)
-		)
-		(stroke
-			(width 0)
-			(type default)
-		)
-	)
-	(wire
-		(pts
 			(xy 146.05 72.39) (xy 222.25 72.39)
 		)
@@
 	(wire
 		(pts
+			(xy 39.37 69.85) (xy 90.17 69.85)
+		)
+		(stroke
+			(width 0)
+			(type default)
+		)
+	)
+	(wire
+		(pts
 			(xy 166.37 87.63) (xy 229.87 87.63)
 		)
@@
 		(pts
 			(xy 69.85 72.39) (xy 90.17 72.39)
-		)
-		(stroke
-			(width 0)
-			(type default)
-		)
-	)
-	(wire
-		(pts
-			(xy 25.4 85.09) (xy 90.17 85.09)
 		)
 		(stroke
@@
 		)
 	)
-	(hierarchical_label "GPIO3"
+	(hierarchical_label "UNUSED3"
 		(shape bidirectional)
-		(at 69.85 77.47 180)
+		(at 69.85 87.63 180)
 		(fields_autoplaced yes)
 		(effects
@@
 		)
 	)
-	(hierarchical_label "GPIO2"
+	(hierarchical_label "UNUSED2"
 		(shape bidirectional)
-		(at 69.85 74.93 180)
+		(at 69.85 85.09 180)
 		(fields_autoplaced yes)
 		(effects
@@
 	(hierarchical_label "VLED_EN"
 		(shape output)
-		(at 69.85 87.63 180)
+		(at 69.85 72.39 180)
 		(fields_autoplaced yes)
 		(effects
@@
 		)
 	)
-	(hierarchical_label "GPIO1"
+	(hierarchical_label "UNUSED1"
 		(shape bidirectional)
-		(at 69.85 72.39 180)
+		(at 69.85 77.47 180)
 		(fields_autoplaced yes)
 		(effects
@@
 		)
 	)
-	(hierarchical_label "GPIO0"
+	(hierarchical_label "UNUSED0"
 		(shape bidirectional)
-		(at 69.85 69.85 180)
+		(at 69.85 74.93 180)
 		(fields_autoplaced yes)
 		(effects
@@
 			)
 		)
-		(property "LCSC" "C25156"
+		(property "LCSC" "C25100"
 			(at 226.06 74.93 0)
 			(effects
@@
 			)
 		)
-		(property "LCSC" "C25156"
+		(property "LCSC" "C25100"
 			(at 226.06 72.39 0)
 			(effects
@@
 	(symbol
 		(lib_id "Device:R")
-		(at 25.4 72.39 180)
+		(at 35.56 69.85 270)
 		(unit 1)
 		(exclude_from_sim no)
@@
 		(dnp no)
 		(property "Reference" "R32"
-			(at 27.94 72.39 90)
+			(at 35.56 67.31 90)
 			(effects
 				(font
@@
 		)
 		(property "Value" "330"
-			(at 23.114 72.39 90)
+			(at 35.56 72.136 90)
 			(effects
 				(font
@@
 		)
 		(property "Footprint" "Resistor_SMD:R_0402_1005Metric"
-			(at 27.178 72.39 90)
+			(at 35.56 68.072 90)
 			(effects
 				(font
@@
 		)
 		(property "Datasheet" ""
-			(at 25.4 72.39 0)
+			(at 35.56 69.85 0)
 			(effects
 				(font
@@
 		)
 		(property "Description" ""
-			(at 25.4 72.39 0)
-			(effects
-				(font
+			(at 35.56 69.85 0)
+			(effects
+				(font

Commit message: More routing and fixes
Connections:
- net CAMERA: now also U5.4 (MTMS/GPIO4/ADC1_CH4); no longer U5.23 (GPIO15)
- net UNUSED2: now also U5.23 (GPIO15); no longer U5.4 (MTMS/GPIO4/ADC1_CH4)
- net D+ renamed C6_USB1_P
- net D- renamed C6_USB1_N
Changed lines of the file:
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@@
 	(hierarchical_label "CAMERA"
 		(shape output)
-		(at 229.87 92.71 0)
+		(at 69.85 85.09 180)
 		(fields_autoplaced yes)
 		(effects
@@
 				(size 1.27 1.27)
 			)
-			(justify left)
+			(justify right)
 		)
 	)
@@
 		)
 	)
-	(hierarchical_label "D+"
+	(hierarchical_label "C6_USB1_P"
 		(shape bidirectional)
 		(at 229.87 72.39 0)
@@
 		)
 	)
-	(hierarchical_label "D-"
+	(hierarchical_label "C6_USB1_N"
 		(shape bidirectional)
 		(at 229.87 74.93 0)
@@
 	(hierarchical_label "UNUSED2"
 		(shape bidirectional)
-		(at 69.85 85.09 180)
+		(at 229.87 92.71 0)
 		(fields_autoplaced yes)
 		(effects
@@
 				(size 1.27 1.27)
 			)
-			(justify right)
+			(justify left)
 		)
 	)

Commit message: More routing, move PM I2C to ESP32-C6 instead of CH32
Parts:
- removed R13: 10k, Resistor_SMD:R_0402_1005Metric, symbol symbols:R
- added R102, R49: 4k7, Resistor_SMD:R_0402_1005Metric, symbol symbols:R
- added R12: 100k, Resistor_SMD:R_0402_1005Metric, symbol symbols:R
- added R46: 10k, Resistor_SMD:R_0402_1005Metric, symbol symbols:R
- R16: value 100k -> 10k; LCSC C25741 -> C60490
Connections:
- net +3.3V: now also R102.1, R46.2, R49.1
- net EN: now also R12.1
- net GND: now also R12.2
- net UNUSED0 renamed PM_SCL
- net PM_SCL: now also R49.2
- net UNUSED1 renamed PM_SDA
- net PM_SDA: now also R102.2
- net UNUSED2 renamed PM_INT
- net PM_INT: now also R46.1
Other:
- moved on the sheet: C10, R17, R18, R30, R33, R34, R35, R36, R37

Commit message: More routing, moved some more signals
Parts:
- removed D79: Blue LED, LED_SMD:LED_0603_1608Metric, symbol SparkFun-LED:LED
- removed R32: 330, Resistor_SMD:R_0402_1005Metric, symbol Device:R
Connections:
- net E13: now reaches U5.8 (GPIO0/ADC1_CH0/XTAL_32K_P)
- net UNUSED3 renamed E15
- net VLED_EN renamed E14
Changed lines of the file:
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@@
-	(wire
-		(pts
-			(xy 31.75 69.85) (xy 25.4 69.85)
-		)
-		(stroke
-			(width 0)
-			(type default)
-		)
-	)
 	(wire
 		(pts
@@
 	(wire
 		(pts
-			(xy 25.4 69.85) (xy 25.4 66.04)
-		)
-		(stroke
-			(width 0)
-			(type default)
-		)
-	)
-	(wire
-		(pts
 			(xy 173.99 92.71) (xy 173.99 62.23)
 		)
@@
 	(wire
 		(pts
-			(xy 25.4 55.88) (xy 25.4 58.42)
-		)
-		(stroke
-			(width 0)
-			(type default)
-		)
-	)
-	(wire
-		(pts
 			(xy 166.37 87.63) (xy 237.49 87.63)
 		)
@@
 	(wire
 		(pts
+			(xy 62.23 69.85) (xy 90.17 69.85)
+		)
+		(stroke
+			(width 0)
+			(type default)
+		)
+	)
+	(wire
+		(pts
 			(xy 62.23 77.47) (xy 85.09 77.47)
 		)
@@
 		(pts
 			(xy 85.09 63.5) (xy 85.09 77.47)
-		)
-		(stroke
-			(width 0)
-			(type default)
-		)
-	)
-	(wire
-		(pts
-			(xy 39.37 69.85) (xy 90.17 69.85)
 		)
 		(stroke
@@
 		)
 	)
+	(hierarchical_label "E14"
+		(shape bidirectional)
+		(at 62.23 72.39 180)
+		(fields_autoplaced yes)
+		(effects
+			(font
+				(size 1.27 1.27)
+			)
+			(justify right)
+		)
+	)
 	(hierarchical_label "SDIO_DATA0"
 		(shape bidirectional)
@@
 		)
 	)
+	(hierarchical_label "E13"
+		(shape bidirectional)
+		(at 62.23 69.85 180)
+		(fields_autoplaced yes)
+		(effects
+			(font
+				(size 1.27 1.27)
+			)
+			(justify right)
+		)
+	)
 	(hierarchical_label "EN"
 		(shape input)
@@
 		)
 	)
-	(hierarchical_label "UNUSED3"
+	(hierarchical_label "E15"
 		(shape bidirectional)
 		(at 62.23 87.63 180)
@@
 		)
 	)
-	(hierarchical_label "VLED_EN"
-		(shape output)
-		(at 62.23 72.39 180)
-		(fields_autoplaced yes)
-		(effects
-			(font
-				(size 1.27 1.27)
-			)
-			(justify right)
-		)
-	)
 	(hierarchical_label "PM_SCL"
 		(shape bidirectional)
@@
 	)
 	(symbol
-		(lib_id "SparkFun-LED:LED")
-		(at 25.4 62.23 90)
-		(unit 1)
-		(exclude_from_sim no)
-		(in_bom yes)
-		(on_board yes)
-		(dnp no)
-		(property "Reference" "D79"
-			(at 22.606 62.23 0)
-			(effects
-				(font
-					(size 1.27 1.27)
-				)
-			)
-		)
-		(property "Value" "Blue LED"
-			(at 29.972 62.23 0)
-			(effects
-				(font
-					(size 1.27 1.27)
-				)
-			)
-		)
-		(property "Footprint" "LED_SMD:LED_0603_1608Metric"
-			(at 30.48 62.23 0)
-			(effects
-				(font
-					(size 1.27 1.27)
-				)
-				(hide yes)
-			)
-		)
-		(property "Datasheet" "https://datasheet.lcsc.com/lcsc/2402181505_XINGLIGHT-XL-1608BGWC-06_C965809.pdf"
-			(at 25.4 62.23 0)
-			(effects
-				(font
-					(size 1.27 1.27)
-				)
-				(hide yes)
-			)
-		)
-		(property "Description" "Light emitting diode"
-			(at 25.4 62.23 0)
-			(effects
-				(font
-					(size 1.27 1.27)
-				)
-				(hide yes)
-			)
-		)
-		(property "LCSC" "C965809"
-			(at 25.4 62.23 0)
-			(effects
-				(font
-					(size 1.27 1.27)
-				)
-				(hide yes)
-			)
-		)
-		(pin "1"
-		)
-		(pin "2"
-		)
-		(instances
-			(project "why2025"
-				(path "/6a31734e-65de-48f3-8156-2b24b665b183/44fda57d-f8c9-4d6b-8127-d170c04d09fe"
-					(reference "D79")
-					(unit 1)
-				)
-			)
-		)
-	)
-	(symbol
-		(lib_id "Device:R")
-		(at 35.56 69.85 270)
-		(unit 1)
-		(exclude_from_sim no)
-		(in_bom yes)
-		(on_board yes)
-		(dnp no)
-		(property "Reference" "R32"
-			(at 35.56 67.31 90)
-			(effects
-				(font
-					(size 1.27 1.27)
-				)
-			)
-		)
-		(property "Value" "330"
-			(at 35.56 72.136 90)
-			(effects
-				(font
-					(size 1.27 1.27)
-				)
-			)
-		)
-		(property "Footprint" "Resistor_SMD:R_0402_1005Metric"
-			(at 35.56 68.072 90)
-			(effects
-				(font
-					(size 1.27 1.27)
-				)
-				(hide yes)
-			)
-		)
-		(property "Datasheet" ""
-			(at 35.56 69.85 0)
-			(effects
-				(font
-					(size 1.27 1.27)
-				)
-				(hide yes)
-			)
-		)
-		(property "Description" ""
-			(at 35.56 69.85 0)
-			(effects
-				(font
-					(size 1.27 1.27)
-				)
-				(hide yes)
-			)
-		)
-		(pin "1"
-		)
-		(pin "2"
-		)
-		(instances
-			(project "why2025"
-				(path "/6a31734e-65de-48f3-8156-2b24b665b183/44fda57d-f8c9-4d6b-8127-d170c04d09fe"
-					(reference "R32")
-					(unit 1)
-				)
-			)
-		)
-	)
-	(symbol
 		(lib_id "power:+3.3V")
 		(at 118.11 54.61 0)
@@
 					(unit 1)
 				)
-			)
-		)
-	)
-	(symbol
-		(lib_id "power:+3.3V")
-		(at 25.4 55.88 0)
-		(unit 1)
-		(exclude_from_sim no)
-		(in_bom yes)
-		(on_board yes)
-		(dnp no)
-		(property "Reference" "#PWR071"
-			(at 25.4 59.69 0)
-			(effects
-				(font
-					(size 1.27 1.27)
-				)
-				(hide yes)
-			)
-		)
-		(property "Value" "+3.3V"
-			(at 25.4 52.07 0)
-			(effects
-				(font
-					(size 1.27 1.27)
-				)
-			)
-		)
-		(property "Footprint" ""
-			(at 25.4 55.88 0)
-			(effects
-				(font
-					(size 1.27 1.27)
-				)
-				(hide yes)
-			)
-		)
-		(property "Datasheet" ""
-			(at 25.4 55.88 0)
-			(effects
-				(font
-					(size 1.27 1.27)
-				)
-				(hide yes)
-			)
-		)
-		(property "Description" "Power symbol creates a global label with name \"+3.3V\""
-			(at 25.4 55.88 0)
-			(effects
-				(font
-					(size 1.27 1.27)
-				)
-				(hide yes)
-			)
-		)
-		(pin "1"
-		)
-		(instances
-			(project "why2025"
-				(path "/6a31734e-65de-48f3-8156-2b24b665b183/44fda57d-f8c9-4d6b-8127-d170c04d09fe"
-					(reference "#PWR071")
-					(unit 1)
-				)

Commit message: All wires routed, lots of DRC errors to go
Parts:
- R12: LCSC (none) -> C25741
Connections:
- net E13: now also U5.9 (GPIO1/ADC1_CH1/XTAL_32K_N); no longer U5.8 (GPIO0/ADC1_CH0/XTAL_32K_P)
- net E14: now also U5.8 (GPIO0/ADC1_CH0/XTAL_32K_P); no longer U5.9 (GPIO1/ADC1_CH1/XTAL_32K_N)
Changed lines of the file:
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@@
 	(hierarchical_label "E14"
 		(shape bidirectional)
-		(at 62.23 72.39 180)
+		(at 62.23 69.85 180)
 		(fields_autoplaced yes)
 		(effects
@@
 	(hierarchical_label "E13"
 		(shape bidirectional)
-		(at 62.23 69.85 180)
+		(at 62.23 72.39 180)
 		(fields_autoplaced yes)
 		(effects
@@
 			)
 		)
-		(property "Datasheet" ""
+		(property "Datasheet" "https://datasheet.lcsc.com/lcsc/2110260030_UNI-ROYAL-Uniroyal-Elec-0402WGF1003TCE_C25741.pdf"
 			(at 69.85 125.73 0)
 			(effects
@@
 			)
 		)
-		(property "LCSC" ""
+		(property "LCSC" "C25741"
 			(at 69.85 125.73 0)
 			(effects

Commit message: More fabrication stuff for prototype 1
Parts:
- R26, R30, R33, R34, R35, R36, R37: LCSC (none) -> C25794
Changed lines of the file:
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@@
 			)
 		)
-		(property "Datasheet" ""
+		(property "Datasheet" "https://www.lcsc.com/product-detail/Chip-Resistor-Surface-Mount_UNI-ROYAL-Uniroyal-Elec-0402WGF5102TCE_C25794.html"
 			(at 204.47 58.42 0)
 			(effects
@@
 			)
 		)
-		(property "LCSC" ""
+		(property "LCSC" "C25794"
 			(at 204.47 58.42 0)
 			(effects
@@
 			)
 		)
-		(property "Datasheet" ""
+		(property "Datasheet" "https://www.lcsc.com/product-detail/Chip-Resistor-Surface-Mount_UNI-ROYAL-Uniroyal-Elec-0402WGF5102TCE_C25794.html"
 			(at 212.09 58.42 0)
 			(effects
@@
 			)
 		)
-		(property "LCSC" ""
+		(property "LCSC" "C25794"
 			(at 212.09 58.42 0)
 			(effects
@@
 			)
 		)
-		(property "Datasheet" ""
+		(property "Datasheet" "https://www.lcsc.com/product-detail/Chip-Resistor-Surface-Mount_UNI-ROYAL-Uniroyal-Elec-0402WGF5102TCE_C25794.html"
 			(at 219.71 58.42 0)
 			(effects
@@
 			)
 		)
-		(property "LCSC" ""
+		(property "LCSC" "C25794"
 			(at 219.71 58.42 0)
 			(effects
@@
 			)
 		)
-		(property "Datasheet" ""
+		(property "Datasheet" "https://www.lcsc.com/product-detail/Chip-Resistor-Surface-Mount_UNI-ROYAL-Uniroyal-Elec-0402WGF5102TCE_C25794.html"
 			(at 158.75 115.57 0)
 			(effects
@@
 			)
 		)
-		(property "LCSC" ""
+		(property "LCSC" "C25794"
 			(at 158.75 115.57 0)
 			(effects
@@
 			)
 		)
-		(property "Datasheet" ""
+		(property "Datasheet" "https://www.lcsc.com/product-detail/Chip-Resistor-Surface-Mount_UNI-ROYAL-Uniroyal-Elec-0402WGF5102TCE_C25794.html"
 			(at 181.61 58.42 0)
 			(effects
@@
 			)
 		)
-		(property "LCSC" ""
+		(property "LCSC" "C25794"
 			(at 181.61 58.42 0)
 			(effects
@@
 			)
 		)
-		(property "Datasheet" ""
+		(property "Datasheet" "https://www.lcsc.com/product-detail/Chip-Resistor-Surface-Mount_UNI-ROYAL-Uniroyal-Elec-0402WGF5102TCE_C25794.html"
 			(at 196.85 58.42 0)
 			(effects
@@
 			)
 		)
-		(property "LCSC" ""
+		(property "LCSC" "C25794"
 			(at 196.85 58.42 0)
 			(effects
@@
 			)
 		)
-		(property "Datasheet" ""
+		(property "Datasheet" "https://www.lcsc.com/product-detail/Chip-Resistor-Surface-Mount_UNI-ROYAL-Uniroyal-Elec-0402WGF5102TCE_C25794.html"
 			(at 189.23 58.42 0)
 			(effects
@@
 			)
 		)
-		(property "LCSC" ""
+		(property "LCSC" "C25794"
 			(at 189.23 58.42 0)
 			(effects

Commit message: Rerouting to get LORA chip fitted.
Parts:
- added J3: Conn_Coaxial_Small, symbol Connector:Conn_Coaxial_Small
- added L5: RA-01SH, RF_Module:Ai-Thinker-Ra-01-LoRa, symbol RA-01SH:RA-01SH
Connections:
- net +3.3V: now also L5.3 (3.3V)
- net GND: now also J3.2 (Ext), L5.16 (GND), L5.2 (GND), L5.9 (GND)
- new net: J3.1 (In), L5.1 (ANT)
