File: radio.kicad_sch (KiCad schematic)
At the start: 20 parts, among them J3 LoRa, U5 ESP32-C6-WROOM-1

Commit message: Small fixes
Parts:
- renumbered L5 to U27
Changed lines of the file:
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@@
 		(dnp yes)
 		(fields_autoplaced yes)
-		(property "Reference" "L5"
+		(property "Reference" "U27"
 			(at 89.8241 127 0)
 			(effects
@@
 			(project ""
 				(path "/6a31734e-65de-48f3-8156-2b24b665b183/44fda57d-f8c9-4d6b-8127-d170c04d09fe"
-					(reference "L5")
+					(reference "U27")
 					(unit 1)
 				)

Commit message: More SAO
Connections:
- net TX: now reaches TP16.1, U5.25 (U0TXD/GPIO16)
- net RX: now reaches TP17.1, U5.24 (U0RXD/GPIO17)
Changed lines of the file:
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@@
+		)
+	)
+	(hierarchical_label "RX"
+		(shape input)
+		(at 207.01 36.83 0)
+		(fields_autoplaced yes)
+		(effects
+			(font
+				(size 1.27 1.27)
+			)
+			(justify left)
 		)
 	)
@@
 		(fields_autoplaced yes)
 		(effects
+			(font
+				(size 1.27 1.27)
+			)
+			(justify left)
+		)
+	)
+	(hierarchical_label "TX"
+		(shape output)
+		(at 207.01 34.29 0)
+		(fields_autoplaced yes)
+		(effects

Commit message: Small fixes
Parts:
- C42: LCSC C394158 -> C307331
- J3: LCSC (none) -> -
Changed lines of the file:
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@@
 	(title_block
 		(title "WHY2025 badge")
-		(date "2024-08-23")
+		(date "2024-08-24")
 		(rev "Prototype 2")
 		(company "Badge.Team")
@@
 			)
 		)
-		(property "Datasheet" ""
+		(property "Datasheet" "https://datasheet.lcsc.com/lcsc/2304140030_Samsung-Electro-Mechanics-CL05B104KB54PNC_C307331.pdf"
 			(at 81.28 128.27 0)
 			(effects
@@
 			)
 		)
-		(property "Description" "Unpolarized capacitor"
+		(property "Description" ""
 			(at 81.28 128.27 0)
 			(effects
@@
 			)
 		)
-		(property "LCSC" "C394158"
+		(property "LCSC" "C307331"
 			(at 81.28 128.27 0)
 			(effects
@@
 			(at 113.03 134.62 0)
 			(effects
+				(font
+					(size 1.27 1.27)
+				)
+				(hide yes)
+			)
+		)
+		(property "LCSC" "-"
+			(at 113.03 134.62 0)
+			(effects

Commit message: Add 1.5k pull-up to D+ of C6, remove logos, add JTAG connector, fix SAO pinout
Parts:
- added R83: 1.5k, Resistor_SMD:R_0402_1005Metric, symbol symbols:R
Connections:
- net EN: now also R83.2
- net C6_USB1_INT_N: now reaches R18.2, U5.13 (GPIO12/USB_D-)
- net C6_USB1_INT_P: now reaches R17.2, U5.14 (GPIO13/USB_D+)
- net C6_USB1_INT_P: now also R83.1
Other:
- note added: "Workaround for USB enumeration problem"
Changed lines of the file:
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@@
+	)
+	(junction
+		(at 50.8 34.29)
+		(diameter 0)
+		(color 0 0 0 0)
 	)
 	(junction
@@
 	(wire
 		(pts
+			(xy 50.8 34.29) (xy 59.69 34.29)
+		)
+		(stroke
+			(width 0)
+			(type default)
+		)
+	)
+	(wire
+		(pts
 			(xy 31.75 34.29) (xy 31.75 91.44)
 		)
@@
 	(wire
 		(pts
+			(xy 53.34 25.4) (xy 50.8 25.4)
+		)
+		(stroke
+			(width 0)
+			(type default)
+		)
+	)
+	(wire
+		(pts
 			(xy 135.89 31.75) (xy 135.89 57.15)
 		)
@@
 	(wire
 		(pts
+			(xy 50.8 25.4) (xy 50.8 26.67)
+		)
+		(stroke
+			(width 0)
+			(type default)
+		)
+	)
+	(wire
+		(pts
 			(xy 128.27 88.9) (xy 128.27 101.6)
 		)
@@
 	(wire
 		(pts
-			(xy 31.75 34.29) (xy 59.69 34.29)
+			(xy 31.75 34.29) (xy 50.8 34.29)
 		)
 		(stroke
@@
 		)
 	)
+	(text "Workaround for USB\nenumeration problem"
+		(exclude_from_sim no)
+		(at 58.166 22.098 0)
+		(effects
+			(font
+				(size 1.27 1.27)
+			)
+		)
+	)
+	(label "C6_USB1_INT_P"
+		(at 116.84 41.91 0)
+		(fields_autoplaced yes)
+		(effects
+			(font
+				(size 1.27 1.27)
+			)
+			(justify left bottom)
+		)
+	)
+	(label "C6_USB1_INT_N"
+		(at 116.84 44.45 0)
+		(fields_autoplaced yes)
+		(effects
+			(font
+				(size 1.27 1.27)
+			)
+			(justify left bottom)
+		)
+	)
 	(global_label "LORA_SCK"
 		(shape input)
@@
 				)
 				(justify right)
+				(hide yes)
+			)
+		)
+	)
+	(global_label "C6_USB1_INT_P"
+		(shape output)
+		(at 53.34 25.4 0)
+		(fields_autoplaced yes)
+		(effects
+			(font
+				(size 1.016 1.016)
+			)
+			(justify left)
+		)
+		(property "Intersheetrefs" "${INTERSHEET_REFS}"
+			(at 67.3877 25.4 0)
+			(effects
+				(font
+					(size 1.27 1.27)
+				)
+				(justify left)
 				(hide yes)
 			)
@@
 					(unit 1)
 				)
+			)
+		)
+	)
+	(symbol
+		(lib_id "symbols:R")
+		(at 50.8 30.48 0)
+		(mirror y)
+		(unit 1)
+		(exclude_from_sim no)
+		(in_bom yes)
+		(on_board yes)
+		(dnp no)
+		(property "Reference" "R83"
+			(at 54.61 31.75 0)
+			(effects
+				(font
+					(size 1.27 1.27)
+				)
+			)
+		)
+		(property "Value" "1.5k"
+			(at 54.61 29.21 0)
+			(effects
+				(font
+					(size 1.27 1.27)
+				)
+			)
+		)
+		(property "Footprint" "Resistor_SMD:R_0402_1005Metric"
+			(at 52.578 30.48 90)
+			(effects
+				(font
+					(size 1.27 1.27)
+				)
+				(hide yes)
+			)
+		)
+		(property "Datasheet" ""
+			(at 50.8 30.48 0)
+			(effects
+				(font
+					(size 1.27 1.27)
+				)
+				(hide yes)
+			)
+		)
+		(property "Description" ""
+			(at 50.8 30.48 0)
+			(effects
+				(font
+					(size 1.27 1.27)
+				)
+				(hide yes)
+			)
+		)
+		(property "LCSC" ""
+			(at 50.8 30.48 0)
+			(effects
+				(font
+					(size 1.27 1.27)
+				)
+				(hide yes)
+			)
+		)
+		(pin "1"
+		)
+		(pin "2"
+		)
+		(instances
+			(project "why2025"
+				(path "/6a31734e-65de-48f3-8156-2b24b665b183/44fda57d-f8c9-4d6b-8127-d170c04d09fe"
+					(reference "R83")
+					(unit 1)
+				)

Commit message: 85: Changed SMA footprint for LORA to use: Samtec_SMA-J-P-H-ST-EM1_EdgeMount
Parts:
- J3: footprint Connector_Coaxial:SMA_Amphenol_132289_EdgeMount -> Connector_Coaxial:SMA_Samtec_SMA-J-P-H-ST-EM1_EdgeMount
Changed lines of the file:
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@@
 			)
 		)
-		(property "Footprint" "Connector_Coaxial:SMA_Amphenol_132289_EdgeMount"
+		(property "Footprint" "Connector_Coaxial:SMA_Samtec_SMA-J-P-H-ST-EM1_EdgeMount"
 			(at 113.03 134.62 0)
 			(effects
