File: esp32p4.kicad_sch (KiCad schematic)
At the start: 52 parts, among them U13 W25Q128JVS, U3 TLV62569DBV, U8 ESP32P4-REV0, Y3 40MHz

Commit message: Small tweaks and fixes, update LCSC numbers on some components, change to new key type for power key
Parts:
- added R42, R45: 4k7, Resistor_SMD:R_0402_1005Metric, symbol Device:R
- R40, R41: LCSC (none) -> C137971
- R44, R52: LCSC (none) -> C43251
Connections:
- net +3.3V: now also U8.102 (VDDA), U8.103 (VBAT), R42.2, R45.2
- net GND: now also U8.105 (GND)
- net GPIO35: now also R45.1
- net GPIO36: now also R42.1
- net Protection/~{RESET} renamed ~{RESET}
Other:
- note added: "Boot: high = normal, low = download"
- note added: "Download boot: high = joint, low = SPI"
- note added: "Must be high for SPI download mode"
- note added: "Must be low for SPI download mode"
- moved on the sheet: C56, R54, R55, R56, R57, R58, R59, U8L

Commit message: Some more component placement
Changed lines of the file:
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@@
-	(wire
-		(pts
-			(xy 36.83 15.24) (xy 36.83 16.51)
-		)
-		(stroke
-			(width 0)
-			(type default)
-		)
-	)
 	(wire
 		(pts
@@
 		)
 		(stroke
-			(width 0)
-			(type default)
-		)
-	)
-	(wire
-		(pts
-			(xy 40.64 16.51) (xy 40.64 15.24)
-		)
-		(stroke

Commit message: More routing, small fixes in schematic
Parts:
- added C30: 1u, Capacitor_SMD:C_0603_1608Metric, symbol mch2021-rescue:C-Device
Connections:
- net GND: now also C30.2
- net VSDCARD: now also C30.1
Changed lines of the file:
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@@
 	)
 	(junction
+		(at 168.91 156.21)
+		(diameter 0)
+		(color 0 0 0 0)
+	)
+	(junction
 		(at 27.94 190.5)
 		(diameter 0)
@@
 	(wire
 		(pts
-			(xy 168.91 129.54) (xy 168.91 157.48)
+			(xy 168.91 129.54) (xy 168.91 156.21)
 		)
 		(stroke
@@
 	(wire
 		(pts
+			(xy 168.91 156.21) (xy 168.91 157.48)
+		)
+		(stroke
+			(width 0)
+			(type default)
+		)
+	)
+	(wire
+		(pts
 			(xy 26.67 190.5) (xy 27.94 190.5)
 		)
@@
 	(wire
 		(pts
+			(xy 162.56 157.48) (xy 162.56 156.21)
+		)
+		(stroke
+			(width 0)
+			(type default)
+		)
+	)
+	(wire
+		(pts
 			(xy 149.86 120.65) (xy 143.51 120.65)
 		)
@@
 	(wire
 		(pts
+			(xy 162.56 156.21) (xy 168.91 156.21)
+		)
+		(stroke
+			(width 0)
+			(type default)
+		)
+	)
+	(wire
+		(pts
 			(xy 137.16 120.65) (xy 130.81 120.65)
 		)
@@
 	)
 	(symbol
+		(lib_id "mch2021-rescue:GND-power")
+		(at 162.56 165.1 0)
+		(unit 1)
+		(exclude_from_sim no)
+		(in_bom yes)
+		(on_board yes)
+		(dnp no)
+		(property "Reference" "#PWR0205"
+			(at 162.56 171.45 0)
+			(effects
+				(font
+					(size 1.27 1.27)
+				)
+				(hide yes)
+			)
+		)
+		(property "Value" "GND"
+			(at 162.56 170.18 0)
+			(effects
+				(font
+					(size 1.27 1.27)
+				)
+			)
+		)
+		(property "Footprint" ""
+			(at 162.56 165.1 0)
+			(effects
+				(font
+					(size 1.27 1.27)
+				)
+				(hide yes)
+			)
+		)
+		(property "Datasheet" ""
+			(at 162.56 165.1 0)
+			(effects
+				(font
+					(size 1.27 1.27)
+				)
+				(hide yes)
+			)
+		)
+		(property "Description" ""
+			(at 162.56 165.1 0)
+			(effects
+				(font
+					(size 1.27 1.27)
+				)
+				(hide yes)
+			)
+		)
+		(pin "1"
+		)
+		(instances
+			(project "why2025"
+				(path "/6a31734e-65de-48f3-8156-2b24b665b183/3d60835a-4261-467a-b239-9fb76f6e13a1"
+					(reference "#PWR0205")
+					(unit 1)
+				)
+			)
+		)
+	)
+	(symbol
 		(lib_id "Device:R")
 		(at 238.76 118.11 0)
@@
 					(unit 1)
 				)
+			)
+		)
+	)
+	(symbol
+		(lib_id "mch2021-rescue:C-Device")
+		(at 162.56 161.29 0)
+		(unit 1)
+		(exclude_from_sim no)
+		(in_bom yes)
+		(on_board yes)
+		(dnp no)
+		(property "Reference" "C30"
+			(at 155.956 160.782 0)
+			(effects
+				(font
+					(size 1.27 1.27)
+				)
+				(justify left)
+			)
+		)
+		(property "Value" "1u"
+			(at 156.972 162.814 0)
+			(effects
+				(font
+					(size 1.27 1.27)
+				)
+				(justify left)
+			)
+		)
+		(property "Footprint" "Capacitor_SMD:C_0603_1608Metric"
+			(at 163.5252 165.1 0)
+			(effects
+				(font
+					(size 1.27 1.27)
+				)
+				(hide yes)
+			)
+		)
+		(property "Datasheet" "https://datasheet.lcsc.com/lcsc/2304140030_Samsung-Electro-Mechanics-CL05A105KQ5NNNC_C107372.pdf"
+			(at 162.56 161.29 0)
+			(effects
+				(font
+					(size 1.27 1.27)
+				)
+				(hide yes)
+			)
+		)
+		(property "Description" ""
+			(at 162.56 161.29 0)
+			(effects
+				(font
+					(size 1.27 1.27)
+				)
+				(hide yes)
+			)
+		)
+		(property "LCSC" "C107372"
+			(at 162.56 161.29 0)
+			(effects
+				(font
+					(size 1.27 1.27)
+				)
+				(hide yes)
+			)
+		)
+		(pin "1"
+		)
+		(pin "2"
+		)
+		(instances
+			(project "why2025"
+				(path "/6a31734e-65de-48f3-8156-2b24b665b183/3d60835a-4261-467a-b239-9fb76f6e13a1"
+					(reference "C30")
+					(unit 1)
+				)

Commit message: More routing and fixes
Connections:
- net C6_CLK: now also U8.19 (GPIO17); no longer U8.23 (GPIO20)
- net C6_CMD: now also U8.18 (GPIO16); no longer U8.24 (GPIO21)
- net C6_D0: now also U8.20 (GPIO18); no longer U8.18 (GPIO16)
- net C6_D1: now also U8.21 (GPIO19); no longer U8.19 (GPIO17)
- net C6_D2: now also U8.23 (GPIO20); no longer U8.20 (GPIO18)
- net C6_D3: now also U8.24 (GPIO21); no longer U8.21 (GPIO19)
- net at C48.1, U8.100 (XTAL_N): now also Y3.3; no longer Y3.1
- net at C47.1, U8.101 (XTAL_P): now also Y3.1; no longer Y3.3
- net USB_DM renamed USB2_N
- net USB_DP renamed USB2_P
Changed lines of the file:
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@@
 	(hierarchical_label "C6_D0"
 		(shape bidirectional)
-		(at 27.94 69.85 180)
+		(at 27.94 74.93 180)
 		(fields_autoplaced yes)
 		(effects
@@
 	(hierarchical_label "C6_D1"
 		(shape bidirectional)
-		(at 27.94 72.39 180)
+		(at 27.94 77.47 180)
 		(fields_autoplaced yes)
 		(effects
@@
 	(hierarchical_label "C6_CLK"
 		(shape output)
-		(at 26.67 109.22 180)
+		(at 27.94 72.39 180)
 		(fields_autoplaced yes)
 		(effects
@@
 	(hierarchical_label "C6_CMD"
 		(shape output)
-		(at 26.67 111.76 180)
+		(at 27.94 69.85 180)
 		(fields_autoplaced yes)
 		(effects
@@
 	(hierarchical_label "C6_D3"
 		(shape bidirectional)
-		(at 27.94 77.47 180)
+		(at 26.67 111.76 180)
 		(fields_autoplaced yes)
 		(effects
@@
 		)
 	)
-	(hierarchical_label "USB_DP"
+	(hierarchical_label "USB2_P"
 		(shape bidirectional)
 		(at 255.27 144.78 180)
@@
 	(hierarchical_label "C6_D2"
 		(shape bidirectional)
-		(at 27.94 74.93 180)
+		(at 26.67 109.22 180)
 		(fields_autoplaced yes)
 		(effects
@@
 		)
 	)
-	(hierarchical_label "USB_DM"
+	(hierarchical_label "USB2_N"
 		(shape bidirectional)
 		(at 255.27 142.24 180)
@@
 		(lib_id "Device:Crystal_GND24_Small")
 		(at 120.65 59.69 90)
+		(mirror x)
 		(unit 1)
 		(exclude_from_sim no)
@@
 		(dnp no)
 		(property "Reference" "Y3"
-			(at 114.3 58.166 90)
+			(at 114.3 61.214 90)
 			(effects
 				(font
@@
 		)
 		(property "Value" "40MHz"
-			(at 114.3 60.198 90)
-			(effects
-				(font
+			(at 114.3 59.182 90)
+			(effects
+				(font

Commit message: More routing, move PM I2C to ESP32-C6 instead of CH32
Parts:
- removed C46: 100n, Capacitor_SMD:C_0402_1005Metric, symbol symbols:C
- removed R53, R60, R61: 4k7, Resistor_SMD:R_0402_1005Metric, symbol Device:R
- R62: value 4k7 -> 10k; LCSC C25900 -> (none)

Commit message: More routing, moved some more signals
Parts:
- removed R62: 10k, Resistor_SMD:R_0402_1005Metric, symbol Device:R
- removed R63, R64: 4k7, Resistor_SMD:R_0402_1005Metric, symbol Device:R
- added R13, R15: 4k7, Resistor_SMD:R_0402_1005Metric, symbol Device:R
- added R25: 10k, Resistor_SMD:R_0402_1005Metric, symbol Device:R
Connections:
- net +3.3V: now also R13.2, R15.2, R25.2
- net EXT_INT: now also R25.1
- net GPIO52: no longer U8.96 (GPIO52)
- net GPIO53: no longer U8.98 (GPIO53)
- net GPIO54: no longer U8.99 (GPIO54)
- net SAO_IO1: now also U8.17 (GPIO15); no longer U8.16 (GPIO14)
- net SAO_IO2: now also U8.16 (GPIO14); no longer U8.17 (GPIO15)
- new net LCD_RESET: U8.99 (GPIO54)
- new net SYS_SCL: R13.1, U8.98 (GPIO53)
- new net SYS_SDA: R15.1, U8.96 (GPIO52)
- no-connect marks 6 -> 18
Other:
- note added: "These pins are moved to GPIO 49 to 53 temporarily on prototype 1!!!!"
- note removed: "Will be connected when production chip is available"

Commit message: All wires routed, lots of DRC errors to go
Parts:
- removed C42: 100n, Capacitor_SMD:C_0402_1005Metric, symbol symbols:C
- removed C49: 1u, Capacitor_SMD:C_0603_1608Metric, symbol symbols:C
- C25: footprint Capacitor_SMD:C_1206_3216Metric -> Capacitor_SMD:C_0805_2012Metric; LCSC C13585 -> C3039694
- C44: value 100n -> 1u; footprint Capacitor_SMD:C_0402_1005Metric -> Capacitor_SMD:C_0603_1608Metric; LCSC C307331 -> C107372
- R25: LCSC (none) -> C60490
Connections:
- net +3.3V: no longer C44.1
- net C6_INT: now also U8.95 (GPIO51); no longer U8.94 (GPIO50)
- net EXT_INT: now also U8.94 (GPIO50); no longer U8.95 (GPIO51)
- net LCD_RESET: now also U8.1 (GPIO0); no longer U8.99 (GPIO54)
- net LCD_TE: now also U8.99 (GPIO54); no longer U8.1 (GPIO0)
- net VFLASH: now also C44.1
- net GPIO34 renamed E2
- net GPIO35 renamed E1
- net GPIO36 renamed E0
- net GPIO45 renamed E3
- net GPIO46 renamed E6
- net GPIO47 renamed E5
- net GPIO48 renamed E4
Other:
- moved on the sheet: C38, C39, C40, C41, C45, C50, C51, U8C, U8G

Commit message: More fabrication stuff for prototype 1
Parts:
- C24: now left out of the parts list
- R54, R55, R56, R57, R58, R59: LCSC (none) -> C25794
Changed lines of the file:
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@@
 			)
 		)
-		(property "Datasheet" ""
+		(property "Datasheet" "https://www.lcsc.com/product-detail/Chip-Resistor-Surface-Mount_YAGEO-RC0402FR-07499KL_C137971.html"
 			(at 260.35 41.91 0)
 			(effects
@@
 			)
 		)
-		(property "Datasheet" ""
+		(property "Datasheet" "https://www.lcsc.com/product-detail/Chip-Resistor-Surface-Mount_UNI-ROYAL-Uniroyal-Elec-0402WGF5102TCE_C25794.html"
 			(at 124.46 125.73 0)
 			(effects
@@
 			)
 		)
+		(property "LCSC" "C25794"
+			(at 124.46 125.73 0)
+			(effects
+				(font
+					(size 1.27 1.27)
+				)
+				(hide yes)
+			)
+		)
 		(pin "1"
 		)
@@
 			)
 		)
-		(property "Datasheet" ""
+		(property "Datasheet" "https://www.lcsc.com/product-detail/Chip-Resistor-Surface-Mount_UNI-ROYAL-Uniroyal-Elec-0402WGF5102TCE_C25794.html"
 			(at 130.81 125.73 0)
 			(effects
@@
 			)
 		)
+		(property "LCSC" "C25794"
+			(at 130.81 125.73 0)
+			(effects
+				(font
+					(size 1.27 1.27)
+				)
+				(hide yes)
+			)
+		)
 		(pin "1"
 		)
@@
 			)
 		)
-		(property "Datasheet" ""
+		(property "Datasheet" "https://www.lcsc.com/product-detail/Chip-Resistor-Surface-Mount_UNI-ROYAL-Uniroyal-Elec-0402WGF5102TCE_C25794.html"
 			(at 143.51 125.73 0)
 			(effects
@@
 			)
 		)
+		(property "LCSC" "C25794"
+			(at 143.51 125.73 0)
+			(effects
+				(font
+					(size 1.27 1.27)
+				)
+				(hide yes)
+			)
+		)
 		(pin "1"
 		)
@@
 			)
 		)
-		(property "Datasheet" ""
+		(property "Datasheet" "https://www.lcsc.com/product-detail/Chip-Resistor-Surface-Mount_YAGEO-RC0402FR-07499KL_C137971.html"
 			(at 260.35 29.21 0)
 			(effects
@@
 			)
 		)
-		(property "Datasheet" ""
+		(property "Datasheet" "https://www.lcsc.com/product-detail/Chip-Resistor-Surface-Mount_UNI-ROYAL-Uniroyal-Elec-0402WGF5102TCE_C25794.html"
 			(at 156.21 125.73 0)
 			(effects
@@
 			)
 		)
+		(property "LCSC" "C25794"
+			(at 156.21 125.73 0)
+			(effects
+				(font
+					(size 1.27 1.27)
+				)
+				(hide yes)
+			)
+		)
 		(pin "1"
 		)
@@
 		(unit 1)
 		(exclude_from_sim no)
-		(in_bom yes)
+		(in_bom no)
 		(on_board yes)
 		(dnp yes)
@@
 			)
 		)
-		(property "Datasheet" ""
+		(property "Datasheet" "https://www.lcsc.com/product-detail/Chip-Resistor-Surface-Mount_UNI-ROYAL-Uniroyal-Elec-0402WGF5102TCE_C25794.html"
 			(at 137.16 125.73 0)
 			(effects
@@
 			)
 		)
+		(property "LCSC" "C25794"
+			(at 137.16 125.73 0)
+			(effects
+				(font
+					(size 1.27 1.27)
+				)
+				(hide yes)
+			)
+		)
 		(pin "1"
 		)
@@
 			)
 		)
-		(property "Datasheet" ""
+		(property "Datasheet" "https://www.lcsc.com/product-detail/Chip-Resistor-Surface-Mount_UNI-ROYAL-Uniroyal-Elec-0402WGF5102TCE_C25794.html"
 			(at 149.86 125.73 0)
 			(effects
@@
 			(at 149.86 125.73 0)
 			(effects
+				(font
+					(size 1.27 1.27)
+				)
+				(hide yes)
+			)
+		)
+		(property "LCSC" "C25794"
+			(at 149.86 125.73 0)
+			(effects
