File: esp32p4.kicad_sch (KiCad schematic)
At the start: 62 parts, among them Q5 AO3400 (A09T), Q6 AO3400 (A09T), U13 W25Q128JVS, U3 TLV62569DBV, U7 CH340K, U8 ESP32-P4, Y3 40MHz

Commit message: VBUS trace wider to PMIC, moved signal out under USB diff pair line, fix RX/TX P4.
Parts:
- added R82: 51k, Resistor_SMD:R_0402_1005Metric, symbol Device:R
Connections:
- net +3.3V: now also R82.2
- net E2: now also R82.1
- net P4_RX: now also U8.70 (GPIO38); no longer U8.69 (GPIO37)
- net P4_TX: now also U8.69 (GPIO37); no longer U8.70 (GPIO38)
Changed lines of the file:
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@@
 	)
 	(junction
+		(at 46.99 154.94)
+		(diameter 0)
+		(color 0 0 0 0)
+	)
+	(junction
 		(at 181.61 46.99)
 		(diameter 0)
@@
 	)
 	(junction
+		(at 46.99 120.65)
+		(diameter 0)
+		(color 0 0 0 0)
+	)
+	(junction
 		(at 135.89 161.29)
 		(diameter 0)
@@
 	(wire
 		(pts
+			(xy 46.99 120.65) (xy 66.04 120.65)
+		)
+		(stroke
+			(width 0)
+			(type default)
+		)
+	)
+	(wire
+		(pts
 			(xy 27.94 193.04) (xy 82.55 193.04)
 		)
@@
 	(wire
 		(pts
+			(xy 46.99 154.94) (xy 82.55 154.94)
+		)
+		(stroke
+			(width 0)
+			(type default)
+		)
+	)
+	(wire
+		(pts
 			(xy 118.11 26.67) (xy 123.19 26.67)
 		)
@@
 	(wire
 		(pts
+			(xy 46.99 128.27) (xy 46.99 154.94)
+		)
+		(stroke
+			(width 0)
+			(type default)
+		)
+	)
+	(wire
+		(pts
 			(xy 120.65 21.59) (xy 120.65 24.13)
 		)
@@
 	(wire
 		(pts
+			(xy 41.91 120.65) (xy 46.99 120.65)
+		)
+		(stroke
+			(width 0)
+			(type default)
+		)
+	)
+	(wire
+		(pts
 			(xy 64.77 168.91) (xy 64.77 177.8)
 		)
@@
 	(wire
 		(pts
-			(xy 41.91 120.65) (xy 66.04 120.65)
-		)
-		(stroke
-			(width 0)
-			(type default)
-		)
-	)
-	(wire
-		(pts
 			(xy 236.22 86.36) (xy 260.35 86.36)
 		)
@@
 	(wire
 		(pts
-			(xy 26.67 154.94) (xy 82.55 154.94)
+			(xy 26.67 154.94) (xy 46.99 154.94)
 		)
 		(stroke
@@
 	(global_label "P4_RX"
 		(shape input)
-		(at 26.67 162.56 180)
+		(at 26.67 165.1 180)
 		(fields_autoplaced yes)
 		(effects
@@
 		)
 		(property "Intersheetrefs" "${INTERSHEET_REFS}"
-			(at 19.5408 162.56 0)
+			(at 19.5408 165.1 0)
 			(effects
 				(font
@@
 	(global_label "P4_TX"
 		(shape output)
-		(at 26.67 165.1 180)
+		(at 26.67 162.56 180)
 		(fields_autoplaced yes)
 		(effects
@@
 		)
 		(property "Intersheetrefs" "${INTERSHEET_REFS}"
-			(at 19.7827 165.1 0)
+			(at 19.7827 162.56 0)
 			(effects
 				(font
@@
 					(unit 1)
 				)
+			)
+		)
+	)
+	(symbol
+		(lib_id "Device:R")
+		(at 46.99 124.46 0)
+		(mirror x)
+		(unit 1)
+		(exclude_from_sim no)
+		(in_bom yes)
+		(on_board yes)
+		(dnp no)
+		(property "Reference" "R82"
+			(at 50.292 123.444 0)
+			(effects
+				(font
+					(size 1.27 1.27)
+				)
+			)
+		)
+		(property "Value" "51k"
+			(at 50.292 125.73 0)
+			(effects
+				(font
+					(size 1.27 1.27)
+				)
+			)
+		)
+		(property "Footprint" "Resistor_SMD:R_0402_1005Metric"
+			(at 45.212 124.46 90)
+			(effects
+				(font
+					(size 1.27 1.27)
+				)
+				(hide yes)
+			)
+		)
+		(property "Datasheet" "https://www.lcsc.com/product-detail/Chip-Resistor-Surface-Mount_UNI-ROYAL-Uniroyal-Elec-0402WGF5102TCE_C25794.html"
+			(at 46.99 124.46 0)
+			(effects
+				(font
+					(size 1.27 1.27)
+				)
+				(hide yes)
+			)
+		)
+		(property "Description" ""
+			(at 46.99 124.46 0)
+			(effects
+				(font
+					(size 1.27 1.27)
+				)
+				(hide yes)
+			)
+		)
+		(property "LCSC" "C25794"
+			(at 46.99 124.46 0)
+			(effects
+				(font
+					(size 1.27 1.27)
+				)
+				(hide yes)
+			)
+		)
+		(pin "1"
+		)
+		(pin "2"
+		)
+		(instances
+			(project "why2025"
+				(path "/6a31734e-65de-48f3-8156-2b24b665b183/3d60835a-4261-467a-b239-9fb76f6e13a1"
+					(reference "R82")
+					(unit 1)
+				)

Commit message: Add 1.5k pull-up to D+ of C6, remove logos, add JTAG connector, fix SAO pinout
Parts:
- added J11: JTAG, Connector_PinHeader_1.27mm:PinHeader_2x05_P1.27mm_Vertical_SMD, symbol Connector:Conn_ARM_JTAG_SWD_10
- added R84: 1.5k, Resistor_SMD:R_0402_1005Metric, symbol symbols:R
Connections:
- net +3.3V: now also J11.1 (VTref)
- net E2: now also R84.2
- net GND: now also J11.3 (GND), J11.5 (GND)
- net MTCK: now also J11.4 (SWCLK/TCK)
- net MTDI: now also J11.8 (NC/TDI)
- net MTDO: now also J11.6 (SWO/TDO)
- net MTMS: now also J11.2 (SWDIO/TMS)
- net P4_RESET: now also J11.10 (~{RESET})
- net SAO_IO1: now also U8.16 (GPIO15); no longer U8.104 (GPIO0)
- net SAO_IO2: now also U8.104 (GPIO0); no longer U8.16 (GPIO15)
- new net: J11.9 (GNDDetect), R84.1
Other:
- moved on the sheet: C28, C30, C38, C39, C40, C41, C43, C45, C47, C48, C51, C53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

Commit message: Made more space around the D87, smooth curve LORA antenna.
Changed lines of the file:
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@@
 		)
 		(property "Value" "51k"
-			(at 51.562 101.6 0)
+			(at 51.562 101.092 0)
 			(effects
 				(font

Commit message: Add extra header for JTAG reset and detect.
Parts:
- removed J11: JTAG, Connector_PinHeader_1.27mm:PinHeader_2x05_P1.27mm_Vertical_SMD, symbol Connector:Conn_ARM_JTAG_SWD_10
- removed R84: 1.5k, Resistor_SMD:R_0402_1005Metric, symbol symbols:R

Commit message: Swapped GPIO32 and GPIO00, added functionality to use 1 3v3 pin as the P4 RESET.
Connections:
- net E2: now also U8.104 (GPIO0); no longer R82.1, U8.65 (GPIO34)
- net SAO_IO2: now also R82.1, U8.65 (GPIO34); no longer U8.104 (GPIO0)
Changed lines of the file:
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@@
 	(hierarchical_label "E2"
 		(shape bidirectional)
-		(at 27.94 130.81 180)
+		(at 27.94 26.67 180)
 		(fields_autoplaced yes)
 		(effects
@@
 	(hierarchical_label "SAO_IO2"
 		(shape bidirectional)
-		(at 27.94 26.67 180)
-		(fields_autoplaced yes)
-		(effects
+		(at 27.94 130.81 180)
+		(fields_autoplaced yes)
+		(effects

Commit message: Change internal I2C bus 4.7k pullups to 2.2k, in order to get a better rise time on the signal.
Parts:
- R13, R15: value 4k7 -> 2k2; LCSC C25900 -> C25879
Changed lines of the file:
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@@
 			)
 		)
-		(property "Value" "4k7"
+		(property "Value" "2k2"
 			(at 48.26 19.05 90)
 			(effects
@@
 			)
 		)
-		(property "LCSC" "C25900"
+		(property "LCSC" "C25879"
 			(at 48.26 19.05 0)
 			(effects
@@
 		(on_board yes)
 		(dnp no)
+		(fields_autoplaced yes)
 		(property "Reference" "R15"
 			(at 50.038 19.05 90)
@@
 			)
 		)
-		(property "Value" "4k7"
+		(property "Value" "2k2"
 			(at 52.07 19.05 90)
 			(effects
@@
 			)
 		)
-		(property "LCSC" "C25900"
+		(property "LCSC" "C25879"
 			(at 52.07 19.05 0)
 			(effects

Commit message: Switch SDA and SCL I3C bus as they were switched.
Connections:
- net I3C_SCL: now also U8.63 (GPIO32); no longer U8.64 (GPIO33)
- net I3C_SDA: now also U8.64 (GPIO33); no longer U8.63 (GPIO32)
Changed lines of the file:
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@@
 	(hierarchical_label "I3C_SCL"
 		(shape output)
-		(at 27.94 128.27 180)
+		(at 27.94 125.73 180)
 		(fields_autoplaced yes)
 		(effects
@@
 	(hierarchical_label "I3C_SDA"
 		(shape bidirectional)
-		(at 27.94 125.73 180)
+		(at 27.94 128.27 180)
 		(fields_autoplaced yes)
 		(effects
