File: audio.kicad_sch (KiCad schematic)
At the start: 0 parts

Commit message: More schematics
Changed lines of the file:
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@@
 		(date "2024-04-02")
+	)
+	(wire
+		(pts
+			(xy 140.97 82.55) (xy 143.51 82.55)
+		)
+		(stroke
+			(width 0)
+			(type default)
+		)
+	)
+	(wire
+		(pts
+			(xy 140.97 80.01) (xy 140.97 82.55)
+		)
+		(stroke
+			(width 0)
+			(type default)
+		)
+	)
+	(wire
+		(pts
+			(xy 143.51 80.01) (xy 140.97 80.01)
+		)
+		(stroke
+			(width 0)
+			(type default)
+		)
+	)
+	(hierarchical_label "SPEAKER"
+		(shape output)
+		(at 143.51 82.55 0)
+		(fields_autoplaced yes)
+		(effects
+			(font
+				(size 1.27 1.27)
+			)
+			(justify left)
+		)
 	)
 	(hierarchical_label "HP_R"
@@
 		)
 	)
+	(hierarchical_label "I2S_MCLK"
+		(shape input)
+		(at 86.36 58.42 180)
+		(fields_autoplaced yes)
+		(effects
+			(font
+				(size 1.27 1.27)
+			)
+			(justify right)
+		)
+	)
+	(hierarchical_label "I2S_LRCK"
+		(shape input)
+		(at 86.36 55.88 180)
+		(fields_autoplaced yes)
+		(effects
+			(font
+				(size 1.27 1.27)
+			)
+			(justify right)
+		)
+	)
+	(hierarchical_label "I2S_SCLK"
+		(shape input)
+		(at 86.36 53.34 180)
+		(fields_autoplaced yes)
+		(effects
+			(font
+				(size 1.27 1.27)
+			)
+			(justify right)
+		)
+	)
+	(hierarchical_label "HP_NC"
+		(shape input)
+		(at 143.51 80.01 0)
+		(fields_autoplaced yes)
+		(effects
+			(font
+				(size 1.27 1.27)
+			)
+			(justify left)
+		)
+	)
+	(hierarchical_label "I2S_DATA"
+		(shape input)
+		(at 86.36 50.8 180)
+		(fields_autoplaced yes)
+		(effects
+			(font
+				(size 1.27 1.27)
+			)
+			(justify right)
+		)
+	)

Commit message: More work on the schematic, add protection circuit, fix display pinout
Parts:
- added C59, C60: 0.39u, tanoshii:C_0603_1608Metric, symbol symbols:C
- added C61, C62, C63, C67: 1u, Capacitor_SMD:C_0603_1608Metric, symbol Device:C
- added C64: 100n, Capacitor_SMD:C_0402_1005Metric, symbol Device:C
- added C65, C66: 22u, Capacitor_SMD:C_1206_3216Metric, symbol Device:C
- added C68, C69: 1u, tanoshii:C_0402_1005Metric, symbol symbols:C
- added C70: 100n, tanoshii:C_0402_1005Metric, symbol symbols:C
- added C71, C72: 22p, Capacitor_SMD:C_0402_1005Metric, symbol Device:C
- added Q3: AP2302B, hh24:SOT-23, symbol symbols:Q_NMOS_GSD
- added Q4: AP2302B, Package_TO_SOT_SMD:SOT-23, symbol mch2021-rescue:Q_NMOS_GSD-Device
- added R67, R68: 33, Resistor_SMD:R_0402_1005Metric, symbol Device:R
- added R69, R73: 0, Resistor_SMD:R_0402_1005Metric, symbol Device:R
- added R70, R72: 100k, Resistor_SMD:R_0402_1005Metric, symbol Device:R
- added R71: 100k, tanoshii:R_0402_1005Metric, symbol symbols:R
- added R74: 4k7, tanoshii:R_0402_1005Metric, symbol symbols:R
- added R75: 10k, tanoshii:R_0402_1005Metric, symbol symbols:R
- added R76, R77, R78, R79: 5k1, tanoshii:R_0402_1005Metric, symbol symbols:R
- added U14: ~, Package_DFN_QFN:VQFN-20-1EP_3x3mm_P0.4mm_EP1.7x1.7mm, symbol ES8156:ES8156
- added U16: FM8002A, Package_SO:SSOP-8_3.9x5.05mm_P1.27mm, symbol symbols:FM8002A
Connections:
- net HP_L: now also R67.2
- net HP_R: now also R68.2
- net I2S_DATA: now also U14.8 (SDIN)
- net I2S_LRCK: now also U14.9 (LRCK)
- net I2S_MCLK: now also U14.3 (MCLK)
- net I2S_SCLK: now also U14.7 (SCLK)
- new net: R78.1, U16.4 (-IN)
- new net: R76.1, R78.2
- new net: Q4.1 (G), R74.2
- new net: Q4.3 (D), R75.2, U16.1 (SHUTDOWN)
- new net: C66.2, R68.1
- new net: R79.1, U16.3 (+IN)
- new net: R77.1, R79.2
- new net: C60.2, C65.1, C72.1, U14.15 (LOUTP)
- new net: C68.2, U16.2 (BYPASS)
- new net: C61.1, U14.18 (VMID)
- new net: C59.2, C71.1, U14.14 (LOUTN)
- new net: C59.1, R76.2
- new net: C66.1, U14.11 (ROUTP)
- new net: C62.1, U14.17 (VRP)
- new net: C60.1, R77.2
- new net: C65.2, R67.1
- new net +3.3V: C63.1, C64.1, R73.1, U14.4 (DVDD), U14.5 (PVDD)
- new net +3.3VA: C67.1, R70.2, R72.2, R73.2, U14.16 (AVDD)
- new net AMP_EN: R71.1, R74.1
- new net GND: R69.1
- new net GNDA: C61.2, C62.2, C63.2, C64.2, C67.2, C68.1, C69.2, C70.2, C71.2, C72.2, Q3.2 (S), Q4.2 (S), R69.2, R71.2, U14.13 (AGND), U14.19 (CE), U14.21 (PGND), U14.6 (DGND), U16.7 (GND)
- new net HP_DET: Q3.3 (D), R70.1
- new net HP_S: Q3.1 (G), R72.1
- new net SCL: U14.2 (CCLK)
- new net SDA: U14.1 (CDATA)
- new net SPK+: U16.8 (VO2)
- new net SPK-: U16.5 (VO1)
- new net VSYS: C69.1, C70.1, R75.1, U16.6 (VDD)
- no-connect marks 0 -> 3
Other:
- note added: "To-do For improved audio quality use LDO for AVDD"
- company: (none) -> Badge.Team
- title: (none) -> WHY2025 badge

Commit message: Assign footprints, create P4 footprint
Parts:
- C59, C60: footprint tanoshii:C_0603_1608Metric -> Capacitor_SMD:C_0603_1608Metric
- C68, C69: footprint tanoshii:C_0402_1005Metric -> Capacitor_SMD:C_0603_1608Metric
- C70: footprint tanoshii:C_0402_1005Metric -> Capacitor_SMD:C_0402_1005Metric
- Q3: footprint hh24:SOT-23 -> Package_TO_SOT_SMD:SOT-23
- R71, R74, R75, R76, R77, R78, R79: footprint tanoshii:R_0402_1005Metric -> Resistor_SMD:R_0402_1005Metric

Commit message: Bill of materials part 1
Parts:
- C61, C62, C63, C67: LCSC (none) -> C107372
- C64: LCSC (none) -> C307331
- Q3: Link https://www.lcsc.com/product-detail/MOSFETs_ALLPOWER-ShenZh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 -> (none)
- Q4: Buy early Y -> (none); Category Transistors -> (none); MANUFACTURER ALLPOWER -> (none); MPN AP2302B -> (none); Manufacturer Allpower -> (none); Mouser - -> (none); Sponsored N -> (none)
- R70, R72: LCSC (none) -> C25741
- R75: LCSC C25744 -> C60490
- R76, R77, R78, R79: LCSC C25941 -> C25905
- U14: value ~ -> ES8156; LCSC (none) -> C2887138

Commit message: Bill of materials part 2
Parts:
- C65, C66: LCSC (none) -> C342620
- C71, C72: LCSC (none) -> C1555
Changed lines of the file:
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@@
 			)
 		)
-		(property "Datasheet" ""
+		(property "Datasheet" "https://datasheet.lcsc.com/lcsc/2304140030_FH--Guangdong-Fenghua-Advanced-Tech-0402CG220J500NT_C1555.pdf"
 			(at 120.65 120.65 0)
 			(effects
@@
 			)
 		)
-		(property "Description" "Unpolarized capacitor"
+		(property "Description" ""
+			(at 120.65 120.65 0)
+			(effects
+				(font
+					(size 1.27 1.27)
+				)
+				(hide yes)
+			)
+		)
+		(property "LCSC" "C1555"
 			(at 120.65 120.65 0)
 			(effects
@@
 			)
 		)
-		(property "Datasheet" ""
+		(property "Datasheet" "https://datasheet.lcsc.com/lcsc/2304140030_FH--Guangdong-Fenghua-Advanced-Tech-0402CG220J500NT_C1555.pdf"
 			(at 115.57 120.65 0)
 			(effects
@@
 			)
 		)
-		(property "Description" "Unpolarized capacitor"
+		(property "Description" ""
+			(at 115.57 120.65 0)
+			(effects
+				(font
+					(size 1.27 1.27)
+				)
+				(hide yes)
+			)
+		)
+		(property "LCSC" "C1555"
 			(at 115.57 120.65 0)
 			(effects
@@
 			)
 		)
-		(property "Datasheet" ""
+		(property "Datasheet" "https://datasheet.lcsc.com/lcsc/2304140030_TDK-C3216X5R1V226MTJ00E_C342620.pdf"
 			(at 88.9 99.06 0)
 			(effects
@@
 		)
 		(property "Description" ""
+			(at 88.9 99.06 0)
+			(effects
+				(font
+					(size 1.27 1.27)
+				)
+				(hide yes)
+			)
+		)
+		(property "LCSC" "C342620"
 			(at 88.9 99.06 0)
 			(effects
@@
 			)
 		)
-		(property "Datasheet" ""
+		(property "Datasheet" "https://datasheet.lcsc.com/lcsc/2304140030_TDK-C3216X5R1V226MTJ00E_C342620.pdf"
 			(at 88.9 91.44 0)
 			(effects
@@
 			(at 88.9 91.44 0)
 			(effects
+				(font
+					(size 1.27 1.27)
+				)
+				(hide yes)
+			)
+		)
+		(property "LCSC" "C342620"
+			(at 88.9 91.44 0)
+			(effects
