File: audio.kicad_sch (KiCad schematic)
At the start: 31 parts, among them Q3 AP2302B, Q4 AP2302B, U14 ES8156, U16 FM8002A

Commit message: Small tweaks and fixes, update LCSC numbers on some components, change to new key type for power key
Parts:
- R67, R68: LCSC (none) -> C25105
- R69, R73: LCSC (none) -> C17168
Changed lines of the file:
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@@
 			)
 		)
-		(property "Description" "Resistor"
+		(property "Description" ""
+			(at 96.52 99.06 0)
+			(effects
+				(font
+					(size 1.27 1.27)
+				)
+				(hide yes)
+			)
+		)
+		(property "LCSC" "C25105"
 			(at 96.52 99.06 0)
 			(effects
@@
 			)
 		)
-		(property "Description" "Resistor"
+		(property "Description" ""
+			(at 30.48 52.07 0)
+			(effects
+				(font
+					(size 1.27 1.27)
+				)
+				(hide yes)
+			)
+		)
+		(property "LCSC" "C17168"
 			(at 30.48 52.07 0)
 			(effects
@@
 			)
 		)
-		(property "Description" "Resistor"
+		(property "Description" ""
+			(at 30.48 124.46 0)
+			(effects
+				(font
+					(size 1.27 1.27)
+				)
+				(hide yes)
+			)
+		)
+		(property "LCSC" "C17168"
 			(at 30.48 124.46 0)
 			(effects
@@
 			)
 		)
-		(property "Description" "Resistor"
+		(property "Description" ""
 			(at 96.52 91.44 0)
 			(effects
+				(font
+					(size 1.27 1.27)
+				)
+				(hide yes)
+			)
+		)
+		(property "LCSC" "C25105"
+			(at 96.52 91.44 0)
+			(effects

Commit message: More routing, moved some more signals
Parts:
- removed R73: 0, Resistor_SMD:R_0402_1005Metric, symbol Device:R
Connections:
- net +3.3VA is gone; now on net +3.3V: C67.1, R70.2, R72.2, U14.16 (AVDD)
Changed lines of the file:
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@@
-	(wire
-		(pts
-			(xy 36.83 52.07) (xy 34.29 52.07)
-		)
-		(stroke
-			(width 0)
-			(type default)
-		)
-	)
 	(wire
 		(pts
@@
 	(wire
 		(pts
-			(xy 26.67 52.07) (xy 24.13 52.07)
+			(xy 24.13 52.07) (xy 36.83 52.07)
 		)
 		(stroke
@@
 					(unit 1)
 				)
-			)
-		)
-	)
-	(symbol
-		(lib_id "Device:R")
-		(at 30.48 52.07 90)
-		(unit 1)
-		(exclude_from_sim no)
-		(in_bom yes)
-		(on_board yes)
-		(dnp no)
-		(property "Reference" "R73"
-			(at 30.48 49.784 90)
-			(effects
-				(font
-					(size 1.27 1.27)
-				)
-			)
-		)
-		(property "Value" "0"
-			(at 30.48 54.61 90)
-			(effects
-				(font
-					(size 1.27 1.27)
-				)
-			)
-		)
-		(property "Footprint" "Resistor_SMD:R_0402_1005Metric"
-			(at 30.48 53.848 90)
-			(effects
-				(font
-					(size 1.27 1.27)
-				)
-				(hide yes)
-			)
-		)
-		(property "Datasheet" ""
-			(at 30.48 52.07 0)
-			(effects
-				(font
-					(size 1.27 1.27)
-				)
-				(hide yes)
-			)
-		)
-		(property "Description" ""
-			(at 30.48 52.07 0)
-			(effects
-				(font
-					(size 1.27 1.27)
-				)
-				(hide yes)
-			)
-		)
-		(property "LCSC" "C17168"
-			(at 30.48 52.07 0)
-			(effects
-				(font
-					(size 1.27 1.27)
-				)
-				(hide yes)
-			)
-		)
-		(pin "2"
-		)
-		(pin "1"
-		)
-		(instances
-			(project "why2025"
-				(path "/6a31734e-65de-48f3-8156-2b24b665b183/26e0a3c5-321c-4e16-844f-a29ed28cc9bc"
-					(reference "R73")
-					(unit 1)
-				)

Commit message: All wires routed, lots of DRC errors to go
Parts:
- C65, C66: footprint Capacitor_SMD:C_1206_3216Metric -> Capacitor_SMD:C_0805_2012Metric; LCSC C342620 -> C45783
Changed lines of the file:
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@@
 			)
 		)
-		(property "Footprint" "Capacitor_SMD:C_1206_3216Metric"
+		(property "Footprint" "Capacitor_SMD:C_0805_2012Metric"
 			(at 92.71 98.0948 0)
 			(effects
@@
 			)
 		)
-		(property "Datasheet" "https://datasheet.lcsc.com/lcsc/2304140030_TDK-C3216X5R1V226MTJ00E_C342620.pdf"
+		(property "Datasheet" "https://www.lcsc.com/product-detail/Multilayer-Ceramic-Capacitors-MLCC-SMD-SMT_Samsung-Electro-Mechanics-CL21A226MAQNNNE_C45783.html"
 			(at 88.9 99.06 0)
 			(effects
@@
 			)
 		)
-		(property "LCSC" "C342620"
+		(property "LCSC" "C45783"
 			(at 88.9 99.06 0)
 			(effects
@@
 			)
 		)
-		(property "Footprint" "Capacitor_SMD:C_1206_3216Metric"
+		(property "Footprint" "Capacitor_SMD:C_0805_2012Metric"
 			(at 92.71 90.4748 0)
 			(effects
@@
 			)
 		)
-		(property "Datasheet" "https://datasheet.lcsc.com/lcsc/2304140030_TDK-C3216X5R1V226MTJ00E_C342620.pdf"
+		(property "Datasheet" "https://www.lcsc.com/product-detail/Multilayer-Ceramic-Capacitors-MLCC-SMD-SMT_Samsung-Electro-Mechanics-CL21A226MAQNNNE_C45783.html"
 			(at 88.9 91.44 0)
 			(effects
@@
 			)
 		)
-		(property "LCSC" "C342620"
+		(property "LCSC" "C45783"
 			(at 88.9 91.44 0)
 			(effects
@@
 			)
 		)
-		(property "Description" "Resistor"
+		(property "Description" ""
 			(at 256.54 107.95 0)
 			(effects
@@
 			)
 		)
-		(property "Description" "Resistor"
+		(property "Description" ""
 			(at 266.7 107.95 0)
 			(effects

Commit message: Frontpanel :D
Parts:
- C61, C62, C63, C67, C68, C69: LCSC C107372 -> C5199872
Changed lines of the file:
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@@
 			)
 		)
-		(property "LCSC" "C107372"
+		(property "LCSC" "C5199872"
 			(at 48.26 58.42 0)
 			(effects
@@
 			)
 		)
-		(property "LCSC" "C107372"
+		(property "LCSC" "C5199872"
 			(at 52.07 123.19 0)
 			(effects
@@
 			)
 		)
-		(property "LCSC" "C107372"
+		(property "LCSC" "C5199872"
 			(at 77.47 58.42 0)
 			(effects
@@
 			)
 		)
-		(property "LCSC" "C107372"
+		(property "LCSC" "C5199872"
 			(at 44.45 123.19 0)
 			(effects
@@
 			)
 		)
-		(property "LCSC" "C107372"
+		(property "LCSC" "C5199872"
 			(at 179.07 110.49 0)
 			(effects
@@
 			)
 		)
-		(property "LCSC" "C107372"
+		(property "LCSC" "C5199872"
 			(at 231.14 109.22 0)
 			(effects

Commit message: Fix audio amplifier circuit
Parts:
- removed C59: 0.39u, Capacitor_SMD:C_0603_1608Metric, symbol symbols:C
- removed R76, R78: 5k1, Resistor_SMD:R_0402_1005Metric, symbol symbols:R
- added R62, R63: 10k, Resistor_SMD:R_0402_1005Metric, symbol Device:R
- added TP20: SCLK, TestPoint:TestPoint_Pad_1.0x1.0mm, symbol Connector:TestPoint
- added TP21: LRCK, TestPoint:TestPoint_Pad_1.0x1.0mm, symbol Connector:TestPoint
- added TP22: DATA, TestPoint:TestPoint_Pad_1.0x1.0mm, symbol Connector:TestPoint
- added TP23: DOUT, TestPoint:TestPoint_Pad_1.0x1.0mm, symbol Connector:TestPoint
- added TP4: HPCOM, TestPoint:TestPoint_Pad_1.0x1.0mm, symbol Connector:TestPoint
- added TP7: MCLK, TestPoint:TestPoint_Pad_1.0x1.0mm, symbol Connector:TestPoint
Connections:
- net I2S_DATA: now also TP22.1
- net I2S_LRCK: now also TP21.1
- net I2S_MCLK: now also TP7.1
- net I2S_SCLK: now also TP20.1
- net SPK-: now also R63.2
- net at U16.4 (-IN): now also R79.1, R62.1
- net at U16.3 (+IN): now also C68.2, U16.2 (BYPASS); no longer R79.1
- net at C60.2, C65.1, U14.15 (LOUTP): now also C71.1; no longer C72.1
- net at U14.14 (LOUTN): no longer C71.1
- net at C66.1, U14.11 (ROUTP): now also C72.1
- net at U14.10 (HPCOM): now also TP4.1
- net at U14.20 (SDOUT): now also TP23.1
- new net: R62.2, R63.1
- no-connect marks 3 -> 2
Other:
- moved on the sheet: C60, C65, C66, C68, C71, C72, Q3, R67, R68, R70, R72, R77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
