File: display.kicad_sch (KiCad schematic)
At the start: 2 parts, among them J12 DF40C-24DS-0.4V_51_

Commit message: More work on the schematic, add protection circuit, fix display pinout
Parts:
- removed J12: DF40C-24DS-0.4V_51_, library:HIROSE_DF40C-24DS-0.4V_51_, symbol DF40C-24DS-0.4V_51_:DF40C-24DS-0.4V_51_
- added J14: LH397K, library:LH397K-IC01, symbol LH397K-IC01:LH397K-IC01
- added R98: 10k, Resistor_SMD:R_0402_1005Metric, symbol Device:R
Connections:
- net +3.3V: now also J14.23 (VCI), J14.24 (IOVCC), R98.2
- net +BL-LCD: now also J14.2 (LEDA)
- net -BL-LCD: now also J14.1 (LEDK)
- net CLK_N: now also J14.8 (TCN)
- net CLK_P: now also J14.7 (TCP)
- net D0_N: now also J14.5 (TDN0)
- net D0_P: now also J14.4 (TDP0)
- net D1_N: now also J14.11 (TDN1)
- net D1_P: now also J14.10 (TDP1)
- net GND: now also J14.12 (GND), J14.13 (GND), J14.14 (GND), J14.15 (GND), J14.16 (GND), J14.17 (GND), J14.18 (GND), J14.19 (GND), J14.22 (GND), J14.3 (GND), J14.6 (GND), J14.9 (GND)
- net RST: now also J14.21 (RESET)
- new net TE: J14.20 (TE), R98.1
Other:
- note added: "To-do This display is one of the options we're evaluating, might change."
- company: (none) -> Badge.Team
- title: (none) -> WHY2025 badge
- moved on the sheet: R50

Commit message: Bill of materials part 1
Parts:
- J14: LCSC (none) -> C424640
- R50, R98: LCSC (none) -> C60490
Other:
- note removed: "To-do This display is one of the options we're evaluating, might change."
