File: display.kicad_sch (KiCad schematic)
At the start: 3 parts, among them J14 LH397K

Commit message: 18-Add correct display connector
Parts:
- removed J14: LH397K, library:LH397K-IC01, symbol LH397K-IC01:LH397K-IC01
- added CN1: DF37NB-24DS-0.4V(51), lcsc:CONN-SMD_DF37NB-24DS-0.4V, symbol lcsc:DF37NB-24DS-0.4V(51)
Connections:
- net +3.3V: now also CN1.2, CN1.4
- net +BL-LCD: now also CN1.3
- net -BL-LCD: now also CN1.1
- net CLK_N: now also CN1.15
- net CLK_P: now also CN1.13
- net D0_N: now also CN1.9
- net D0_P: now also CN1.7
- net D1_N: now also CN1.21
- net D1_P: now also CN1.19
- net GND: now also CN1.11, CN1.12, CN1.14, CN1.16, CN1.17, CN1.18, CN1.20, CN1.22, CN1.23, CN1.24, CN1.25, CN1.26, CN1.5, CN1.6
- net RST: now also CN1.8
- net TE: now also CN1.10
Other:
- note added: "!! The Footprint is numbered criss cross, in the display datasheet it's not. In the display datasheet: start, top left 1 down to 12 then, right bottom up 13 to 24. So some mapping needs to be done here, if another footprint is inserted here."
- moved on the sheet: R50, R98

Commit message: Disconnect PG from reset of P4, connect to GPIO of CH32, fix warnings, make some vias bigger, add BHI360
Changed lines of the file:
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@@
 	(wire
 		(pts
-			(xy 133.35 106.68) (xy 133.35 109.22)
+			(xy 133.35 106.68) (xy 133.35 111.76)
 		)
 		(stroke
@@
 	(wire
 		(pts
-			(xy 153.67 106.68) (xy 153.67 109.22)
+			(xy 153.67 106.68) (xy 153.67 111.76)
 		)
 		(stroke
@@
 	(symbol
 		(lib_id "power:GND")
-		(at 133.35 109.22 0)
+		(at 133.35 111.76 0)
 		(unit 1)
 		(exclude_from_sim no)
@@
 		(fields_autoplaced yes)
 		(property "Reference" "#PWR0190"
-			(at 133.35 115.57 0)
+			(at 133.35 118.11 0)
 			(effects
 				(font
@@
 		)
 		(property "Value" "GND"
-			(at 133.35 114.3 0)
+			(at 133.35 116.84 0)
 			(effects
 				(font
@@
 		)
 		(property "Footprint" ""
-			(at 133.35 109.22 0)
+			(at 133.35 111.76 0)
 			(effects
 				(font
@@
 		)
 		(property "Datasheet" ""
-			(at 133.35 109.22 0)
+			(at 133.35 111.76 0)
 			(effects
 				(font
@@
 		)
 		(property "Description" ""
-			(at 133.35 109.22 0)
+			(at 133.35 111.76 0)
 			(effects
 				(font
@@
 	(symbol
 		(lib_id "power:GND")
-		(at 153.67 109.22 0)
+		(at 153.67 111.76 0)
 		(unit 1)
 		(exclude_from_sim no)
@@
 		(fields_autoplaced yes)
 		(property "Reference" "#PWR0191"
-			(at 153.67 115.57 0)
+			(at 153.67 118.11 0)
 			(effects
 				(font
@@
 		)
 		(property "Value" "GND"
-			(at 153.67 114.3 0)
+			(at 153.67 116.84 0)
 			(effects
 				(font
@@
 		)
 		(property "Footprint" ""
-			(at 153.67 109.22 0)
+			(at 153.67 111.76 0)
 			(effects
 				(font
@@
 		)
 		(property "Datasheet" ""
-			(at 153.67 109.22 0)
+			(at 153.67 111.76 0)
 			(effects
 				(font
@@
 		)
 		(property "Description" ""
-			(at 153.67 109.22 0)
-			(effects
-				(font
+			(at 153.67 111.76 0)
+			(effects
+				(font

Commit message: Moved antenna more away from wifi, replaced more 0.2 with 0.3 mm vias.
Parts:
- added C49, C58: 10n, Capacitor_SMD:C_0402_1005Metric, symbol Device:C
Connections:
- net +3.3V: now also C49.1, C58.1
- net GND: now also C49.2, C58.2

Commit message: Add datasheet for df3znb connector.
Parts:
- added C26, C46: 10n, Capacitor_SMD:C_0402_1005Metric, symbol Device:C
Connections:
- net +3.3V: now also C26.1, C46.1
- net GND: now also C26.2, C46.2
Changed lines of the file:
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@@
+	)
+	(junction
+		(at 73.66 81.28)
+		(diameter 0)
+		(color 0 0 0 0)
 	)
 	(junction
@@
 	)
 	(junction
+		(at 73.66 73.66)
+		(diameter 0)
+		(color 0 0 0 0)
+	)
+	(junction
 		(at 85.09 73.66)
 		(diameter 0)
@@
 	(wire
 		(pts
+			(xy 73.66 81.28) (xy 85.09 81.28)
+		)
+		(stroke
+			(width 0)
+			(type default)
+		)
+	)
+	(wire
+		(pts
+			(xy 62.23 81.28) (xy 73.66 81.28)
+		)
+		(stroke
+			(width 0)
+			(type default)
+		)
+	)
+	(wire
+		(pts
 			(xy 151.13 91.44) (xy 153.67 91.44)
 		)
@@
 	(wire
 		(pts
+			(xy 62.23 73.66) (xy 73.66 73.66)
+		)
+		(stroke
+			(width 0)
+			(type default)
+		)
+	)
+	(wire
+		(pts
 			(xy 130.81 93.98) (xy 135.89 93.98)
 		)
@@
 		(pts
 			(xy 151.13 99.06) (xy 153.67 99.06)
+		)
+		(stroke
+			(width 0)
+			(type default)
+		)
+	)
+	(wire
+		(pts
+			(xy 73.66 73.66) (xy 85.09 73.66)
 		)
 		(stroke
@@
 			)
 			(justify right)
+		)
+	)
+	(symbol
+		(lib_id "Device:C")
+		(at 73.66 77.47 0)
+		(unit 1)
+		(exclude_from_sim no)
+		(in_bom yes)
+		(on_board yes)
+		(dnp no)
+		(fields_autoplaced yes)
+		(property "Reference" "C46"
+			(at 77.47 76.1999 0)
+			(effects
+				(font
+					(size 1.27 1.27)
+				)
+				(justify left)
+			)
+		)
+		(property "Value" "10n"
+			(at 77.47 78.7399 0)
+			(effects
+				(font
+					(size 1.27 1.27)
+				)
+				(justify left)
+			)
+		)
+		(property "Footprint" "Capacitor_SMD:C_0402_1005Metric"
+			(at 74.6252 81.28 0)
+			(effects
+				(font
+					(size 1.27 1.27)
+				)
+				(hide yes)
+			)
+		)
+		(property "Datasheet" "https://wmsc.lcsc.com/wmsc/upload/file/pdf/v2/lcsc/2304140030_Samsung-Electro-Mechanics-CL05B103KB5NNNC_C15195.pdf"
+			(at 73.66 77.47 0)
+			(effects
+				(font
+					(size 1.27 1.27)
+				)
+				(hide yes)
+			)
+		)
+		(property "Description" "Unpolarized capacitor"
+			(at 73.66 77.47 0)
+			(effects
+				(font
+					(size 1.27 1.27)
+				)
+				(hide yes)
+			)
+		)
+		(property "LCSC" "C15195"
+			(at 73.66 77.47 0)
+			(effects
+				(font
+					(size 1.27 1.27)
+				)
+				(hide yes)
+			)
+		)
+		(pin "2"
+		)
+		(pin "1"
+		)
+		(instances
+			(project "why2025"
+				(path "/6a31734e-65de-48f3-8156-2b24b665b183/f71ac64f-0729-4b77-85b6-53947ac74ff8"
+					(reference "C46")
+					(unit 1)
+				)
+			)
+		)
+	)
+	(symbol
+		(lib_id "Device:C")
+		(at 62.23 77.47 0)
+		(unit 1)
+		(exclude_from_sim no)
+		(in_bom yes)
+		(on_board yes)
+		(dnp no)
+		(fields_autoplaced yes)
+		(property "Reference" "C26"
+			(at 66.04 76.1999 0)
+			(effects
+				(font
+					(size 1.27 1.27)
+				)
+				(justify left)
+			)
+		)
+		(property "Value" "10n"
+			(at 66.04 78.7399 0)
+			(effects
+				(font
+					(size 1.27 1.27)
+				)
+				(justify left)
+			)
+		)
+		(property "Footprint" "Capacitor_SMD:C_0402_1005Metric"
+			(at 63.1952 81.28 0)
+			(effects
+				(font
+					(size 1.27 1.27)
+				)
+				(hide yes)
+			)
+		)
+		(property "Datasheet" "https://wmsc.lcsc.com/wmsc/upload/file/pdf/v2/lcsc/2304140030_Samsung-Electro-Mechanics-CL05B103KB5NNNC_C15195.pdf"
+			(at 62.23 77.47 0)
+			(effects
+				(font
+					(size 1.27 1.27)
+				)
+				(hide yes)
+			)
+		)
+		(property "Description" "Unpolarized capacitor"
+			(at 62.23 77.47 0)
+			(effects
+				(font
+					(size 1.27 1.27)
+				)
+				(hide yes)
+			)
+		)
+		(property "LCSC" "C15195"
+			(at 62.23 77.47 0)
+			(effects
+				(font
+					(size 1.27 1.27)
+				)
+				(hide yes)
+			)
+		)
+		(pin "2"
+		)
+		(pin "1"
+		)
+		(instances
+			(project "why2025"
+				(path "/6a31734e-65de-48f3-8156-2b24b665b183/f71ac64f-0729-4b77-85b6-53947ac74ff8"
+					(reference "C26")
+					(unit 1)
+				)
+			)
 		)
 	)
@@
 			)
 		)
-		(property "Datasheet" ""
+		(property "Datasheet" "https://www.lcsc.com/datasheet/lcsc_datasheet_2304282030_HRS-Hirose-DF37NB-24DS-0-4V-51_C3036280.pdf"
 			(at 143.51 92.71 0)
 			(effects
