File: display.kicad_sch (KiCad schematic)
At the start: 7 parts, among them CN1 DF37NB-24DS-0.4V(51)

Commit message: Small fixes
Parts:
- CN1: LCSC (none) -> C3036280
Changed lines of the file:
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@@
 	(title_block
 		(title "WHY2025 badge")
-		(date "2024-08-23")
+		(date "2024-08-24")
 		(rev "Prototype 2")
 		(company "Badge.Team")
@@
 			(effects
 				(font
+					(size 1.27 1.27)
+				)
+				(hide yes)
+			)
+		)
+		(property "LCSC" "C3036280"
+			(at 143.51 92.71 0)
+			(effects
+				(font

Commit message: Change TE resistor to 100k pull-down and export production files
Parts:
- CN1: LCSC Part C3036280 -> (none)
- R98: value 10k -> 100k; LCSC C60490 -> C25741
Connections:
- net +3.3V: no longer R98.2
- net GND: now also R98.2
Other:
- moved on the sheet: R98
