File: keyboard_matrix.kicad_sch (KiCad schematic)
At the start: 85 parts

Commit message: Relabeling of ESP32-C6 GPIO, route signals to expansion header for testing
Parts:
- added D77, D78, D79, D80, D81: LED, badgeteam:LTW-010DCG-SR-G, symbol Device:LED
Connections:
- net at D75.1 (K): now also D74.2 (A)
- net at D75.2 (A): now also D76.1 (K)
- net at D73.1 (K): now also D81.1 (K)
- net at D73.2 (A): now also D74.1 (K)
- net at D76.2 (A): now also D77.2 (A)
- new net: D80.1 (K), D81.2 (A)
- new net: D79.1 (K), D80.2 (A)
- new net: D77.1 (K), D78.2 (A)
- new net: D78.1 (K), D79.2 (A)
Other:
- moved on the sheet: D1, D10, D11, D12, D13, D14, D15, D16, D17, D18, D19, D2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

Commit message: More fixes, add display, update display backlight driver circuit, fix some of the footprint associations
Parts:
- removed D79: LED, badgeteam:LTW-010DCG-SR-G, symbol Device:LED
Connections:
- net -BL-KB: now reaches D73.1 (K), D81.1 (K)
- net at D80.2 (A): now also D78.1 (K)
- net +BL-KB: now reaches D76.2 (A), D77.2 (A)
- net EXT renamed EXT_I
- net ROW8 renamed EXT_O
- no-connect marks 1 -> 0
Other:
- moved on the sheet: D73, D74, D75, D76, D77, D78, D80, D81

Commit message: Bill of materials part 1
Parts:
- D1, D10, D11, D12, D13, D14, D15, D16, D17, D18, D19, D2, D20, D21, D22, D23, D24, D25, D26, D27, D28, D29, D3, D30, D31, D32, D33, D34, D35, D36, D37, D38, D39, D4, D40, D41, D42, D43, D44, D45, D46, D47, D48, D49, D5, D50, D51, D52, D53, D54, D55, D56, D57, D58, D59, D6, D60, D61, D62, D63, D64, D65, D66, D67, D68, D69, D7, D70, D71, D72, D8, D9: value LL4148 -> 1N4148WS; LCSC C2891733 -> C2843305
- D73, D74, D75, D76, D77, D78, D80, D81: value LED -> LTW-010DCG-SR-G; LCSC (none) -> C5175311
- U2: value ~ -> Keyboard; LCSC (none) -> -
