File: keyboard_matrix.kicad_sch (KiCad schematic)
At the start: 89 parts, among them U2 Keyboard

Commit message: Small tweaks and fixes, update LCSC numbers on some components, change to new key type for power key
Parts:
- added Q2: AP2302B, Package_TO_SOT_SMD:SOT-23, symbol symbols:Q_NMOS_GSD
- added R100: 4k7, Resistor_SMD:R_0402_1005Metric, symbol Device:R
- added R101: 100k, Resistor_SMD:R_0402_1005Metric, symbol symbols:R
Connections:
- net GND: now also R101.1
- net EXT_I: no longer names the net of D48.2 (A)
- net EXT_I: now also Q2.2 (S)
- net EXT_O renamed ROW8
- net ROW8: now also Q2.3 (D)
- new net: Q2.1 (G), R100.2
- new net EXT: R100.1, R101.2
Other:
- note removed: "Extra button can be connected between ROW8 and EXT"

Commit message: More fabrication stuff for prototype 1
Parts:
- U2: now left out of the parts list
Changed lines of the file:
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@@
 		(unit 1)
 		(exclude_from_sim no)
-		(in_bom yes)
+		(in_bom no)
 		(on_board yes)
 		(dnp no)
