File: keyboard_matrix.kicad_sch (KiCad schematic)
At the start: 92 parts, among them Q2 AP2302B, U2 Keyboard

Commit message: Change TE resistor to 100k pull-down and export production files
Parts:
- D73, D74, D75, D76, D77, D78, D80, D81: LCSC C5175311 -> C5175309
Other:
- moved on the sheet: D73, D74, D75, D76
