File: leds.kicad_sch (KiCad schematic)
At the start: 0 parts

Commit message: More work on the schematic, add protection circuit, fix display pinout
Parts:
- added U17, U18, U19: SK6805, leds:SK6805-EC20, symbol button_matrix:SK6805-EC20
- added U20: 74LVC1G125, Package_TO_SOT_SMD:SOT-353_SC-70-5, symbol 74xGxx:74LVC1G125
Connections:
- new net: U17.2 (DOUT), U18.4 (DIN)
- new net: U17.4 (DIN), U20.4
- new net: U18.2 (DOUT), U19.4 (DIN)
- new net DIN: U20.2
- new net DOUT: U19.2 (DOUT)
- new net GND: U17.3 (VSS), U18.3 (VSS), U19.3 (VSS), U20.1, U20.3 (GND)
- new net VLED: U17.1 (VDD), U18.1 (VDD), U19.1 (VDD), U20.5 (VCC)
Other:
- note added: "To-do The idea is to have these LEDs act as status indicators, behind symbols cut out of the frontpanel PCB The exact amount is to be discussed, for now I've added 3."
- company: (none) -> Badge.Team
- title: (none) -> WHY2025 badge

Commit message: Assign footprints, create P4 footprint
Parts:
- U17, U18, U19: footprint leds:SK6805-EC20 -> library:SK6805-EC20

Commit message: Bill of materials part 1
Parts:
- U20: Link https://www.lcsc.com/product-detail/Buffer-Driver-Transceiv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 -> (none)
