File: leds.kicad_sch (KiCad schematic)
At the start: 4 parts, among them U17 SK6805, U18 SK6805, U19 SK6805, U20 74LVC1G125

Commit message: Some more component placement
Parts:
- added U22, U9: SK6805, library:SK6805-EC20, symbol button_matrix:SK6805-EC20
Connections:
- net DOUT: now also U22.2 (DOUT); no longer U19.2 (DOUT)
- net GND: now also U22.3 (VSS), U9.3 (VSS)
- net VLED: now also U22.1 (VDD), U9.1 (VDD)
- new net: U22.4 (DIN), U9.2 (DOUT)
- new net: U19.2 (DOUT), U9.4 (DIN)

Commit message: More routing, small fixes in schematic
Connections:
- net VLED renamed VOTG

Commit message: Remove some items from BOM, generate fabrication files
Other:
- note removed: "To-do The idea is to have these LEDs act as status indicators, behind symbols cut out of the frontpanel PCB The exact amount is to be discussed, for now I've added 3."
Changed lines of the file:
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@@
-		)
-	)
-	(text "To-do\n\nThe idea is to have these LEDs act as status indicators, behind symbols cut out of the frontpanel PCB\nThe exact amount is to be discussed, for now I've added 3."
-		(exclude_from_sim no)
-		(at 143.51 114.046 0)
-		(effects
-			(font
-				(size 1.27 1.27)
-			)
 		)
 	)

Commit message: Add LEDs for artwork
Parts:
- removed U22, U9: SK6805, library:SK6805-EC20, symbol button_matrix:SK6805-EC20
- added U23, U24, U25, U26, U27, U28: SK6805, library:SK6805-EC20, symbol button_matrix:SK6805-EC20
Connections:
- net DOUT: now also U28.2 (DOUT)
- net GND: now also U23.3 (VSS), U24.3 (VSS), U25.3 (VSS), U26.3 (VSS), U27.3 (VSS), U28.3 (VSS)
- net VOTG: now also U23.1 (VDD), U24.1 (VDD), U25.1 (VDD), U26.1 (VDD), U27.1 (VDD), U28.1 (VDD)
- net at U19.2 (DOUT): now also U23.4 (DIN)
- new net: U23.2 (DOUT), U24.4 (DIN)
- new net: U25.2 (DOUT), U26.4 (DIN)
- new net: U24.2 (DOUT), U25.4 (DIN)
- new net: U26.2 (DOUT), U27.4 (DIN)
- new net: U27.2 (DOUT), U28.4 (DIN)
Other:
- moved on the sheet: U17, U18, U19, U20
