File: leds.kicad_sch (KiCad schematic)
At the start: 9 parts, among them U17 SK6805, U18 SK6805, U19 SK6805, U20 74LVC1G125, U22 SK6805, U24 SY6280AAC, U9 SK6805

Commit message: Small fixes
Parts:
- added C87, C88: 10u, Capacitor_SMD:C_0805_2012Metric, symbol Device:C
Connections:
- net GND: now also C87.2, C88.2
- net VLED: now also C87.1, C88.1
- net VOTG renamed VSYS

Commit message: More fixes, replace the external expansion header with through hole connector
Parts:
- R78, R80: LCSC C25744 -> C60490
Changed lines of the file:
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@@
 			)
 		)
-		(property "Datasheet" "https://datasheet.lcsc.com/lcsc/2110260030_UNI-ROYAL-Uniroyal-Elec-0402WGF1002TCE_C25744.pdf"
-			(at 62.23 156.21 0)
-			(effects
-				(font
-					(size 1.27 1.27)
-				)
-				(hide yes)
-			)
-		)
-		(property "Description" "Generic part"
+		(property "Datasheet" "https://datasheet.lcsc.com/lcsc/2304140030_YAGEO-RC0402FR-0710KL_C60490.pdf"
+			(at 62.23 156.21 0)
+			(effects
+				(font
+					(size 1.27 1.27)
+				)
+				(hide yes)
+			)
+		)
+		(property "Description" ""
 			(at 62.23 156.21 0)
 			(effects
@@
 			)
 		)
-		(property "LCSC" "C25744"
+		(property "LCSC" "C60490"
 			(at 62.23 156.21 0)
 			(effects
@@
 			)
 		)
-		(property "Datasheet" "https://datasheet.lcsc.com/lcsc/2110260030_UNI-ROYAL-Uniroyal-Elec-0402WGF1002TCE_C25744.pdf"
+		(property "Datasheet" "https://datasheet.lcsc.com/lcsc/2304140030_YAGEO-RC0402FR-0710KL_C60490.pdf"
 			(at 85.09 156.21 0)
 			(effects
@@
 			)
 		)
-		(property "Description" "Generic part"
+		(property "Description" ""
 			(at 85.09 156.21 0)
 			(effects
@@
 			)
 		)
-		(property "LCSC" "C25744"
+		(property "LCSC" "C60490"
 			(at 85.09 156.21 0)
 			(effects

Commit message: Connect C6 RX/TX, change exp header pinout
Parts:
- U20: value 74LVC1G125 -> 74LVC1G17GW,125; LCSC C12519 -> C426705
Changed lines of the file:
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@@
 		(dnp no)
 		(property "Reference" "U20"
-			(at 44.196 93.218 0)
+			(at 41.91 82.296 0)
 			(effects
 				(font
@@
 			)
 		)
-		(property "Value" "74LVC1G125"
-			(at 46.482 90.678 0)
+		(property "Value" "74LVC1G17GW,125"
+			(at 49.022 84.328 0)
 			(effects
 				(font
@@
 			)
 		)
-		(property "Datasheet" "https://www.ti.com/lit/ds/symlink/sn74lvc1g125.pdf"
+		(property "Datasheet" "https://www.lcsc.com/product-detail/Buffer-Driver-Transceiver_Nexperia-74LVC1G17GW-125_C426705.html"
 			(at 40.64 96.52 0)
 			(effects
@@
 			)
 		)
-		(property "Description" "Single Buffer Gate Tri-State, Low-Voltage CMOS"
+		(property "Description" ""
 			(at 40.64 96.52 0)
 			(effects
@@
 			)
 		)
-		(property "LCSC" "C12519 "
+		(property "LCSC" "C426705"
 			(at 40.64 96.52 0)
 			(effects

Commit message: WIP: change LED, camera, LoRa and C6 pins and add USB-A port 1A current limit
Parts:
- removed C87, C88: 10u, Capacitor_SMD:C_0805_2012Metric, symbol Device:C
- removed R78, R80: 10k, Resistor_SMD:R_0402_1005Metric, symbol mch2021-rescue:R-Device
- removed U24: SY6280AAC, Package_TO_SOT_SMD:SOT-23-5, symbol mch2021-rescue:AAT4610BIGV-1-T1-Power_Management
Connections:
- net VLED renamed VOTG
Other:
- note removed: "Iset = 0.68A = 6800 / 10kOhm"
- note removed: "Switched power: Vin for LEDs"
