File: protection.kicad_sch (KiCad schematic)
At the start: 33 parts, among them U21 LM339

Commit message: Assign footprints, create P4 footprint
Parts:
- R80, R81, R82, R83, R84, R85, R86, R87, R88, R89, R90, R91, R92, R93, R94, R95, R96, R97: footprint (none) -> Resistor_SMD:R_0402_1005Metric

Commit message: Bill of materials part 1
Parts:
- JP2: value EN -> PROT_PSRAM_EN; LCSC (none) -> -
- JP3: value EN -> PROT_MIPI_EN; LCSC (none) -> -
- JP4: value EN -> PROT_FLASH_EN; LCSC (none) -> -
- JP5: value EN -> PROT_HP_EN; LCSC (none) -> -
- R82, R87, R94, R97: LCSC (none) -> C60490
- R84, R85, R95, R96: LCSC (none) -> C25741
- TP3, TP4, TP5, TP6, TP7: LCSC (none) -> -
- U21: LCSC (none) -> C19193841

Commit message: Updated voltage regulator safety
Parts:
- R80: value 30k -> 866
- R83: value 120k -> 4k70
- R84: value 100k -> 3k9
- R85: value 100k -> 4k70
- R88: value 510k -> 7k5
- R90: value 360k -> 2k80
- R91: value 160k -> 1k20
- R93: value 300k -> 4k7
- R94: value 10k -> 4k7
- R95: value 100k -> 3.9k
- R96: value 100k -> 4k7
Connections:
- net at R80.1, R83.2: now also C75.1, U21.8 (-); no longer R82.2
- net at R84.1, R85.2: now also C29.1, U21.10 (-); no longer R87.2
- net at C73.1, R90.1, R91.2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: now also R82.2, R87.2, R94.2, R97.2; no longer U21.10 (-), U21.4 (-), U21.6 (-), U21.8 (-)
- net at R81.2, R82.1, U21.9 (+): no longer C75.1
- net at R92.2, R97.1, U21.5 (+): no longer C74.1
- net at R89.2, R94.1, U21.7 (+): no longer C28.1
- net at R86.2, R87.1, U21.11 (+): no longer C29.1
- net at R95.1, R96.2: now also C74.1, U21.4 (-); no longer R97.2
- net at R88.1, R93.2: now also C28.1, U21.6 (-); no longer R94.2
Other:
- moved on the sheet: C28, C29, C73, C74, C75, JP2, JP3, JP4, JP5, R80, R81, R82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
