File: protection.kicad_sch (KiCad schematic)
At the start: 33 parts, among them U21 LM339

Commit message: Small tweaks and fixes, update LCSC numbers on some components, change to new key type for power key
Parts:
- R80: LCSC (none) -> C423129
- R81, R86, R89, R92: LCSC (none) -> C25790
- R83: value 4k70 -> 4k7; LCSC (none) -> C25900
- R84, R95: LCSC C25741 -> C51721
- R85: value 4k70 -> 4k7; LCSC C25741 -> C25900
- R88: LCSC (none) -> C25918
- R90: value 2k80 -> 2k8; LCSC (none) -> C62741
- R91: value 1k20 -> 1k2; LCSC (none) -> C11702
- R93: LCSC (none) -> C25900
- R94: LCSC C60490 -> C25900
- R96: LCSC C25741 -> C25900
Other:
- moved on the sheet: C28, C29, C73, C74, C75, JP2, JP3, JP4, JP5, R80, R81, R82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

Commit message: Routed more stuff.
Parts:
- removed TP3: PR1, TestPoint:TestPoint_Pad_D1.0mm, symbol Connector:TestPoint
- removed TP4: PR2, TestPoint:TestPoint_Pad_D1.0mm, symbol Connector:TestPoint
- removed TP5: PR3, TestPoint:TestPoint_Pad_D1.0mm, symbol Connector:TestPoint
- removed TP6: PR4, TestPoint:TestPoint_Pad_D1.0mm, symbol Connector:TestPoint

Commit message: All wires routed, lots of DRC errors to go
Changed lines of the file:
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@@
 			)
 		)
-		(property "Description" "1%"
+		(property "Description" ""
 			(at 233.68 73.914 90)
 			(effects
@@
 			)
 		)
-		(property "Description" "1%"
+		(property "Description" ""
 			(at 128.524 102.616 0)
 			(effects
@@
 			)
 		)
-		(property "Description" "1%"
+		(property "Description" ""
 			(at 225.044 102.362 0)
 			(effects
@@
 			)
 		)
-		(property "Description" "1%"
+		(property "Description" ""
 			(at 78.994 102.362 0)
 			(effects
@@
 			)
 		)
-		(property "Description" "1%"
+		(property "Description" ""
 			(at 180.34 74.168 90)
 			(effects
@@
 			)
 		)
-		(property "Description" "1%"
+		(property "Description" ""
 			(at 134.62 74.168 90)
 			(effects
@@
 			)
 		)
-		(property "Description" "1%"
+		(property "Description" ""
 			(at 174.498 102.616 0)
 			(effects
@@
 			)
 		)
-		(property "Description" "1%"
+		(property "Description" ""
 			(at 87.63 74.168 90)
 			(effects

Commit message: Remove some items from BOM, generate fabrication files
Parts:
- TP7: now left out of the parts list
Changed lines of the file:
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@@
 		(unit 1)
 		(exclude_from_sim no)
-		(in_bom yes)
+		(in_bom no)
 		(on_board yes)
 		(dnp no)

Commit message: More fabrication stuff for prototype 1
Parts:
- JP2, JP3, JP4, JP5: now left out of the parts list
- R95: value 3.9k -> 3k9
Changed lines of the file:
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@@
 		(unit 1)
 		(exclude_from_sim yes)
-		(in_bom yes)
+		(in_bom no)
 		(on_board yes)
 		(dnp no)
@@
 			)
 		)
-		(property "Value" "3.9k"
+		(property "Value" "3k9"
 			(at 77.47 87.6299 0)
 			(effects
@@
 			)
 		)
-		(property "Description" ""
+		(property "Description" "1%"
 			(at 128.524 102.616 0)
 			(effects
@@
 		(unit 1)
 		(exclude_from_sim yes)
-		(in_bom yes)
+		(in_bom no)
 		(on_board yes)
 		(dnp no)
@@
 		(unit 1)
 		(exclude_from_sim yes)
-		(in_bom yes)
+		(in_bom no)
 		(on_board yes)
 		(dnp no)
@@
 			)
 		)
-		(property "Description" ""
+		(property "Description" "1%"
 			(at 225.044 102.362 0)
 			(effects
@@
 			)
 		)
-		(property "Description" ""
+		(property "Description" "1%"
 			(at 78.994 102.362 0)
 			(effects
@@
 		(unit 1)
 		(exclude_from_sim yes)
-		(in_bom yes)
+		(in_bom no)
 		(on_board yes)
 		(dnp no)
@@
 			)
 		)
-		(property "Description" ""
+		(property "Description" "1%"
 			(at 174.498 102.616 0)
 			(effects

Commit message: Production version of prototype 1
Parts:
- C28, C29, C74, C75: value 100n -> 10n; LCSC C307331 -> C565544
- U21: value LM339 -> LM339DR
Other:
- moved on the sheet: C73, TP7
Changed lines of the file:
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@@
 	(title_block
 		(title "WHY2025 badge")
-		(date "2024-05-10")
+		(date "2024-05-22")
 		(rev "Prototype 1")
 		(company "Badge.Team")
 		(comment 1 "Copyright 2024 Nicolai Electronics")
 		(comment 2 "License: CERN-OHL-P")
-		(comment 3 "PROTOYPE DESIGN UNTESTED")
+		(comment 3 "Untested prototype design")
 		(comment 4 "(Work in progress!)")
 	)
@@
 	)
 	(junction
-		(at 40.64 92.71)
-		(diameter 0)
-		(color 0 0 0 0)
-	)
-	(junction
 		(at 173.99 66.04)
 		(diameter 0)
@@
 	)
 	(junction
+		(at 64.77 92.71)
+		(diameter 0)
+		(color 0 0 0 0)
+	)
+	(junction
 		(at 93.98 76.2)
 		(diameter 0)
@@
 	(wire
 		(pts
-			(xy 40.64 90.17) (xy 40.64 92.71)
-		)
-		(stroke
-			(width 0)
-			(type default)
-		)
-	)
-	(wire
-		(pts
 			(xy 52.07 95.25) (xy 52.07 92.71)
 		)
@@
 	(wire
 		(pts
-			(xy 52.07 92.71) (xy 40.64 92.71)
-		)
-		(stroke
-			(width 0)
-			(type default)
-		)
-	)
-	(wire
-		(pts
 			(xy 154.94 76.2) (xy 161.29 76.2)
 		)
@@
 	(wire
 		(pts
-			(xy 40.64 92.71) (xy 40.64 95.25)
+			(xy 93.98 102.87) (xy 93.98 110.49)
 		)
 		(stroke
@@
 	(wire
 		(pts
-			(xy 93.98 102.87) (xy 93.98 110.49)
+			(xy 140.97 102.87) (xy 140.97 110.49)
 		)
 		(stroke
@@
 	(wire
 		(pts
-			(xy 140.97 102.87) (xy 140.97 110.49)
+			(xy 93.98 87.63) (xy 96.52 87.63)
 		)
 		(stroke
@@
 	(wire
 		(pts
-			(xy 93.98 87.63) (xy 96.52 87.63)
+			(xy 161.29 90.17) (xy 161.29 100.33)
 		)
 		(stroke
@@
 	(wire
 		(pts
-			(xy 161.29 90.17) (xy 161.29 100.33)
+			(xy 114.3 76.2) (xy 114.3 90.17)
 		)
 		(stroke
@@
 	(wire
 		(pts
-			(xy 114.3 76.2) (xy 114.3 90.17)
+			(xy 124.46 102.87) (xy 124.46 110.49)
 		)
 		(stroke
@@
 	(wire
 		(pts
-			(xy 124.46 102.87) (xy 124.46 110.49)
+			(xy 161.29 76.2) (xy 161.29 90.17)
 		)
 		(stroke
@@
 	(wire
 		(pts
-			(xy 161.29 76.2) (xy 161.29 90.17)
+			(xy 64.77 92.71) (xy 64.77 95.25)
 		)
 		(stroke
@@
 	(wire
 		(pts
-			(xy 40.64 102.87) (xy 40.64 110.49)
+			(xy 64.77 102.87) (xy 64.77 110.49)
 		)
 		(stroke
@@
 	(text "1v ref."
 		(exclude_from_sim no)
-		(at 48.514 87.122 0)
+		(at 64.262 91.694 0)
 		(effects
 			(font
@@
 			)
 		)
-		(property "Value" "LM339"
+		(property "Value" "LM339DR"
 			(at 250.19 82.55 0)
 			(effects
@@
 			)
 		)
-		(property "Datasheet" "https://datasheet.lcsc.com/lcsc/2311161808_IDCHIP-LM339S_C19193841.pdf"
+		(property "Datasheet" "https://www.lcsc.com/product-detail/Comparators_Texas-Instruments-LM339DR_C7948.html"
 			(at 251.46 85.09 0)
 			(effects
@@
 			)
 		)
-		(property "Value" "100n"
+		(property "Value" "10n"
 			(at 138.049 100.203 0)
 			(effects
@@
 			)
 		)
-		(property "Datasheet" "https://datasheet.lcsc.com/lcsc/2304140030_Samsung-Electro-Mechanics-CL05B104KB54PNC_C307331.pdf"
+		(property "Datasheet" "https://www.lcsc.com/product-detail/Multilayer-Ceramic-Capacitors-MLCC-SMD-SMT_PSA-Prosperity-Dielectrics-FN15F103Z500PNG_C565544.html"
 			(at 140.97 99.06 0)
 			(effects
@@
 			)
 		)
-		(property "LCSC" "C307331"
+		(property "LCSC" "C565544"
 			(at 140.97 99.06 0)
 			(effects
@@
 			)
 		)
-		(property "Value" "100n"
+		(property "Value" "10n"
 			(at 91.059 100.203 0)
 			(effects
@@
 			)
 		)
-		(property "Datasheet" "https://datasheet.lcsc.com/lcsc/2304140030_Samsung-Electro-Mechanics-CL05B104KB54PNC_C307331.pdf"
+		(property "Datasheet" "https://www.lcsc.com/product-detail/Multilayer-Ceramic-Capacitors-MLCC-SMD-SMT_PSA-Prosperity-Dielectrics-FN15F103Z500PNG_C565544.html"
 			(at 93.98 99.06 0)
 			(effects
@@
 			)
 		)
-		(property "LCSC" "C307331"
+		(property "LCSC" "C565544"
 			(at 93.98 99.06 0)
 			(effects
@@
 			)
 		)
-		(property "Value" "LM339"
+		(property "Value" "LM339DR"
 			(at 196.85 82.55 0)
 			(effects
@@
 			)
 		)
-		(property "Datasheet" "https://datasheet.lcsc.com/lcsc/2311161808_IDCHIP-LM339S_C19193841.pdf"
+		(property "Datasheet" "https://www.lcsc.com/product-detail/Comparators_Texas-Instruments-LM339DR_C7948.html"
 			(at 198.12 85.09 0)
 			(effects
@@
 			)
 		)
-		(property "Value" "LM339"
+		(property "Value" "LM339DR"
 			(at 27.94 96.5199 0)
 			(effects
@@
 			)
 		)
-		(property "Datasheet" "https://datasheet.lcsc.com/lcsc/2311161808_IDCHIP-LM339S_C19193841.pdf"
+		(property "Datasheet" "https://www.lcsc.com/product-detail/Comparators_Texas-Instruments-LM339DR_C7948.html"
 			(at 30.48 90.17 0)
 			(effects
@@
 			)
 		)
-		(property "Description" ""
+		(property "Description" "1%"
 			(at 233.68 73.914 90)
 			(effects
@@
 	(symbol
 		(lib_id "Connector:TestPoint")
-		(at 40.64 90.17 0)
+		(at 52.07 92.71 90)
 		(unit 1)
 		(exclude_from_sim no)
@@
 		(dnp no)
 		(property "Reference" "TP7"
-			(at 39.37 85.852 0)
+			(at 43.434 91.948 90)
 			(effects
 				(font
@@
 		)
 		(property "Value" "PRR"
-			(at 39.37 88.392 0)
+			(at 43.434 93.98 90)
 			(effects
 				(font
@@
 		)
 		(property "Footprint" "TestPoint:TestPoint_Pad_D1.0mm"
-			(at 45.72 90.17 0)
+			(at 52.07 87.63 0)
 			(effects
 				(font
@@
 		)
 		(property "Datasheet" "-"
-			(at 45.72 90.17 0)
+			(at 52.07 87.63 0)
 			(effects
 				(font
@@
 		)
 		(property "Description" "test point"
-			(at 40.64 90.17 0)
+			(at 52.07 92.71 0)
 			(effects
 				(font
@@
 		)
 		(property "LCSC" "-"
-			(at 40.64 90.17 0)
+			(at 52.07 92.71 0)
 			(effects
 				(font
@@
 			)
 		)
-		(property "Value" "100n"
+		(property "Value" "10n"
 			(at 237.109 100.203 0)
 			(effects
@@
 			)
 		)
-		(property "Datasheet" "https://datasheet.lcsc.com/lcsc/2304140030_Samsung-Electro-Mechanics-CL05B104KB54PNC_C307331.pdf"
+		(property "Datasheet" "https://www.lcsc.com/product-detail/Multilayer-Ceramic-Capacitors-MLCC-SMD-SMT_PSA-Prosperity-Dielectrics-FN15F103Z500PNG_C565544.html"
 			(at 240.03 99.06 0)
 			(effects
@@
 			)
 		)
-		(property "LCSC" "C307331"
+		(property "LCSC" "C565544"
 			(at 240.03 99.06 0)
 			(effects
@@
 			)
 		)
-		(property "Value" "LM339"
+		(property "Value" "LM339DR"
 			(at 104.14 82.55 0)
 			(effects
@@
 			)
 		)
-		(property "Datasheet" "https://datasheet.lcsc.com/lcsc/2311161808_IDCHIP-LM339S_C19193841.pdf"
+		(property "Datasheet" "https://www.lcsc.com/product-detail/Comparators_Texas-Instruments-LM339DR_C7948.html"
 			(at 105.41 85.09 0)
 			(effects
@@
 			)
 		)
-		(property "Value" "100n"
+		(property "Value" "10n"
 			(at 183.769 100.203 0)
 			(effects
@@
 			)
 		)
-		(property "Datasheet" "https://datasheet.lcsc.com/lcsc/2304140030_Samsung-Electro-Mechanics-CL05B104KB54PNC_C307331.pdf"
+		(property "Datasheet" "https://www.lcsc.com/product-detail/Multilayer-Ceramic-Capacitors-MLCC-SMD-SMT_PSA-Prosperity-Dielectrics-FN15F103Z500PNG_C565544.html"
 			(at 186.69 99.06 0)
 			(effects
@@
 			)
 		)
-		(property "LCSC" "C307331"
+		(property "LCSC" "C565544"
 			(at 186.69 99.06 0)
 			(effects
@@
 	(symbol
 		(lib_id "power:GND")
-		(at 40.64 110.49 0)
+		(at 64.77 110.49 0)
 		(unit 1)
 		(exclude_from_sim no)
@@
 		(fields_autoplaced yes)
 		(property "Reference" "#PWR0257"
-			(at 40.64 116.84 0)
+			(at 64.77 116.84 0)
 			(effects
 				(font
@@
 		)
 		(property "Value" "GND"
-			(at 40.64 115.57 0)
+			(at 64.77 115.57 0)
 			(effects
 				(font
@@
 		)
 		(property "Footprint" ""
-			(at 40.64 110.49 0)
+			(at 64.77 110.49 0)
 			(effects
 				(font
@@
 		)
 		(property "Datasheet" ""
-			(at 40.64 110.49 0)
+			(at 64.77 110.49 0)
 			(effects
 				(font
@@
 		)
 		(property "Description" ""
-			(at 40.64 110.49 0)
+			(at 64.77 110.49 0)
 			(effects
 				(font
@@
 			)
 		)
-		(property "Value" "LM339"
+		(property "Value" "LM339DR"
 			(at 151.13 82.55 0)
 			(effects
@@
 			)
 		)
-		(property "Datasheet" "https://datasheet.lcsc.com/lcsc/2311161808_IDCHIP-LM339S_C19193841.pdf"
+		(property "Datasheet" "https://www.lcsc.com/product-detail/Comparators_Texas-Instruments-LM339DR_C7948.html"
 			(at 152.4 85.09 0)
 			(effects
@@
 	(symbol
 		(lib_id "symbols:C")
-		(at 40.64 99.06 0)
+		(at 64.77 99.06 0)
 		(unit 1)
 		(exclude_from_sim no)
@@
 		(dnp no)
 		(property "Reference" "C73"
-			(at 43.561 97.8916 0)
+			(at 67.691 97.8916 0)
 			(effects
 				(font
@@
 		)
 		(property "Value" "100n"
-			(at 43.561 100.203 0)
+			(at 67.691 100.203 0)
 			(effects
 				(font
@@
 		)
 		(property "Footprint" "Capacitor_SMD:C_0402_1005Metric"
-			(at 41.6052 102.87 0)
+			(at 65.7352 102.87 0)
 			(effects
 				(font
@@
 		)
 		(property "Datasheet" "https://datasheet.lcsc.com/lcsc/2304140030_Samsung-Electro-Mechanics-CL05B104KB54PNC_C307331.pdf"
-			(at 40.64 99.06 0)
+			(at 64.77 99.06 0)
 			(effects
 				(font
@@
 		)
 		(property "Description" ""
-			(at 40.64 99.06 0)
+			(at 64.77 99.06 0)
 			(effects
 				(font
@@
 		)
 		(property "LCSC" "C307331"
-			(at 40.64 99.06 0)
+			(at 64.77 99.06 0)
 			(effects
 				(font
@@
 			)
 		)
-		(property "Description" ""
+		(property "Description" "1%"
 			(at 180.34 74.168 90)
 			(effects
@@
 			)
 		)
-		(property "Description" ""
+		(property "Description" "1%"
 			(at 134.62 74.168 90)
 			(effects

Commit message: Replaced voltage comparitor circuit with zener setup. Also changed couple of 0.2mm vias to 0.3
Parts:
- removed C28, C29, C74, C75: 10n, Capacitor_SMD:C_0402_1005Metric, symbol symbols:C
- removed C73: 100n, Capacitor_SMD:C_0402_1005Metric, symbol symbols:C
- removed JP2: PROT_PSRAM_EN, Jumper:SolderJumper-2_P1.3mm_Open_RoundedPad1.0x1.5mm, symbol Jumper:Jumper_2_Open
- removed JP3: PROT_MIPI_EN, Jumper:SolderJumper-2_P1.3mm_Open_RoundedPad1.0x1.5mm, symbol Jumper:Jumper_2_Open
- removed JP4: PROT_FLASH_EN, Jumper:SolderJumper-2_P1.3mm_Open_RoundedPad1.0x1.5mm, symbol Jumper:Jumper_2_Open
- removed JP5: PROT_HP_EN, Jumper:SolderJumper-2_P1.3mm_Open_RoundedPad1.0x1.5mm, symbol Jumper:Jumper_2_Open
- removed R80: 866, Resistor_SMD:R_0402_1005Metric, symbol Device:R
- removed R81, R86, R89, R92: 470k, Resistor_SMD:R_0402_1005Metric, symbol Device:R
- removed R82, R87, R97: 10k, Resistor_SMD:R_0402_1005Metric, symbol Device:R
- removed R83, R85, R93, R94, R96: 4k7, Resistor_SMD:R_0402_1005Metric, symbol Device:R
- removed R84, R95: 3k9, Resistor_SMD:R_0402_1005Metric, symbol Device:R
- removed R88: 7k5, Resistor_SMD:R_0402_1005Metric, symbol Device:R
- removed R90: 2k8, Resistor_SMD:R_0402_1005Metric, symbol Device:R
- removed R91: 1k2, Resistor_SMD:R_0402_1005Metric, symbol Device:R
- removed TP7: PRR, TestPoint:TestPoint_Pad_D1.0mm, symbol Connector:TestPoint
- removed U21: LM339DR, Package_SO:SOIC-14_3.9x8.7mm_P1.27mm, symbol Comparator:LM339
- added D79, D85: D_Zener, Diode_SMD:D_SOD-123, symbol Device:D_Zener
- added D86: D_Zener, Diode_SMD:D_SOD-323F, symbol Device:D_Zener
- added JP2, JP3, JP4: Jumper_2_Bridged, Jumper:SolderJumper-2_P1.3mm_Bridged_RoundedPad1.0x1.5mm, symbol Jumper:Jumper_2_Bridged
Connections:
- net GND: now also D79.2 (A), D85.2 (A), D86.2 (A)
- net VFLASH: now also JP4.2 (B)
- net VMIPI: now also JP3.2 (B)
- net VPSRAM: now also JP2.2 (B)
- new net: D79.1 (K), JP2.1 (A)
- new net: D85.1 (K), JP4.1 (A)
- new net: D86.1 (K), JP3.1 (A)
Other:
- note removed: "1v ref."

Commit message: Move protection diode for VFLASH, solve DRC errors, clean up
Parts:
- removed JP4: Jumper_2_Bridged, Jumper:SolderJumper-2_P1.3mm_Bridged_RoundedPad1.0x1.5mm, symbol Jumper:Jumper_2_Bridged
Connections:
- net VFLASH: now also D85.1 (K)
Changed lines of the file:
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@@
 	(wire
 		(pts
-			(xy 74.93 43.18) (xy 74.93 50.8)
+			(xy 74.93 27.94) (xy 74.93 50.8)
 		)
 		(stroke
@@
 		(pts
 			(xy 30.48 43.18) (xy 30.48 50.8)
-		)
-		(stroke
-			(width 0)
-			(type default)
-		)
-	)
-	(wire
-		(pts
-			(xy 74.93 27.94) (xy 74.93 33.02)
 		)
 		(stroke
@@
 					(unit 1)
 				)
-			)
-		)
-	)
-	(symbol
-		(lib_id "Jumper:Jumper_2_Bridged")
-		(at 74.93 38.1 90)
-		(unit 1)
-		(exclude_from_sim yes)
-		(in_bom yes)
-		(on_board yes)
-		(dnp no)
-		(fields_autoplaced yes)
-		(property "Reference" "JP4"
-			(at 76.2 36.8299 90)
-			(effects
-				(font
-					(size 1.27 1.27)
-				)
-				(justify right)
-			)
-		)
-		(property "Value" "Jumper_2_Bridged"
-			(at 76.2 39.3699 90)
-			(effects
-				(font
-					(size 1.27 1.27)
-				)
-				(justify right)
-			)
-		)
-		(property "Footprint" "Jumper:SolderJumper-2_P1.3mm_Bridged_RoundedPad1.0x1.5mm"
-			(at 74.93 38.1 0)
-			(effects
-				(font
-					(size 1.27 1.27)
-				)
-				(hide yes)
-			)
-		)
-		(property "Datasheet" "~"
-			(at 74.93 38.1 0)
-			(effects
-				(font
-					(size 1.27 1.27)
-				)
-				(hide yes)
-			)
-		)
-		(property "Description" "Jumper, 2-pole, closed/bridged"
-			(at 74.93 38.1 0)
-			(effects
-				(font
-					(size 1.27 1.27)
-				)
-				(hide yes)
-			)
-		)
-		(pin "1"
-		)
-		(pin "2"
-		)
-		(instances
-			(project "why2025"
-				(path "/6a31734e-65de-48f3-8156-2b24b665b183/3d60835a-4261-467a-b239-9fb76f6e13a1/ff07b197-d1d2-4b00-87d3-a97f534a0288"
-					(reference "JP4")
-					(unit 1)
-				)
