File: protection.kicad_sch (KiCad schematic)
At the start: 5 parts

Commit message: Add the missing LCSC number to the Zener, add comment VESPHP is not related with a Zener.
Parts:
- D86: LCSC (none) -> C550976
Other:
- note added: "Not protected at the moment, if protection is needed, a Zener will not work. The current capacity of the rail is too high, and zener diodes don't come at ~1V"
Changed lines of the file:
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@@
 		)
 	)
-	(text_box "The protection for the software programmable LDO outputs of the ESP32P4. \nWe want to limit the LDO voltages to U_nom +0.3V. If that occurs, the ESP32P4 ~{RESET} signal\nwill become low.\n\nThis circuit uses a LM339 quad comparator with a reference voltage of 1.0 V. The circuit uses a\nthreshold at +0.2V above nominal. They are configured as an inverting comparator with hysteresis.\nThe LM339 has open collector outputs, so we can combine them.\n"
-		(exclude_from_sim no)
-		(at 31.115 168.275 0)
-		(size 100.33 15.24)
-		(stroke
-			(width 0)
-			(type default)
-		)
-		(fill
-			(type none)
-		)
+	(text "Not protected at the moment, if protection is needed, a Zener will not work.\nThe current capacity of the rail is too high, and zener diodes don't come at ~1V"
+		(exclude_from_sim no)
+		(at 141.478 39.116 0)
 		(effects
 			(font
 				(size 1.27 1.27)
 			)
-			(justify left top)
 		)
 	)
@@
 			)
 		)
-		(property "Field6" ""
-			(at 30.48 54.61 90)
-			(effects
-				(font
-					(size 1.27 1.27)
-				)
-				(hide yes)
-			)
-		)
 		(pin "2"
 		)
@@
 			(effects
 				(font
+					(size 1.27 1.27)
+				)
+				(hide yes)
+			)
+		)
+		(property "LCSC" "C550976"
+			(at 53.34 54.61 90)
+			(effects
+				(font

Commit message: Add protection for overvoltage vcore, via Opamp that pulls enable low on regulator when vcore > 1.2V
Parts:
- added C29: 100n, Capacitor_SMD:C_0402_1005Metric, symbol symbols:C
- added JP1, JP4: Jumper_2_Bridged, Jumper:SolderJumper-2_P1.3mm_Bridged_RoundedPad1.0x1.5mm, symbol Jumper:Jumper_2_Bridged
- added R14, R60: 4k7, Resistor_SMD:R_0402_1005Metric, symbol Device:R
- added R61: 499k, Resistor_SMD:R_0402_1005Metric, symbol Device:R
- added U21: LM385DBZ-1.2RG, Package_TO_SOT_SMD:SOT-23-3, symbol lcsc:LM385BZ-1.2
- added U24: LMV321IDBVRG, lcsc:SOT-23-5_L2.9-W1.6-P0.95-LS2.8-BR, symbol lcsc:LMV321IDBVRG
Connections:
- net GND: now also C29.1, U21.2 (A), U24.2 (VSS)
- net VESPHP: now also R60.2
- net VFLASH: now also JP1.2 (B); no longer D85.1 (K)
- new net: D85.1 (K), JP1.1 (A)
- new net: JP4.1 (A), R61.1, U24.4 (OUT)
- new net: R14.1, U21.1 (K), U24.3 (IN-)
- new net: C29.2, R60.1, U24.1 (IN+)
- new net +3.3V: R14.2, R61.2, U24.5 (VDD)
- new net EN_DCDC: JP4.2 (B)
- no-connect marks 0 -> 1
Other:
- note added: "1.2V reference used to compare VESPHP against. Is it going above? The dcdc enable line is pulled low to disable it"
- note added: "Normal: 1.0v Limit: 1.2v"
- note removed: "Normal: 1.0v Limit: 1.25v"
- note removed: "Not protected at the moment, if protection is needed, a Zener will not work. The current capacity of the rail is too high, and zener diodes don't come at ~1V"
