File: power.kicad_sch (KiCad schematic)
At the start: 51 parts, among them J13 Battery, Q1 AP2302B, SW1 Power, U11 AP3032KTR, U12 AP3032KTR, U15 DS8561-25S3, U6 BQ25895RTW, U7 TLV62595DMQR

Commit message: More fabrication stuff for prototype 1
Parts:
- R19: LCSC (none) -> C25879
- R23: LCSC (none) -> C26980
- SW1: LCSC (none) -> C318992
Changed lines of the file:
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@@
 			)
 		)
-		(property "Datasheet" ""
+		(property "Datasheet" "https://www.lcsc.com/product-detail/Tactile-Switches_XKB-Connection-TC-1101V-C-A-W_C318992.html"
 			(at 60.96 80.01 0)
 			(effects
@@
 			)
 		)
-		(property "Description" "Power switch"
+		(property "Description" "Power button"
 			(at 55.88 80.01 0)
+			(effects
+				(font
+					(size 1.27 1.27)
+				)
+				(hide yes)
+			)
+		)
+		(property "LCSC" "C318992"
+			(at 55.88 80.01 90)
 			(effects
 				(font
@@
 			)
 		)
-		(property "Datasheet" ""
+		(property "Datasheet" "https://www.lcsc.com/product-detail/Chip-Resistor-Surface-Mount_UNI-ROYAL-Uniroyal-Elec-0402WGF4532TCE_C26980.html"
 			(at 190.5 38.1 0)
 			(effects
@@
 		)
 		(property "Description" ""
+			(at 190.5 38.1 0)
+			(effects
+				(font
+					(size 1.27 1.27)
+				)
+				(hide yes)
+			)
+		)
+		(property "LCSC" "C26980"
 			(at 190.5 38.1 0)
 			(effects
@@
 			)
 		)
-		(property "Datasheet" ""
+		(property "Datasheet" "https://www.lcsc.com/product-detail/Chip-Resistor-Surface-Mount_UNI-ROYAL-Uniroyal-Elec-0402WGF2201TCE_C25879.html"
 			(at 20.32 40.64 0)
 			(effects
@@
 			(at 20.32 40.64 0)
 			(effects
+				(font
+					(size 1.27 1.27)
+				)
+				(hide yes)
+			)
+		)
+		(property "LCSC" "C25879"
+			(at 20.32 40.64 0)
+			(effects

Commit message: Production version of prototype 1
Parts:
- U15: value DS8561-25S3 -> LR8341A-M25; footprint Package_TO_SOT_SMD:SOT-23 -> Package_TO_SOT_SMD:SOT-89-3; symbol Regulator_Linear:MCP1700x-250xxTT -> Regulator_Linear:MCP1700x-280xxMB; LCSC C5795630 -> C5205210
Connections:
- net +2.5vsb: now also U15.3 (VO); no longer U15.2 (VO)
- net VBATT: now also U15.2 (VI); no longer U15.3 (VI)
Changed lines of the file:
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@@
 	(title_block
 		(title "WHY2025 badge")
-		(date "2024-05-10")
+		(date "2024-05-22")
 		(rev "Prototype 1")
 		(company "Badge.Team")
 		(comment 1 "Copyright 2024 Nicolai Electronics")
 		(comment 2 "License: CERN-OHL-P")
-		(comment 3 "PROTOYPE DESIGN UNTESTED")
+		(comment 3 "Untested prototype design")
 		(comment 4 "(Work in progress!)")
 	)
@@
 	)
 	(symbol
-		(lib_id "Regulator_Linear:MCP1700x-250xxTT")
+		(lib_id "Regulator_Linear:MCP1700x-280xxMB")
 		(at 259.08 35.56 0)
 		(unit 1)
@@
 			)
 		)
-		(property "Value" "DS8561-25S3"
+		(property "Value" "LR8341A-M25"
 			(at 259.08 32.512 0)
 			(effects
@@
 			)
 		)
-		(property "Footprint" "Package_TO_SOT_SMD:SOT-23"
-			(at 259.08 29.845 0)
+		(property "Footprint" "Package_TO_SOT_SMD:SOT-89-3"
+			(at 259.08 30.48 0)
 			(effects
 				(font
@@
 			)
 		)
-		(property "Datasheet" "https://datasheet.lcsc.com/lcsc/2305121703_DSTECH-DS8561-25S3_C5795630.pdf"
-			(at 259.08 35.56 0)
+		(property "Datasheet" "https://www.lcsc.com/product-detail/Linear-Voltage-Regulators-LDO_LR-LR8341A-M25_C5205210.html"
+			(at 259.08 36.83 0)
 			(effects
 				(font
@@
 			)
 		)
-		(property "Description" "2.5v LDO"
+		(property "Description" ""
 			(at 259.08 35.56 0)
 			(effects
@@
 			)
 		)
-		(property "LCSC" "C5795630"
+		(property "LCSC" "C5205210"
 			(at 259.08 35.56 0)
 			(effects

Commit message: Frontpanel :D
Parts:
- C20, C32, C34, C9: LCSC C107372 -> C5199872
Changed lines of the file:
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@@
 			)
 		)
-		(property "LCSC" "C107372"
+		(property "LCSC" "C5199872"
 			(at 166.37 152.4 0)
 			(effects
@@
 			)
 		)
-		(property "LCSC" "C107372"
+		(property "LCSC" "C5199872"
 			(at 91.44 31.75 0)
 			(effects
@@
 			)
 		)
-		(property "LCSC" "C107372"
+		(property "LCSC" "C5199872"
 			(at 53.34 31.75 0)
 			(effects
@@
 			)
 		)
-		(property "LCSC" "C107372"
+		(property "LCSC" "C5199872"
 			(at 256.54 151.13 0)
 			(effects
