File: power.kicad_sch (KiCad schematic)
At the start: 62 parts, among them J13 Battery, Q1 AP2302B, SW1 Power, U11 AP3032KTR, U12 AP3032KTR, U15 LR8341A-M25, U23 TPS63020DSJR, U25 65K5., U6 BQ25895RTW

Commit message: Last fixes, different coils for backlight dc/dc
Parts:
- L4, L6: footprint Inductor_SMD:L_1008_2520Metric -> library:IND-SMD_L4.0-W4.0; LCSC C2041474 -> C520306
Changed lines of the file:
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@@
 			)
 		)
-		(property "Footprint" "Inductor_SMD:L_1008_2520Metric"
+		(property "Footprint" "library:IND-SMD_L4.0-W4.0"
 			(at 144.78 135.89 0)
 			(effects
@@
 			)
 		)
-		(property "Datasheet" "https://datasheet.lcsc.com/lcsc/2304140030_Murata-Electronics-DFE252012F-6R8M-P2_C2041474.pdf"
+		(property "Datasheet" "https://jlcpcb.com/partdetail/Ceaiya-CR40186R8M/C520306"
 			(at 144.78 135.89 0)
 			(effects
@@
 			)
 		)
-		(property "LCSC" "C2041474"
+		(property "LCSC" "C520306"
 			(at 144.78 135.89 0)
 			(effects
@@
 			)
 		)
-		(property "Footprint" "Inductor_SMD:L_1008_2520Metric"
+		(property "Footprint" "library:IND-SMD_L4.0-W4.0"
 			(at 234.95 134.62 0)
 			(effects
@@
 			)
 		)
-		(property "Datasheet" "https://datasheet.lcsc.com/lcsc/2304140030_Murata-Electronics-DFE252012F-6R8M-P2_C2041474.pdf"
+		(property "Datasheet" "https://jlcpcb.com/partdetail/Ceaiya-CR40186R8M/C520306"
 			(at 234.95 134.62 0)
 			(effects
@@
 			)
 		)
-		(property "LCSC" "C2041474"
+		(property "LCSC" "C520306"
 			(at 234.95 134.62 0)
 			(effects

Commit message: Add extra capacitance to VSYS to decouple the backlight driver more from VSYS.
Parts:
- added C89: 10u, Capacitor_SMD:C_0805_2012Metric, symbol Device:C_Small
Connections:
- net GND: now also C89.2
- net VSYS: now also C89.1
Other:
- moved on the sheet: R27, TP2
Changed lines of the file:
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@@
 	)
 	(junction
-		(at 118.11 146.05)
-		(diameter 0)
-		(color 0 0 0 0)
-	)
-	(junction
 		(at 92.71 67.31)
 		(diameter 0)
@@
 	)
 	(junction
-		(at 113.03 146.05)
+		(at 101.6 146.05)
 		(diameter 1.016)
 		(color 0 0 0 0)
@@
 	)
 	(junction
+		(at 128.27 154.94)
+		(diameter 0)
+		(color 0 0 0 0)
+	)
+	(junction
 		(at 33.02 151.13)
 		(diameter 0)
@@
 	)
 	(junction
+		(at 106.68 146.05)
+		(diameter 0)
+		(color 0 0 0 0)
+	)
+	(junction
 		(at 256.54 134.62)
 		(diameter 0)
@@
 	(wire
 		(pts
-			(xy 118.11 143.51) (xy 118.11 146.05)
+			(xy 106.68 143.51) (xy 106.68 146.05)
 		)
 		(stroke
@@
 	(wire
 		(pts
-			(xy 113.03 146.05) (xy 107.95 146.05)
+			(xy 101.6 146.05) (xy 96.52 146.05)
 		)
 		(stroke
@@
 	(wire
 		(pts
+			(xy 119.38 135.89) (xy 119.38 149.86)
+		)
+		(stroke
+			(width 0)
+			(type default)
+		)
+	)
+	(wire
+		(pts
 			(xy 128.27 135.89) (xy 128.27 133.35)
 		)
@@
 	(wire
 		(pts
-			(xy 113.03 146.05) (xy 118.11 146.05)
+			(xy 101.6 146.05) (xy 106.68 146.05)
 		)
 		(stroke
@@
 	(wire
 		(pts
+			(xy 119.38 154.94) (xy 128.27 154.94)
+		)
+		(stroke
+			(width 0)
+			(type solid)
+		)
+	)
+	(wire
+		(pts
 			(xy 40.64 73.66) (xy 43.18 73.66)
 		)
@@
 	(wire
 		(pts
-			(xy 113.03 144.78) (xy 113.03 146.05)
+			(xy 101.6 144.78) (xy 101.6 146.05)
 		)
 		(stroke
@@
 	(wire
 		(pts
-			(xy 118.11 146.05) (xy 134.62 146.05)
-		)
-		(stroke
-			(width 0)
-			(type solid)
-		)
-	)
-	(wire
-		(pts
 			(xy 74.93 73.66) (xy 74.93 74.93)
 		)
@@
 	(wire
 		(pts
+			(xy 106.68 146.05) (xy 134.62 146.05)
+		)
+		(stroke
+			(width 0)
+			(type solid)
+		)
+	)
+	(wire
+		(pts
 			(xy 215.9 69.85) (xy 231.14 69.85)
 		)
@@
 	(wire
 		(pts
-			(xy 113.03 133.35) (xy 113.03 137.16)
+			(xy 101.6 133.35) (xy 101.6 137.16)
 		)
 		(stroke
@@
 	(wire
 		(pts
+			(xy 119.38 135.89) (xy 128.27 135.89)
+		)
+		(stroke
+			(width 0)
+			(type default)
+		)
+	)
+	(wire
+		(pts
 			(xy 246.38 134.62) (xy 248.92 134.62)
 		)
@@
 	(text "20mA @ 24v"
 		(exclude_from_sim no)
-		(at 117.348 127.254 0)
+		(at 105.918 127.254 0)
 		(effects
 			(font
@@
 	(hierarchical_label "DISPLAY"
 		(shape input)
-		(at 107.95 146.05 180)
+		(at 96.52 146.05 180)
 		(fields_autoplaced yes)
 		(effects
@@
 	(symbol
 		(lib_id "power:+3.3V")
-		(at 113.03 133.35 0)
+		(at 101.6 133.35 0)
 		(unit 1)
 		(exclude_from_sim no)
@@
 		(dnp no)
 		(property "Reference" "#PWR0125"
-			(at 113.03 137.16 0)
+			(at 101.6 137.16 0)
 			(effects
 				(font
@@
 		)
 		(property "Value" "+3.3V"
-			(at 112.776 129.54 0)
+			(at 101.346 129.54 0)
 			(effects
 				(font
@@
 		)
 		(property "Footprint" ""
-			(at 113.03 133.35 0)
+			(at 101.6 133.35 0)
 			(effects
 				(font
@@
 		)
 		(property "Datasheet" ""
-			(at 113.03 133.35 0)
+			(at 101.6 133.35 0)
 			(effects
 				(font
@@
 		)
 		(property "Description" "Power symbol creates a global label with name \"+3.3V\""
-			(at 113.03 133.35 0)
+			(at 101.6 133.35 0)
 			(effects
 				(font
@@
 	)
 	(symbol
+		(lib_id "Device:C_Small")
+		(at 119.38 152.4 0)
+		(unit 1)
+		(exclude_from_sim no)
+		(in_bom yes)
+		(on_board yes)
+		(dnp no)
+		(property "Reference" "C89"
+			(at 116.586 150.622 0)
+			(effects
+				(font
+					(size 1.27 1.27)
+				)
+				(justify right)
+			)
+		)
+		(property "Value" "10u"
+			(at 112.522 152.654 0)
+			(effects
+				(font
+					(size 1.27 1.27)
+				)
+				(justify left)
+			)
+		)
+		(property "Footprint" "Capacitor_SMD:C_0805_2012Metric"
+			(at 119.38 152.4 0)
+			(effects
+				(font
+					(size 1.27 1.27)
+				)
+				(hide yes)
+			)
+		)
+		(property "Datasheet" "https://www.lcsc.com/product-detail/Multilayer-Ceramic-Capacitors-MLCC-SMD-SMT_Samsung-Electro-Mechanics-CL21B106KAYQNNE_C3039694.html"
+			(at 119.38 152.4 0)
+			(effects
+				(font
+					(size 1.27 1.27)
+				)
+				(hide yes)
+			)
+		)
+		(property "Description" ""
+			(at 119.38 152.4 0)
+			(effects
+				(font
+					(size 1.27 1.27)
+				)
+				(hide yes)
+			)
+		)
+		(property "LCSC" "C3039694"
+			(at 119.38 152.4 0)
+			(effects
+				(font
+					(size 1.27 1.27)
+				)
+				(hide yes)
+			)
+		)
+		(pin "1"
+		)
+		(pin "2"
+		)
+		(instances
+			(project "why2025"
+				(path "/6a31734e-65de-48f3-8156-2b24b665b183/1b21cacd-3ed4-4137-bf19-1f15d3ffa268"
+					(reference "C89")
+					(unit 1)
+				)
+			)
+		)
+	)
+	(symbol
 		(lib_id "power:+3.3V")
 		(at 33.02 147.32 0)
@@
 	(symbol
 		(lib_id "Device:R")
-		(at 113.03 140.97 180)
+		(at 101.6 140.97 180)
 		(unit 1)
 		(exclude_from_sim no)
@@
 		(dnp no)
 		(property "Reference" "R27"
-			(at 110.49 140.97 90)
+			(at 99.06 140.97 90)
 			(effects
 				(font
@@
 		)
 		(property "Value" "100k"
-			(at 115.316 140.97 90)
+			(at 103.886 140.97 90)
 			(effects
 				(font
@@
 		)
 		(property "Footprint" "Resistor_SMD:R_0402_1005Metric"
-			(at 114.808 140.97 90)
+			(at 103.378 140.97 90)
 			(effects
 				(font
@@
 		)
 		(property "Datasheet" "https://datasheet.lcsc.com/lcsc/2110260030_UNI-ROYAL-Uniroyal-Elec-0402WGF1003TCE_C25741.pdf"
-			(at 113.03 140.97 0)
+			(at 101.6 140.97 0)
 			(effects
 				(font
@@
 		)
 		(property "Description" ""
-			(at 113.03 140.97 0)
+			(at 101.6 140.97 0)
 			(effects
 				(font
@@
 		)
 		(property "LCSC" "C25741"
-			(at 113.03 140.97 0)
+			(at 101.6 140.97 0)
 			(effects
 				(font
@@
 	(symbol
 		(lib_id "Connector:TestPoint")
-		(at 118.11 143.51 0)
+		(at 106.68 143.51 0)
 		(mirror y)
 		(unit 1)
@@
 		(dnp no)
 		(property "Reference" "TP2"
-			(at 119.38 139.7 0)
+			(at 107.95 139.7 0)
 			(effects
 				(font
@@
 		)
 		(property "Value" "BLLC"
-			(at 119.38 142.24 0)
+			(at 107.95 142.24 0)
 			(effects
 				(font
@@
 		)
 		(property "Footprint" "TestPoint:TestPoint_Pad_D1.0mm"
-			(at 113.03 143.51 0)
+			(at 101.6 143.51 0)
 			(effects
 				(font
@@
 		)
 		(property "Datasheet" "-"
-			(at 113.03 143.51 0)
+			(at 101.6 143.51 0)
 			(effects
 				(font
@@
 		)
 		(property "Description" "test point"
-			(at 118.11 143.51 0)
+			(at 106.68 143.51 0)
 			(effects
 				(font
@@
 		)
 		(property "LCSC" "-"
-			(at 118.11 143.51 0)
+			(at 106.68 143.51 0)
 			(effects
 				(font

Commit message: Add schottky diode D87 to make high Aperage OTG conversion more efficient.
Parts:
- added D87: SMD24PL-TP, lcsc:SOD-123_L2.8-W1.8-LS3.7-RD, symbol lcsc:SMD24PL-TP
Connections:
- net VOTG: now also D87.1
- net b2l: now also D87.2
Changed lines of the file:
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@@
 	)
 	(junction
+		(at 95.25 31.75)
+		(diameter 0)
+		(color 0 0 0 0)
+	)
+	(junction
 		(at 246.38 147.32)
 		(diameter 1.016)
@@
 	)
 	(junction
-		(at 59.69 31.75)
+		(at 58.42 31.75)
 		(diameter 0)
 		(color 0 0 0 0)
@@
 	(wire
 		(pts
+			(xy 95.25 22.86) (xy 95.25 31.75)
+		)
+		(stroke
+			(width 0)
+			(type default)
+		)
+	)
+	(wire
+		(pts
 			(xy 106.68 143.51) (xy 106.68 146.05)
 		)
@@
 	(wire
 		(pts
+			(xy 95.25 31.75) (xy 111.76 31.75)
+		)
+		(stroke
+			(width 0)
+			(type default)
+		)
+	)
+	(wire
+		(pts
 			(xy 185.42 44.45) (xy 233.68 44.45)
 		)
@@
 	(wire
 		(pts
+			(xy 82.55 31.75) (xy 95.25 31.75)
+		)
+		(stroke
+			(width 0)
+			(type default)
+		)
+	)
+	(wire
+		(pts
 			(xy 118.11 39.37) (xy 124.46 39.37)
 		)
@@
 	(wire
 		(pts
+			(xy 85.09 22.86) (xy 85.09 36.83)
+		)
+		(stroke
+			(width 0)
+			(type default)
+		)
+	)
+	(wire
+		(pts
 			(xy 254 134.62) (xy 256.54 134.62)
 		)
@@
 	(wire
 		(pts
+			(xy 58.42 31.75) (xy 62.23 31.75)
+		)
+		(stroke
+			(width 0)
+			(type default)
+		)
+	)
+	(wire
+		(pts
 			(xy 269.24 134.62) (xy 269.24 132.08)
 		)
@@
 	(wire
 		(pts
-			(xy 59.69 31.75) (xy 62.23 31.75)
-		)
-		(stroke
-			(width 0)
-			(type default)
-		)
-	)
-	(wire
-		(pts
 			(xy 166.37 146.05) (xy 166.37 135.89)
 		)
@@
 	(wire
 		(pts
-			(xy 57.15 31.75) (xy 59.69 31.75)
+			(xy 57.15 31.75) (xy 58.42 31.75)
 		)
 		(stroke
@@
 	(wire
 		(pts
-			(xy 59.69 29.21) (xy 59.69 31.75)
+			(xy 58.42 29.21) (xy 58.42 31.75)
 		)
 		(stroke
@@
 	(wire
 		(pts
-			(xy 82.55 31.75) (xy 111.76 31.75)
-		)
-		(stroke
-			(width 0)
-			(type default)
-		)
-	)
-	(wire
-		(pts
 			(xy 245.11 142.24) (xy 246.38 142.24)
 		)
@@
 		(on_board yes)
 		(dnp no)
-		(fields_autoplaced yes)
 		(property "Reference" "U6"
-			(at 72.39 24.13 0)
+			(at 90.17 19.05 0)
 			(effects
 				(font
@@
 		)
 		(property "Value" "BQ25895RTW"
-			(at 72.39 26.67 0)
+			(at 72.644 27.686 0)
 			(effects
 				(font
@@
 	)
 	(symbol
+		(lib_id "lcsc:SMD24PL-TP")
+		(at 90.17 22.86 180)
+		(unit 1)
+		(exclude_from_sim no)
+		(in_bom yes)
+		(on_board yes)
+		(dnp no)
+		(fields_autoplaced yes)
+		(property "Reference" "D87"
+			(at 90.425 29.21 0)
+			(effects
+				(font
+					(size 1.27 1.27)
+				)
+			)
+		)
+		(property "Value" "SMD24PL-TP"
+			(at 90.425 26.67 0)
+			(effects
+				(font
+					(size 1.27 1.27)
+				)
+			)
+		)
+		(property "Footprint" "lcsc:SOD-123_L2.8-W1.8-LS3.7-RD"
+			(at 90.17 15.24 0)
+			(effects
+				(font
+					(size 1.27 1.27)
+				)
+				(hide yes)
+			)
+		)
+		(property "Datasheet" "https://lcsc.com/product-detail/Others_Micro-Commercial-Components-MCC-SMD24PL-TP_C151787.html"
+			(at 90.17 12.7 0)
+			(effects
+				(font
+					(size 1.27 1.27)
+				)
+				(hide yes)
+			)
+		)
+		(property "Description" ""
+			(at 90.17 22.86 0)
+			(effects
+				(font
+					(size 1.27 1.27)
+				)
+				(hide yes)
+			)
+		)
+		(property "LCSC Part" "C151787"
+			(at 90.17 10.16 0)
+			(effects
+				(font
+					(size 1.27 1.27)
+				)
+				(hide yes)
+			)
+		)
+		(pin "1"
+		)
+		(pin "2"
+		)
+		(instances
+			(project ""
+				(path "/6a31734e-65de-48f3-8156-2b24b665b183/1b21cacd-3ed4-4137-bf19-1f15d3ffa268"
+					(reference "D87")
+					(unit 1)
+				)
+			)
+		)
+	)
+	(symbol
 		(lib_id "power:GND")
 		(at 92.71 85.09 0)
@@
 	(symbol
 		(lib_id "power:PWR_FLAG")
-		(at 59.69 31.75 180)
+		(at 58.42 31.75 180)
 		(unit 1)
 		(exclude_from_sim no)
@@
 		(fields_autoplaced yes)
 		(property "Reference" "#FLG04"
-			(at 59.69 33.655 0)
+			(at 58.42 33.655 0)
 			(effects
 				(font
@@
 		)
 		(property "Value" "PWR_FLAG"
-			(at 59.69 36.83 0)
+			(at 58.42 36.83 0)
 			(effects
 				(font
@@
 		)
 		(property "Footprint" ""
-			(at 59.69 31.75 0)
+			(at 58.42 31.75 0)
 			(effects
 				(font
@@
 		)
 		(property "Datasheet" "~"
-			(at 59.69 31.75 0)
+			(at 58.42 31.75 0)
 			(effects
 				(font
@@
 		)
 		(property "Description" ""
-			(at 59.69 31.75 0)
+			(at 58.42 31.75 0)
 			(effects
 				(font
@@
 	(symbol
 		(lib_id "power:VBUS")
-		(at 59.69 29.21 0)
+		(at 58.42 29.21 0)
 		(unit 1)
 		(exclude_from_sim no)
@@
 		(dnp no)
 		(property "Reference" "#PWR020"
-			(at 59.69 33.02 0)
+			(at 58.42 33.02 0)
 			(effects
 				(font
@@
 		)
 		(property "Value" "VBUS"
-			(at 59.69 25.4 0)
+			(at 58.42 25.4 0)
 			(effects
 				(font
@@
 		)
 		(property "Footprint" ""
-			(at 59.69 29.21 0)
+			(at 58.42 29.21 0)
 			(effects
 				(font
@@
 		)
 		(property "Datasheet" ""
-			(at 59.69 29.21 0)
+			(at 58.42 29.21 0)
 			(effects
 				(font
@@
 		)
 		(property "Description" "Power symbol creates a global label with name \"VBUS\""
-			(at 59.69 29.21 0)
+			(at 58.42 29.21 0)
 			(effects
 				(font

Commit message: Made more space around the D87, smooth curve LORA antenna.
Parts:
- added TP6: VBAT+, TestPoint:TestPoint_Pad_D1.0mm, symbol Connector:TestPoint
Connections:
- net VBATT: now also TP6.1
Changed lines of the file:
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@@
 	)
 	(junction
+		(at 123.19 49.53)
+		(diameter 0)
+		(color 0 0 0 0)
+	)
+	(junction
 		(at 128.27 154.94)
 		(diameter 0)
@@
 	(wire
 		(pts
-			(xy 115.57 49.53) (xy 128.27 49.53)
+			(xy 115.57 49.53) (xy 123.19 49.53)
 		)
 		(stroke
@@
 	(wire
 		(pts
+			(xy 123.19 49.53) (xy 128.27 49.53)
+		)
+		(stroke
+			(width 0)
+			(type default)
+		)
+	)
+	(wire
+		(pts
 			(xy 224.79 77.47) (xy 224.79 96.52)
 		)
@@
 					(unit 1)
 				)
+			)
+		)
+	)
+	(symbol
+		(lib_id "Connector:TestPoint")
+		(at 123.19 49.53 0)
+		(unit 1)
+		(exclude_from_sim no)
+		(in_bom no)
+		(on_board yes)
+		(dnp no)
+		(property "Reference" "TP6"
+			(at 121.92 45.72 0)
+			(effects
+				(font
+					(size 1.27 1.27)
+				)
+				(justify right)
+			)
+		)
+		(property "Value" "VBAT+"
+			(at 121.92 48.26 0)
+			(effects
+				(font
+					(size 1.27 1.27)
+				)
+				(justify right)
+			)
+		)
+		(property "Footprint" "TestPoint:TestPoint_Pad_D1.0mm"
+			(at 128.27 49.53 0)
+			(effects
+				(font
+					(size 1.27 1.27)
+				)
+				(hide yes)
+			)
+		)
+		(property "Datasheet" "-"
+			(at 128.27 49.53 0)
+			(effects
+				(font
+					(size 1.27 1.27)
+				)
+				(hide yes)
+			)
+		)
+		(property "Description" "test point"
+			(at 123.19 49.53 0)
+			(effects
+				(font
+					(size 1.27 1.27)
+				)
+				(hide yes)
+			)
+		)
+		(property "LCSC" "-"
+			(at 123.19 49.53 0)
+			(effects
+				(font
+					(size 1.27 1.27)
+				)
+				(hide yes)
+			)
+		)
+		(pin "1"
+		)
+		(instances
+			(project "why2025"
+				(path "/6a31734e-65de-48f3-8156-2b24b665b183/1b21cacd-3ed4-4137-bf19-1f15d3ffa268"
+					(reference "TP6")
+					(unit 1)
+				)

Commit message: WIP: change LED, camera, LoRa and C6 pins and add USB-A port 1A current limit
Parts:
- added C87, C88: 10u, Capacitor_SMD:C_0805_2012Metric, symbol Device:C
- added R78: 6.8k, Resistor_SMD:R_0402_1005Metric, symbol mch2021-rescue:R-Device
- added R80: 10k, Resistor_SMD:R_0402_1005Metric, symbol mch2021-rescue:R-Device
- added U24: SY6280AAC, Package_TO_SOT_SMD:SOT-23-5, symbol mch2021-rescue:AAT4610BIGV-1-T1-Power_Management
Connections:
- net GND: now also C87.2, C88.2, R78.2, R80.2, U24.2 (GND)
- net VOTG: now also U24.5 (IN)
- new net: R78.1, U24.3 (SET)
- new net USB_ENABLE: R80.1, U24.4 (ON)
- new net VOTG_OUT: C87.1, C88.1, U24.1 (OUT)
Other:
- note added: "Iset = 1.0A = 6800 / 6.8kOhm"
- note added: "Switched power for USB-A port"
- moved on the sheet: C18, C19, U25
