File: sensors.kicad_sch (KiCad schematic)
At the start: 1 part, among them U10 BHI360

Commit message: Add components to be able to use the bhi360 IC
Parts:
- added C75, C77: 100n, Capacitor_SMD:C_0402_1005Metric, symbol symbols:C
- added C76: 1u, Capacitor_SMD:C_0603_1608Metric, symbol symbols:C
- added C78: 220nF, Capacitor_SMD:C_0603_1608Metric, symbol Device:C_Small
- added R60, R61: 4k7, Resistor_SMD:R_0402_1005Metric, symbol Device:R
- added U21: PCA9517DP,118, lcsc:TSSOP-8_L3.0-W3.0-P0.65-LS4.9-BL, symbol lcsc:PCA9517DP,118
Connections:
- net GND: now also U10.1 (HSDO), C75.2, C76.2, C77.2, C78.2, U21.4 (GND)
- net +1V8: now reaches U10.12 (HCSB)
- net +1V8: now also U10.17 (~{RESET}), U10.5 (VDDIO), U10.8 (VDD), C75.1, C76.1, C77.1, R60.2, R61.2, U21.1 (VCCA)
- net at U10.13 (HSCX): now also R60.1, U21.2 (SCLA)
- net at U10.14 (HSDX): now also R61.1, U21.3 (SDAA)
- net at U10.9 (VREG): now also C78.1
- new net +3.3V: U21.8 (VCCB)
- new net SCL: U21.6 (SDAB)
- new net SDA: U21.7 (SCLB)
- no-connect marks 0 -> 11
Other:
- note added: "interrupt?"

Commit message: Add Bosch sensor, fix small things, add speaker hole etc...
Parts:
- added C86: 100n, Capacitor_SMD:C_0402_1005Metric, symbol mch2021-rescue:C-Device
- added U26: BME680, Package_LGA:Bosch_LGA-8_3x3mm_P0.8mm_ClockwisePinNumbering, symbol mch2021-rescue:BME680-Sensor
- U21: footprint lcsc:TSSOP-8_L3.0-W3.0-P0.65-LS4.9-BL -> library:TSSOP-8_L3.0-W3.0-P0.65-LS4.9-BL
Connections:
- net +3.3V: now also C86.1, U26.2 (CSB), U26.5 (SDO), U26.6 (VDDIO), U26.8 (VDD)
- net GND: now also C86.2, U26.1 (GND), U26.7 (GND)
- net SCL: now also U26.4 (SCK)
- net SDA: now also U26.3 (SDI)
