File: sensors.kicad_sch (KiCad schematic)
At the start: 21 parts, among them U10 BHI360, U21 PCA9517DP,118, U33 BME688_C3664478, U34 BMI270

Commit message: Add pads for connecting to frontpanel
Parts:
- added J11: GND, harwin:Harwin S7091-42R, symbol Connector_Generic:Conn_01x01
- added J14: 3.3v, harwin:Harwin S7091-42R, symbol Connector_Generic:Conn_01x01
- added J15: SDA, harwin:Harwin S7091-42R, symbol Connector_Generic:Conn_01x01
- added J16: SCL, harwin:Harwin S7091-42R, symbol Connector_Generic:Conn_01x01
Connections:
- net +3.3V: now also J14.1 (Pin_1)
- net GND: now also J11.1 (Pin_1)
- net SCL: now also J16.1 (Pin_1)
- net SDA: now also J15.1 (Pin_1)

Commit message: Change TE resistor to 100k pull-down and export production files
Parts:
- C86, C92, C93: Buy early Y -> (none); Category Capacitors -> (none); MPN CL05B104KB54PNC -> (none); Manufacturer Samsung Electro-Mechanics -> (none); Minimal voltage rating 10 -> (none); Mouser - -> (none); Sponsored N -> (none); Voltage rating 50 -> (none)
- J11, J14, J15, J16: LCSC (none) -> -; now left out of the parts list
- U10: MAXIMUM_PACKAGE_HEIGHT 1.00mm -> (none); MF Bosch -> (none); Package VFLGA-20 Bosch -> (none)
- U21: LCSC (none) -> C2652381; LCSC Part C2652381 -> (none)
- U33: LCSC (none) -> C3664478; LCSC Part C3664478 -> (none)

Commit message: fixed SCL SDA swap on PCA9517 chip.
Connections:
- net SCL: now also U21.7 (SCLB); no longer U21.6 (SDAB)
- net SDA: now also U21.6 (SDAB); no longer U21.7 (SCLB)
Changed lines of the file:
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@@
 	(hierarchical_label "SCL"
 		(shape input)
-		(at 33.02 63.5 180)
+		(at 33.02 60.96 180)
 		(fields_autoplaced yes)
 		(effects
@@
 	(hierarchical_label "SDA"
 		(shape bidirectional)
-		(at 33.02 60.96 180)
+		(at 33.02 63.5 180)
 		(fields_autoplaced yes)
 		(effects
