File: why2025.kicad_sch (KiCad schematic)
At the start: 32 parts, among them J1 USB device, J10 Expansion I3C, J2 USB host, J4 Headphone, J5 External Add-On, J6 Internal Add-On, J7 Speaker, J8 Micro_SD_Card, J9 CAMERA, SW3 Boot, U4 CH334R, Y1 12MHz

Commit message: Small fixes
Parts:
- added N4: Espressif, proto1_kicad:Espressif_Logo, symbol Mechanical:Housing
- Y1: footprint Crystal:Crystal_SMD_3225-4Pin_3.2x2.5mm -> Crystal:Crystal_SMD_2520-4Pin_2.5x2.0mm; LCSC C133337 -> C284156
Connections:
- net Audio/SPK+: now also J7.2 (Pin_2); no longer J7.1 (Pin_1)
- net Audio/SPK-: now also J7.1 (Pin_1); no longer J7.2 (Pin_2)
Other:
- moved on the sheet: N3
Changed lines of the file:
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@@
 	)
 	(symbol
+		(lib_id "Mechanical:Housing")
+		(at 105.41 190.5 0)
+		(unit 1)
+		(exclude_from_sim no)
+		(in_bom no)
+		(on_board yes)
+		(dnp no)
+		(fields_autoplaced yes)
+		(property "Reference" "N4"
+			(at 109.22 189.5474 0)
+			(effects
+				(font
+					(size 1.27 1.27)
+				)
+				(justify left)
+			)
+		)
+		(property "Value" "Espressif"
+			(at 109.22 192.0874 0)
+			(effects
+				(font
+					(size 1.27 1.27)
+				)
+				(justify left)
+			)
+		)
+		(property "Footprint" "proto1_kicad:Espressif_Logo"
+			(at 106.68 189.23 0)
+			(effects
+				(font
+					(size 1.27 1.27)
+				)
+				(hide yes)
+			)
+		)
+		(property "Datasheet" "-"
+			(at 106.68 189.23 0)
+			(effects
+				(font
+					(size 1.27 1.27)
+				)
+				(hide yes)
+			)
+		)
+		(property "Description" "Stamp"
+			(at 105.41 190.5 0)
+			(effects
+				(font
+					(size 1.27 1.27)
+				)
+				(hide yes)
+			)
+		)
+		(property "LCSC" "-"
+			(at 105.41 190.5 0)
+			(effects
+				(font
+					(size 1.27 1.27)
+				)
+				(hide yes)
+			)
+		)
+		(instances
+			(project "why2025"
+				(path "/6a31734e-65de-48f3-8156-2b24b665b183"
+					(reference "N4")
+					(unit 1)
+				)
+			)
+		)
+	)
+	(symbol
 		(lib_id "power:GND")
 		(at 62.23 186.69 0)
@@
 	(symbol
 		(lib_id "Mechanical:Housing")
-		(at 107.95 189.23 0)
+		(at 106.68 180.34 0)
 		(unit 1)
 		(exclude_from_sim no)
@@
 		(fields_autoplaced yes)
 		(property "Reference" "N3"
-			(at 111.76 188.2774 0)
+			(at 110.49 179.3874 0)
 			(effects
 				(font
@@
 		)
 		(property "Value" "Nicolai Electronics"
-			(at 111.76 190.8174 0)
+			(at 110.49 181.9274 0)
 			(effects
 				(font
@@
 		)
 		(property "Footprint" "library:logo_nicolai"
-			(at 109.22 187.96 0)
+			(at 107.95 179.07 0)
 			(effects
 				(font
@@
 		)
 		(property "Datasheet" "-"
-			(at 109.22 187.96 0)
+			(at 107.95 179.07 0)
 			(effects
 				(font
@@
 		)
 		(property "Description" "Stamp"
-			(at 107.95 189.23 0)
+			(at 106.68 180.34 0)
 			(effects
 				(font
@@
 		)
 		(property "LCSC" "-"
-			(at 107.95 189.23 0)
+			(at 106.68 180.34 0)
 			(effects
 				(font
@@
 			)
 		)
-		(property "Footprint" "Crystal:Crystal_SMD_3225-4Pin_3.2x2.5mm"
+		(property "Footprint" "Crystal:Crystal_SMD_2520-4Pin_2.5x2.0mm"
 			(at 74.93 73.66 0)
 			(effects
@@
 			)
 		)
-		(property "Datasheet" "https://datasheet.lcsc.com/lcsc/1811151640_Yajingxin-TAXM12M4RFBCCT2T_C133337.pdf"
+		(property "Datasheet" "https://www.lcsc.com/product-detail/Crystals_Yajingxin-TXM12M0004252LBCEO00T_C284156.html"
 			(at 74.93 73.66 0)
 			(effects
@@
 			)
 		)
-		(property "LCSC" "C133337"
+		(property "LCSC" "C284156"
 			(at 74.93 73.66 0)
 			(effects
@@
 		)
 		(pin "SPK+" output
-			(at 255.27 72.39 0)
+			(at 255.27 74.93 0)
 			(effects
 				(font
@@
 		)
 		(pin "SPK-" output
-			(at 255.27 74.93 0)
+			(at 255.27 72.39 0)
 			(effects
 				(font

Commit message: More SAO
Parts:
- added J11, J12: SAO, Connector_PinSocket_2.54mm:PinSocket_2x03_P2.54mm_Vertical_SMD, symbol Connector_Generic:Conn_02x03_Odd_Even
Connections:
- net +3.3V: now also J5.16 (Pin_16), J11.1 (Pin_1), J12.1 (Pin_1); no longer J5.15 (Pin_15)
- net GND: now also J5.15 (Pin_15), J11.2 (Pin_2), J12.2 (Pin_2); no longer J5.16 (Pin_16)
- net LEDs/ENABLE: now also J5.1 (Pin_1)
- net SAO_IO1: now also J5.12 (Pin_12), J12.5 (Pin_5); no longer J5.11 (Pin_11)
- net SAO_IO2: now also J5.11 (Pin_11), J12.6 (Pin_6); no longer J5.12 (Pin_12)
- net SAO_SCL: now also J5.13 (Pin_13), J11.4 (Pin_4), J12.4 (Pin_4); no longer J5.14 (Pin_14)
- net SAO_SDA: now also J5.14 (Pin_14), J11.3 (Pin_3), J12.3 (Pin_3); no longer J5.13 (Pin_13)
- new net C6_RX: J11.6 (Pin_6)
- new net C6_TX: J11.5 (Pin_5)
Other:
- sheet Radio ports: added RX, TX; removed none

Commit message: Small fixes
Other:
- note added: "M2 holes for expansion boards & case"
- note removed: "Standoff holes for expansion boards & case"
- moved on the sheet: H1, H10, H17, H2, H3, H4, H5, H6, H7, H8, H9, J10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

Commit message: More fixes, replace the external expansion header with through hole connector
Parts:
- removed F1: 2A, Fuse:Fuse_0805_2012Metric, symbol mch2021-rescue:Polyfuse_Small-Device
- J5: footprint library:SAMTEC-SMH-108-02-X-D -> Connector_PinSocket_2.54mm:PinSocket_2x08_P2.54mm_Horizontal
Connections:
- net USB_VBUS is gone; now on net VBUS: J1.A4 (VBUS), J1.A9 (VBUS), J1.B4 (VBUS), J1.B9 (VBUS)
- net +3.3V: now also J5.2 (Pin_2); no longer J5.16 (Pin_16)
- net GND: now also J5.1 (Pin_1), J5.11 (Pin_11), J5.8 (Pin_8); no longer J5.10 (Pin_10), J5.15 (Pin_15), J5.5 (Pin_5)
- net LEDs/ENABLE: now also J5.15 (Pin_15); no longer J5.1 (Pin_1)
- net MTCK: now also J5.16 (Pin_16); no longer J5.2 (Pin_2)
- net MTDI: now also J5.14 (Pin_14); no longer J5.4 (Pin_4)
- net MTDO: now also J5.12 (Pin_12); no longer J5.6 (Pin_6)
- net MTMS: now also J5.10 (Pin_10); no longer J5.8 (Pin_8)
- net SAO_IO1: now also J5.6 (Pin_6); no longer J5.12 (Pin_12)
- net SAO_IO2: now also J5.5 (Pin_5); no longer J5.11 (Pin_11)
- net SAO_IO3: now also J5.7 (Pin_7); no longer J5.9 (Pin_9)
- net SAO_SCL: now also J5.3 (Pin_3); no longer J5.13 (Pin_13)
- net SAO_SDA: now also J5.4 (Pin_4); no longer J5.14 (Pin_14)
- net VOTG: now also J5.13 (Pin_13); no longer J5.3 (Pin_3)
- net VSYS: now also J5.9 (Pin_9); no longer J5.7 (Pin_7)
Changed lines of the file:
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@@
 	(wire
 		(pts
-			(xy 41.91 39.37) (xy 53.34 39.37)
+			(xy 41.91 39.37) (xy 60.96 39.37)
 		)
 		(stroke
@@
 	(wire
 		(pts
-			(xy 60.96 39.37) (xy 58.42 39.37)
-		)
-		(stroke
-			(width 0)
-			(type default)
-		)
-	)
-	(wire
-		(pts
 			(xy 100.33 92.71) (xy 139.7 92.71)
 		)
@@
 			)
 		)
-		(property "Description" "Stamp"
+		(property "Description" ""
 			(at 152.4 190.5 0)
 			(effects
@@
 			)
 		)
-		(property "Description" "Stamp"
+		(property "Description" ""
 			(at 132.08 190.5 0)
 			(effects
@@
 			)
 		)
-		(property "Description" "Stamp"
+		(property "Description" ""
 			(at 152.4 180.34 0)
 			(effects
@@
 	)
 	(symbol
-		(lib_id "mch2021-rescue:Polyfuse_Small-Device")
-		(at 55.88 39.37 270)
-		(unit 1)
-		(exclude_from_sim no)
-		(in_bom yes)
-		(on_board yes)
-		(dnp no)
-		(property "Reference" "F1"
-			(at 55.88 37.084 90)
-			(effects
-				(font
-					(size 1.27 1.27)
-				)
-			)
-		)
-		(property "Value" "2A"
-			(at 55.88 41.656 90)
-			(effects
-				(font
-					(size 1.27 1.27)
-				)
-			)
-		)
-		(property "Footprint" "Fuse:Fuse_0805_2012Metric"
-			(at 50.8 40.64 0)
-			(effects
-				(font
-					(size 1.27 1.27)
-				)
-				(justify left)
-				(hide yes)
-			)
-		)
-		(property "Datasheet" "https://datasheet.lcsc.com/lcsc/2304140030_TECHFUSE-SL0805200_C70158.pdf"
-			(at 55.88 39.37 0)
-			(effects
-				(font
-					(size 1.27 1.27)
-				)
-				(hide yes)
-			)
-		)
-		(property "Description" "SL0805200"
-			(at 55.88 39.37 0)
-			(effects
-				(font
-					(size 1.27 1.27)
-				)
-				(hide yes)
-			)
-		)
-		(property "LCSC" "C70158"
-			(at 55.88 39.37 90)
-			(effects
-				(font
-					(size 1.27 1.27)
-				)
-				(hide yes)
-			)
-		)
-		(pin "1"
-		)
-		(pin "2"
-		)
-		(instances
-			(project "why2025"
-				(path "/6a31734e-65de-48f3-8156-2b24b665b183"
-					(reference "F1")
-					(unit 1)
-				)
-			)
-		)
-	)
-	(symbol
 		(lib_id "mch2021-rescue:GND-power")
 		(at 19.05 80.01 0)
@@
 	(symbol
 		(lib_id "Connector_Generic:Conn_02x08_Odd_Even")
-		(at 107.95 163.83 0)
+		(at 107.95 166.37 0)
+		(mirror x)
 		(unit 1)
 		(exclude_from_sim no)
@@
 		(on_board yes)
 		(dnp no)
-		(fields_autoplaced yes)
 		(property "Reference" "J5"
-			(at 109.22 149.86 0)
+			(at 109.22 180.34 0)
 			(effects
 				(font
@@
 		)
 		(property "Value" "External Add-On"
-			(at 109.22 152.4 0)
+			(at 109.22 177.8 0)
 			(effects
 				(font
@@
 			)
 		)
-		(property "Footprint" "library:SAMTEC-SMH-108-02-X-D"
-			(at 107.95 163.83 0)
+		(property "Footprint" "Connector_PinSocket_2.54mm:PinSocket_2x08_P2.54mm_Horizontal"
+			(at 107.95 166.37 0)
 			(effects
 				(font
@@
 		)
 		(property "Datasheet" ""
-			(at 107.95 163.83 0)
+			(at 107.95 166.37 0)
 			(effects
 				(font
@@
 			)
 		)
-		(property "Description" "SMH-108-02-G-D"
-			(at 107.95 163.83 0)
+		(property "Description" ""
+			(at 107.95 166.37 0)
 			(effects
 				(font
@@
 		)
 		(property "LCSC" ""
-			(at 107.95 163.83 0)
+			(at 107.95 166.37 0)
 			(effects
 				(font
@@
 			)
 		)
-		(property "Description" "Board"
+		(property "Description" ""
 			(at 132.08 180.34 0)
 			(effects

Commit message: Add ESD protection to USB ports, remove fuse from USB-C port, small fixes
Parts:
- added U28, U29: USBLC6-2P6, Package_TO_SOT_SMD:SOT-666, symbol Power_Protection:USBLC6-2P6
Connections:
- net Application processor/USB2_N: now also U29.3 (I/O2), U29.4 (I/O2)
- net Application processor/USB2_P: now also U29.1 (I/O1), U29.6 (I/O1)
- net GND: now also U28.2 (GND), U29.2 (GND)
- net USB_DEVICE_N: now also U28.3 (I/O2), U28.4 (I/O2)
- net USB_DEVICE_P: now also U28.1 (I/O1), U28.6 (I/O1)
- net VBUS: now also U28.5 (VBUS)
- net VOTG: now also U29.5 (VBUS)
Other:
- moved on the sheet: J2

Commit message: More ESD protection, design stuff
Parts:
- added N5: OSHW, Symbol:OSHW-Logo2_24.3x20mm_SilkScreen, symbol Mechanical:Housing
- added U30, U31: ESD, library:Diodes_UDFN-10_1.0x2.5mm_P0.5mm, symbol RCLAMP0524P-ES:RCLAMP0524P-ES
- N3: value Nicolai Electronics -> Nicolai
Connections:
- net GND: now also U30.3 (GND), U30.8 (GND), U31.3 (GND), U31.8 (GND)
- net MTCK: now also U31.1 (CHA), U31.10 (CHA)
- net MTDI: now also U31.2 (CHB), U31.9 (CHB)
- net MTDO: now also U31.4 (CHC), U31.7 (CHC)
- net MTMS: now also U31.5 (CHD), U31.6 (CHD)
- net SAO_IO1: now also U30.2 (CHB), U30.9 (CHB)
- net SAO_IO2: now also U30.1 (CHA), U30.10 (CHA)
- net SAO_SCL: now also U30.5 (CHD), U30.6 (CHD)
- net SAO_SDA: now also U30.4 (CHC), U30.7 (CHC)
Other:
- moved on the sheet: J5, N1, N2, N3, N4

Commit message: Add PCB probe/jumper is i2c bus to PMIC, add Ranzbak logo.
Parts:
- added N6: Ranzbak, library:goatse_01, symbol Mechanical:Housing
Changed lines of the file:
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@@
+	)
+	(symbol
+		(lib_id "Mechanical:Housing")
+		(at 97.79 180.34 0)
+		(unit 1)
+		(exclude_from_sim no)
+		(in_bom no)
+		(on_board yes)
+		(dnp no)
+		(fields_autoplaced yes)
+		(property "Reference" "N6"
+			(at 101.6 179.3874 0)
+			(effects
+				(font
+					(size 1.27 1.27)
+				)
+				(justify left)
+			)
+		)
+		(property "Value" "Ranzbak"
+			(at 101.6 181.9274 0)
+			(effects
+				(font
+					(size 1.27 1.27)
+				)
+				(justify left)
+			)
+		)
+		(property "Footprint" "library:goatse_01"
+			(at 99.06 179.07 0)
+			(effects
+				(font
+					(size 1.27 1.27)
+				)
+				(hide yes)
+			)
+		)
+		(property "Datasheet" "-"
+			(at 99.06 179.07 0)
+			(effects
+				(font
+					(size 1.27 1.27)
+				)
+				(hide yes)
+			)
+		)
+		(property "Description" ""
+			(at 97.79 180.34 0)
+			(effects
+				(font
+					(size 1.27 1.27)
+				)
+				(hide yes)
+			)
+		)
+		(property "LCSC" "-"
+			(at 97.79 180.34 0)
+			(effects
+				(font
+					(size 1.27 1.27)
+				)
+				(hide yes)
+			)
+		)
+		(instances
+			(project "why2025"
+				(path "/6a31734e-65de-48f3-8156-2b24b665b183"
+					(reference "N6")
+					(unit 1)
+				)
+			)
+		)
 	)
 	(symbol

Commit message: Fixed some routing, add wireless radiation warning logo.
Parts:
- added N7: Radio-logo, radio-logo:radio-logo, symbol Mechanical:Housing
Changed lines of the file:
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@@
+	)
+	(symbol
+		(lib_id "Mechanical:Housing")
+		(at 97.79 190.5 0)
+		(unit 1)
+		(exclude_from_sim no)
+		(in_bom no)
+		(on_board yes)
+		(dnp no)
+		(fields_autoplaced yes)
+		(property "Reference" "N7"
+			(at 101.6 189.5474 0)
+			(effects
+				(font
+					(size 1.27 1.27)
+				)
+				(justify left)
+			)
+		)
+		(property "Value" "Radio-logo"
+			(at 101.6 192.0874 0)
+			(effects
+				(font
+					(size 1.27 1.27)
+				)
+				(justify left)
+			)
+		)
+		(property "Footprint" "radio-logo:radio-logo"
+			(at 99.06 189.23 0)
+			(effects
+				(font
+					(size 1.27 1.27)
+				)
+				(hide yes)
+			)
+		)
+		(property "Datasheet" "-"
+			(at 99.06 189.23 0)
+			(effects
+				(font
+					(size 1.27 1.27)
+				)
+				(hide yes)
+			)
+		)
+		(property "Description" ""
+			(at 97.79 190.5 0)
+			(effects
+				(font
+					(size 1.27 1.27)
+				)
+				(hide yes)
+			)
+		)
+		(property "LCSC" "-"
+			(at 97.79 190.5 0)
+			(effects
+				(font
+					(size 1.27 1.27)
+				)
+				(hide yes)
+			)
+		)
+		(instances
+			(project "why2025"
+				(path "/6a31734e-65de-48f3-8156-2b24b665b183"
+					(reference "N7")
+					(unit 1)
+				)
+			)
+		)
 	)
 	(symbol
