File: why2025.kicad_sch (KiCad schematic)
At the start: 41 parts, among them J1 USB device, J10 Expansion I3C, J11 SAO, J12 SAO, J2 USB host, J4 Headphone, J5 External Add-On, J6 Internal Add-On, J7 Speaker, J8 Micro_SD_Card, J9 CAMERA, SW3 Boot, U28 USBLC6-2P6, U29 USBLC6-2P6, U30 ESD, U31 ESD, U4 CH334R, Y1 12MHz

Commit message: Make TE a bit bigger, add 3d model of P4, align logos
Parts:
- N5: footprint Symbol:OSHW-Logo2_24.3x20mm_SilkScreen -> Symbol:OSHW-Logo2_14.6x12mm_SilkScreen
Changed lines of the file:
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@@
 			)
 		)
-		(property "Footprint" "Symbol:OSHW-Logo2_24.3x20mm_SilkScreen"
+		(property "Footprint" "Symbol:OSHW-Logo2_14.6x12mm_SilkScreen"
 			(at 161.29 179.07 0)
 			(effects

Commit message: Connect C6 RX/TX, change exp header pinout
Parts:
- removed J11: SAO, Connector_PinSocket_2.54mm:PinSocket_2x03_P2.54mm_Vertical_SMD, symbol Connector_Generic:Conn_02x03_Odd_Even
- added R46: 2k2, Resistor_SMD:R_0402_1005Metric, symbol Device:R
- J5: value External Add-On -> External Add-On (SAO / PMOD); footprint Connector_PinSocket_2.54mm:PinSocket_2x08_P2.54mm_Horizontal -> Connector_PinSocket_2.54mm:PinSocket_2x07_P2.54mm_Horizontal; symbol Connector_Generic:Conn_02x08_Odd_Even -> Connector_Generic:Conn_02x07_Odd_Even; LCSC (none) -> C2936004
Connections:
- net SAO_IO3 is gone; now on net MTMS: J5.7 (Pin_7)
- net +3.3V: now also J5.13 (Pin_13), J5.14 (Pin_14)
- net E12: now also R46.2
- net GND: now also J5.12 (Pin_12); no longer J5.8 (Pin_8)
- net LEDs/ENABLE: no longer J5.15 (Pin_15)
- net MTCK: now also J5.9 (Pin_9); no longer J5.16 (Pin_16)
- net MTDI: now also J5.10 (Pin_10); no longer J5.14 (Pin_14)
- net MTDO: now also J5.8 (Pin_8); no longer J5.12 (Pin_12)
- net MTMS: no longer J5.10 (Pin_10)
- net VOTG: no longer J5.13 (Pin_13)
- net VSYS: no longer J5.9 (Pin_9)
- net CAM_GPIO1: now reaches J9.5 (Pin_5)
- net CAM_GPIO renamed CAM_GPIO0
- new net Radio/TX: R46.1
- no-connect marks 8 -> 7
Other:
- sheet Application processor ports: added CAM_GPIO1; removed SAO_IO3
- note removed: "SAO"

Commit message: Add ESD protection LCSC number
Parts:
- U30, U31: LCSC (none) -> C5180236
Changed lines of the file:
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@@
 			)
 		)
-		(property "Datasheet" ""
+		(property "Datasheet" "https://www.lcsc.com/product-detail/ESD-Protection-Devices_ElecSuper-RCLAMP0524P-ES_C5180236.html"
 			(at 58.42 160.02 0)
 			(effects
@@
 		)
 		(property "Description" ""
+			(at 58.42 160.02 0)
+			(effects
+				(font
+					(size 1.27 1.27)
+				)
+				(hide yes)
+			)
+		)
+		(property "LCSC" "C5180236"
 			(at 58.42 160.02 0)
 			(effects
@@
 			)
 		)
-		(property "Datasheet" ""
+		(property "Datasheet" "https://www.lcsc.com/product-detail/ESD-Protection-Devices_ElecSuper-RCLAMP0524P-ES_C5180236.html"
 			(at 77.47 160.02 0)
 			(effects
@@
 			(at 77.47 160.02 0)
 			(effects
+				(font
+					(size 1.27 1.27)
+				)
+				(hide yes)
+			)
+		)
+		(property "LCSC" "C5180236"
+			(at 77.47 160.02 0)
+			(effects

Commit message: Add Bosch logo, first attempt at creating thermal separation for BME690
Parts:
- added N8: Bosch, proto1_kicad:bosch_logo, symbol Mechanical:Housing
Changed lines of the file:
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@@
+	)
+	(symbol
+		(lib_id "Mechanical:Housing")
+		(at 158.75 190.5 0)
+		(unit 1)
+		(exclude_from_sim no)
+		(in_bom no)
+		(on_board yes)
+		(dnp no)
+		(fields_autoplaced yes)
+		(property "Reference" "N8"
+			(at 162.56 189.5474 0)
+			(effects
+				(font
+					(size 1.27 1.27)
+				)
+				(justify left)
+			)
+		)
+		(property "Value" "Bosch"
+			(at 162.56 192.0874 0)
+			(effects
+				(font
+					(size 1.27 1.27)
+				)
+				(justify left)
+			)
+		)
+		(property "Footprint" "proto1_kicad:bosch_logo"
+			(at 160.02 189.23 0)
+			(effects
+				(font
+					(size 1.27 1.27)
+				)
+				(hide yes)
+			)
+		)
+		(property "Datasheet" "-"
+			(at 160.02 189.23 0)
+			(effects
+				(font
+					(size 1.27 1.27)
+				)
+				(hide yes)
+			)
+		)
+		(property "Description" ""
+			(at 158.75 190.5 0)
+			(effects
+				(font
+					(size 1.27 1.27)
+				)
+				(hide yes)
+			)
+		)
+		(property "LCSC" "-"
+			(at 158.75 190.5 0)
+			(effects
+				(font
+					(size 1.27 1.27)
+				)
+				(hide yes)
+			)
+		)
+		(instances
+			(project "why2025"
+				(path "/6a31734e-65de-48f3-8156-2b24b665b183"
+					(reference "N8")
+					(unit 1)
+				)
+			)
+		)
 	)
 	(symbol

Commit message: Add accelerometer interrupt
Parts:
- added R81: 2k2, Resistor_SMD:R_0402_1005Metric, symbol Device:R
Connections:
- net E11: now also R81.2
- new net Sensors/INT: R81.1
Other:
- sheet Sensors ports: added INT; removed none
Changed lines of the file:
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@@
 	(title_block
 		(title "WHY2025 badge")
-		(date "2024-08-27")
+		(date "2024-09-12")
 		(rev "Prototype 2")
 		(company "Badge.Team")
@@
 	(wire
 		(pts
+			(xy 78.74 119.38) (xy 82.55 119.38)
+		)
+		(stroke
+			(width 0)
+			(type default)
+		)
+	)
+	(wire
+		(pts
 			(xy 223.52 156.21) (xy 226.06 156.21)
 		)
@@
 		)
 	)
+	(global_label "E11"
+		(shape bidirectional)
+		(at 71.12 119.38 180)
+		(fields_autoplaced yes)
+		(effects
+			(font
+				(size 1.016 1.016)
+			)
+			(justify right)
+		)
+		(property "Intersheetrefs" "${INTERSHEET_REFS}"
+			(at 64.9887 119.38 0)
+			(effects
+				(font
+					(size 1.27 1.27)
+				)
+				(justify right)
+				(hide yes)
+			)
+		)
+	)
 	(global_label "E1"
 		(shape bidirectional)
@@
 	)
 	(symbol
+		(lib_id "Device:R")
+		(at 74.93 119.38 270)
+		(unit 1)
+		(exclude_from_sim no)
+		(in_bom yes)
+		(on_board yes)
+		(dnp no)
+		(property "Reference" "R81"
+			(at 79.502 118.11 90)
+			(effects
+				(font
+					(size 1.27 1.27)
+				)
+			)
+		)
+		(property "Value" "2k2"
+			(at 79.502 120.65 90)
+			(effects
+				(font
+					(size 1.27 1.27)
+				)
+			)
+		)
+		(property "Footprint" "Resistor_SMD:R_0402_1005Metric"
+			(at 74.93 117.602 90)
+			(effects
+				(font
+					(size 1.27 1.27)
+				)
+				(hide yes)
+			)
+		)
+		(property "Datasheet" "https://www.lcsc.com/product-detail/Chip-Resistor-Surface-Mount_UNI-ROYAL-Uniroyal-Elec-0402WGF2201TCE_C25879.html"
+			(at 74.93 119.38 0)
+			(effects
+				(font
+					(size 1.27 1.27)
+				)
+				(hide yes)
+			)
+		)
+		(property "Description" ""
+			(at 74.93 119.38 0)
+			(effects
+				(font
+					(size 1.27 1.27)
+				)
+				(hide yes)
+			)
+		)
+		(property "LCSC" "C25879"
+			(at 74.93 119.38 0)
+			(effects
+				(font
+					(size 1.27 1.27)
+				)
+				(hide yes)
+			)
+		)
+		(pin "1"
+		)
+		(pin "2"
+		)
+		(instances
+			(project "why2025"
+				(path "/6a31734e-65de-48f3-8156-2b24b665b183"
+					(reference "R81")
+					(unit 1)
+				)
+			)
+		)
+	)
+	(symbol
 		(lib_id "mch2021-rescue:GND-power")
 		(at 252.73 161.29 270)
@@
 			)
 		)
+		(pin "INT" output
+			(at 82.55 119.38 180)
+			(effects
+				(font
+					(size 1.27 1.27)
+				)
+				(justify left)
+			)
+		)

Commit message: Add 1.5k pull-up to D+ of C6, remove logos, add JTAG connector, fix SAO pinout
Parts:
- removed C7: 1u, Capacitor_SMD:C_0603_1608Metric, symbol mch2021-rescue:C-Device
- removed N2: Stamp, stamp:stamp, symbol Mechanical:Housing
- removed N3: Nicolai, library:logo_nicolai, symbol Mechanical:Housing
- removed N4: Espressif, proto1_kicad:Espressif_Logo, symbol Mechanical:Housing
- removed N6: Ranzbak, library:goatse_01, symbol Mechanical:Housing
- removed N8: Bosch, proto1_kicad:bosch_logo, symbol Mechanical:Housing
- added C7, C90: 10u, Capacitor_SMD:C_0805_2012Metric, symbol Device:C
- added C91: 1u, Capacitor_SMD:C_0603_1608Metric, symbol mch2021-rescue:C-Device
Connections:
- net +3.3V: now also J5.1 (Pin_1); no longer J5.2 (Pin_2)
- net GND: now also J5.2 (Pin_2), C7.1, C90.1, C91.2; no longer J5.1 (Pin_1)
- net SAO_IO1: now also J5.5 (Pin_5), U30.1 (CHA), U30.10 (CHA); no longer J5.6 (Pin_6), U30.2 (CHB), U30.9 (CHB)
- net SAO_IO2: now also J5.6 (Pin_6), U30.2 (CHB), U30.9 (CHB); no longer J5.5 (Pin_5), U30.1 (CHA), U30.10 (CHA)
- net SAO_SCL: now also J5.4 (Pin_4); no longer J5.3 (Pin_3)
- net SAO_SDA: now also J5.3 (Pin_3); no longer J5.4 (Pin_4)
- net VBUS: now also C91.1
- net at C6.1, U4.13 (VDD33): now also C7.2, C90.2
Other:
- moved on the sheet: C8, N1, N5, N7

Commit message: Add extra header for JTAG reset and detect.
Parts:
- added J14: Conn_02x01, Connector_PinSocket_2.54mm:PinSocket_2x01_P2.54mm_Horizontal, symbol Connector_Generic:Conn_02x01
Connections:
- new net JTAG_ENABLE: J14.1 (Pin_1)
- new net P4_RESET: J14.2 (Pin_2)
Changed lines of the file:
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@@
 		)
 	)
+	(global_label "JTAG_ENABLE"
+		(shape input)
+		(at 107.95 175.26 180)
+		(fields_autoplaced yes)
+		(effects
+			(font
+				(size 1.27 1.27)
+			)
+			(justify right)
+		)
+		(property "Intersheetrefs" "${INTERSHEET_REFS}"
+			(at 92.6882 175.26 0)
+			(effects
+				(font
+					(size 1.27 1.27)
+				)
+				(justify right)
+				(hide yes)
+			)
+		)
+	)
 	(global_label "MTDO"
 		(shape output)
@@
 		)
 	)
+	(global_label "P4_RESET"
+		(shape output)
+		(at 120.65 175.26 0)
+		(effects
+			(font
+				(size 1.016 1.016)
+			)
+			(justify left)
+		)
+		(property "Intersheetrefs" "${INTERSHEET_REFS}"
+			(at 120.65 175.26 0)
+			(effects
+				(font
+					(size 1.27 1.27)
+				)
+				(hide yes)
+			)
+		)
+	)
 	(global_label "I2S_MCLK"
 		(shape input)
@@
 					(unit 1)
 				)
+			)
+		)
+	)
+	(symbol
+		(lib_id "Connector_Generic:Conn_02x01")
+		(at 113.03 175.26 0)
+		(mirror x)
+		(unit 1)
+		(exclude_from_sim no)
+		(in_bom yes)
+		(on_board yes)
+		(dnp yes)
+		(property "Reference" "J14"
+			(at 114.3 181.61 0)
+			(effects
+				(font
+					(size 1.27 1.27)
+				)
+			)
+		)
+		(property "Value" "Conn_02x01"
+			(at 114.3 179.07 0)
+			(effects
+				(font
+					(size 1.27 1.27)
+				)
+			)
+		)
+		(property "Footprint" "Connector_PinSocket_2.54mm:PinSocket_2x01_P2.54mm_Horizontal"
+			(at 113.03 175.26 0)
+			(effects
+				(font
+					(size 1.27 1.27)
+				)
+				(hide yes)
+			)
+		)
+		(property "Datasheet" "~"
+			(at 113.03 175.26 0)
+			(effects
+				(font
+					(size 1.27 1.27)
+				)
+				(hide yes)
+			)
+		)
+		(property "Description" "Generic connector, double row, 02x01, this symbol is compatible with counter-clockwise, top-bottom and odd-even numbering schemes., script generated (kicad-library-utils/schlib/autogen/connector/)"
+			(at 113.03 175.26 0)
+			(effects
+				(font
+					(size 1.27 1.27)
+				)
+				(hide yes)
+			)
+		)
+		(pin "2"
+		)
+		(pin "1"
+		)
+		(instances
+			(project ""
+				(path "/6a31734e-65de-48f3-8156-2b24b665b183"
+					(reference "J14")
+					(unit 1)
+				)

Commit message: Fix Ground detect for JTAG pin.
Parts:
- added R84: 1.5k, Resistor_SMD:R_0402_1005Metric, symbol symbols:R
Connections:
- net E2: now also R84.2
- net JTAG_ENABLE: no longer names the net of J14.1 (Pin_1)
- net JTAG_ENABLE: now also R84.1
Changed lines of the file:
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@@
 	(wire
 		(pts
+			(xy 106.68 175.26) (xy 107.95 175.26)
+		)
+		(stroke
+			(width 0)
+			(type default)
+		)
+	)
+	(wire
+		(pts
 			(xy 62.23 54.61) (xy 81.28 54.61)
 		)
@@
 	(wire
 		(pts
+			(xy 96.52 175.26) (xy 99.06 175.26)
+		)
+		(stroke
+			(width 0)
+			(type default)
+		)
+	)
+	(wire
+		(pts
 			(xy 166.37 135.89) (xy 187.96 135.89)
 		)
@@
 		)
 	)
-	(global_label "JTAG_ENABLE"
-		(shape input)
-		(at 107.95 175.26 180)
-		(fields_autoplaced yes)
-		(effects
-			(font
-				(size 1.27 1.27)
-			)
-			(justify right)
-		)
-		(property "Intersheetrefs" "${INTERSHEET_REFS}"
-			(at 92.6882 175.26 0)
-			(effects
-				(font
-					(size 1.27 1.27)
-				)
-				(justify right)
-				(hide yes)
-			)
-		)
-	)
 	(global_label "MTDO"
 		(shape output)
@@
 		)
 	)
+	(hierarchical_label "E2"
+		(shape bidirectional)
+		(at 96.52 175.26 180)
+		(fields_autoplaced yes)
+		(effects
+			(font
+				(size 1.27 1.27)
+			)
+			(justify right)
+		)
+	)
 	(symbol
 		(lib_id "Mechanical:MountingHole_Pad")
@@
 					(unit 1)
 				)
+			)
+		)
+	)
+	(symbol
+		(lib_id "symbols:R")
+		(at 102.87 175.26 270)
+		(mirror x)
+		(unit 1)
+		(exclude_from_sim no)
+		(in_bom yes)
+		(on_board yes)
+		(dnp no)
+		(property "Reference" "R84"
+			(at 101.6 179.07 0)
+			(effects
+				(font
+					(size 1.27 1.27)
+				)
+			)
+		)
+		(property "Value" "1.5k"
+			(at 104.14 179.07 0)
+			(effects
+				(font
+					(size 1.27 1.27)
+				)
+			)
+		)
+		(property "Footprint" "Resistor_SMD:R_0402_1005Metric"
+			(at 102.87 177.038 90)
+			(effects
+				(font
+					(size 1.27 1.27)
+				)
+				(hide yes)
+			)
+		)
+		(property "Datasheet" ""
+			(at 102.87 175.26 0)
+			(effects
+				(font
+					(size 1.27 1.27)
+				)
+				(hide yes)
+			)
+		)
+		(property "Description" ""
+			(at 102.87 175.26 0)
+			(effects
+				(font
+					(size 1.27 1.27)
+				)
+				(hide yes)
+			)
+		)
+		(property "LCSC" ""
+			(at 102.87 175.26 0)
+			(effects
+				(font
+					(size 1.27 1.27)
+				)
+				(hide yes)
+			)
+		)
+		(pin "1"
+		)
+		(pin "2"
+		)
+		(instances
+			(project "why2025"
+				(path "/6a31734e-65de-48f3-8156-2b24b665b183"
+					(reference "R84")
+					(unit 1)
+				)
