File: why2025.kicad_sch (KiCad schematic)
At the start: 42 parts, among them J1 USB device, J10 Expansion I3C, J12 SAO, J14 Conn_02x01, J2 USB host, J4 Headphone, J5 External Add-On (SAO / PMOD), J6 Internal Add-On, J7 Speaker, J8 Micro_SD_Card, J9 CAMERA, SW3 Boot, U28 USBLC6-2P6, U29 USBLC6-2P6, U30 ESD, U31 ESD, U4 CH334R, Y1 12MHz

Commit message: Swapped GPIO32 and GPIO00, added functionality to use 1 3v3 pin as the P4 RESET.
Parts:
- removed J14: Conn_02x01, Connector_PinSocket_2.54mm:PinSocket_2x01_P2.54mm_Horizontal, symbol Connector_Generic:Conn_02x01
- removed R84: 1.5k, Resistor_SMD:R_0402_1005Metric, symbol symbols:R
- added JP4: ~, Jumper:SolderJumper-2_P1.3mm_Bridged_RoundedPad1.0x1.5mm, symbol Jumper:Jumper_2_Bridged
- added R85: 1k, Resistor_SMD:R_0402_1005Metric, symbol Device:R
Connections:
- net +3.3V: now also JP4.1 (A); no longer J5.13 (Pin_13)
- net P4_RESET: now also R85.2
- new net: J5.13 (Pin_13), JP4.2 (B), R85.1
Other:
- moved on the sheet: J5

Commit message: Add latch to power on from the ch32.
Changed lines of the file:
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@@
 	)
 	(sheet
-		(at 82.55 90.17)
-		(size 17.78 22.86)
+		(at 82.55 87.63)
+		(size 17.78 25.4)
 		(fields_autoplaced yes)
 		(stroke
@@
 		)
 		(property "Sheetname" "Power"
-			(at 82.55 89.4584 0)
+			(at 82.55 86.9184 0)
 			(effects
 				(font

Commit message: Fix SR latch circuit
Parts:
- JP4: footprint Jumper:SolderJumper-2_P1.3mm_Bridged_RoundedPad1.0x1.5mm -> Jumper:SolderJumper-2_P1.3mm_Open_RoundedPad1.0x1.5mm
Changed lines of the file:
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@@
 			)
 		)
-		(property "Footprint" "Jumper:SolderJumper-2_P1.3mm_Bridged_RoundedPad1.0x1.5mm"
+		(property "Footprint" "Jumper:SolderJumper-2_P1.3mm_Open_RoundedPad1.0x1.5mm"
 			(at 107.95 152.4 0)
 			(effects

Commit message: WIP: change LED, camera, LoRa and C6 pins and add USB-A port 1A current limit
Connections:
- net VOTG: no longer J2.1 (VBUS), U29.5 (VBUS)
- net CAM_GPIO0 renamed CAM_PWR_EN
- net CAM_GPIO1 renamed CAM_LED_EN
- new net VOTG_OUT: J2.1 (VBUS), U29.5 (VBUS)
Other:
- sheet Application processor ports: added CAM_LED_EN; removed CAM_GPIO1
- sheet Coprocessor ports: added LED_DATA, USB_ENABLE; removed C6_BOOT, CAMERA
- sheet LEDs ports: added none; removed ENABLE
- sheet Power ports: added USB_ENABLE; removed none
- sheet Radio ports: added none; removed LED_DATA, LED_ENABLE
- moved on the sheet: R46, R81

Commit message: Add BMI270 sensor
Parts:
- removed R81: 2k2, Resistor_SMD:R_0402_1005Metric, symbol Device:R
Other:
- sheet Sensors ports: added none; removed INT
Changed lines of the file:
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@@
 	(title_block
 		(title "WHY2025 badge")
-		(date "2024-09-12")
-		(rev "Prototype 2")
+		(date "2024-11-01")
+		(rev "Prototype 3")
 		(company "Badge.Team")
 		(comment 1 "Copyright 2024 Nicolai Electronics")
@@
 	(wire
 		(pts
-			(xy 78.74 124.46) (xy 82.55 124.46)
-		)
-		(stroke
-			(width 0)
-			(type default)
-		)
-	)
-	(wire
-		(pts
 			(xy 223.52 156.21) (xy 226.06 156.21)
 		)
@@
 		)
 	)
-	(global_label "E11"
-		(shape bidirectional)
-		(at 71.12 124.46 180)
-		(fields_autoplaced yes)
-		(effects
-			(font
-				(size 1.016 1.016)
-			)
-			(justify right)
-		)
-		(property "Intersheetrefs" "${INTERSHEET_REFS}"
-			(at 64.9887 124.46 0)
-			(effects
-				(font
-					(size 1.27 1.27)
-				)
-				(justify right)
-				(hide yes)
-			)
-		)
-	)
 	(global_label "E1"
 		(shape bidirectional)
@@
 	)
 	(symbol
-		(lib_id "Device:R")
-		(at 74.93 124.46 270)
-		(unit 1)
-		(exclude_from_sim no)
-		(in_bom yes)
-		(on_board yes)
-		(dnp no)
-		(property "Reference" "R81"
-			(at 79.502 123.19 90)
-			(effects
-				(font
-					(size 1.27 1.27)
-				)
-			)
-		)
-		(property "Value" "2k2"
-			(at 79.502 125.73 90)
-			(effects
-				(font
-					(size 1.27 1.27)
-				)
-			)
-		)
-		(property "Footprint" "Resistor_SMD:R_0402_1005Metric"
-			(at 74.93 122.682 90)
-			(effects
-				(font
-					(size 1.27 1.27)
-				)
-				(hide yes)
-			)
-		)
-		(property "Datasheet" "https://www.lcsc.com/product-detail/Chip-Resistor-Surface-Mount_UNI-ROYAL-Uniroyal-Elec-0402WGF2201TCE_C25879.html"
-			(at 74.93 124.46 0)
-			(effects
-				(font
-					(size 1.27 1.27)
-				)
-				(hide yes)
-			)
-		)
-		(property "Description" ""
-			(at 74.93 124.46 0)
-			(effects
-				(font
-					(size 1.27 1.27)
-				)
-				(hide yes)
-			)
-		)
-		(property "LCSC" "C25879"
-			(at 74.93 124.46 0)
-			(effects
-				(font
-					(size 1.27 1.27)
-				)
-				(hide yes)
-			)
-		)
-		(pin "1"
-		)
-		(pin "2"
-		)
-		(instances
-			(project "why2025"
-				(path "/6a31734e-65de-48f3-8156-2b24b665b183"
-					(reference "R81")
-					(unit 1)
-				)
-			)
-		)
-	)
-	(symbol
 		(lib_id "mch2021-rescue:GND-power")
 		(at 252.73 161.29 270)
@@
 			)
 		)
-		(pin "INT" output
-			(at 82.55 124.46 180)
-			(effects
-				(font
-					(size 1.27 1.27)
-				)
-				(justify left)
-			)
-		)

Commit message: Move micro sd card slot, remove E1 from the expansion header
Connections:
- net E2: now also J6.12 (Pin_12); no longer J6.13 (Pin_13)
- net GND: now also J6.7 (Pin_7)
- net VSDCARD: now also J6.13 (Pin_13); no longer J6.7 (Pin_7)
- net E1 renamed BOOT
- net BOOT: no longer J6.12 (Pin_12)
Changed lines of the file:
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@@
 		)
 	)
-	(global_label "E1"
-		(shape bidirectional)
+	(global_label "BOOT"
+		(shape input)
 		(at 226.06 128.27 0)
 		(fields_autoplaced yes)
@@
 		)
 		(property "Intersheetrefs" "${INTERSHEET_REFS}"
-			(at 231.2237 128.27 0)
+			(at 232.3668 128.27 0)
 			(effects
 				(font
@@
 	(global_label "E2"
 		(shape bidirectional)
-		(at 252.73 133.35 180)
+		(at 265.43 130.81 0)
 		(fields_autoplaced yes)
 		(effects
@@
 				(size 1.016 1.016)
 			)
-			(justify right)
+			(justify left)
 		)
 		(property "Intersheetrefs" "${INTERSHEET_REFS}"
-			(at 247.5663 133.35 0)
+			(at 270.5937 130.81 0)
 			(effects
 				(font
 					(size 1.27 1.27)
 				)
-				(justify right)
+				(justify left)
 				(hide yes)
 			)
@@
 		)
 	)
-	(global_label "E1"
-		(shape bidirectional)
+	(global_label "BOOT"
+		(shape output)
 		(at 62.23 132.08 0)
 		(fields_autoplaced yes)
@@
 		)
 		(property "Intersheetrefs" "${INTERSHEET_REFS}"
-			(at 67.3937 132.08 0)
+			(at 68.5368 132.08 0)
 			(effects
 				(font
@@
 		)
 	)
-	(global_label "E1"
-		(shape bidirectional)
-		(at 265.43 130.81 0)
-		(fields_autoplaced yes)
-		(effects
-			(font
-				(size 1.016 1.016)
-			)
-			(justify left)
-		)
-		(property "Intersheetrefs" "${INTERSHEET_REFS}"
-			(at 270.5937 130.81 0)
-			(effects
-				(font
-					(size 1.27 1.27)
-				)
-				(justify left)
-				(hide yes)
-			)
-		)
-	)
 	(global_label "EXT_USB_P"
 		(shape bidirectional)
@@
 	)
 	(symbol
+		(lib_id "mch2021-rescue:GND-power")
+		(at 252.73 125.73 270)
+		(unit 1)
+		(exclude_from_sim no)
+		(in_bom yes)
+		(on_board yes)
+		(dnp no)
+		(property "Reference" "#PWR0314"
+			(at 246.38 125.73 0)
+			(effects
+				(font
+					(size 1.27 1.27)
+				)
+				(hide yes)
+			)
+		)
+		(property "Value" "GND"
+			(at 247.904 125.73 90)
+			(effects
+				(font
+					(size 1.27 1.27)
+				)
+			)
+		)
+		(property "Footprint" ""
+			(at 252.73 125.73 0)
+			(effects
+				(font
+					(size 1.27 1.27)
+				)
+				(hide yes)
+			)
+		)
+		(property "Datasheet" ""
+			(at 252.73 125.73 0)
+			(effects
+				(font
+					(size 1.27 1.27)
+				)
+				(hide yes)
+			)
+		)
+		(property "Description" ""
+			(at 252.73 125.73 0)
+			(effects
+				(font
+					(size 1.27 1.27)
+				)
+				(hide yes)
+			)
+		)
+		(pin "1"
+		)
+		(instances
+			(project "why2025"
+				(path "/6a31734e-65de-48f3-8156-2b24b665b183"
+					(reference "#PWR0314")
+					(unit 1)
+				)
+			)
+		)
+	)
+	(symbol
 		(lib_id "power:GND")
 		(at 58.42 144.78 0)
@@
 	(symbol
 		(lib_id "custom-power:VSDCARD")
-		(at 252.73 125.73 90)
+		(at 252.73 133.35 90)
 		(unit 1)
 		(exclude_from_sim no)
@@
 		(dnp no)
 		(property "Reference" "#PWR0197"
-			(at 256.54 125.73 0)
+			(at 256.54 133.35 0)
 			(effects
 				(font
@@
 		)
 		(property "Value" "VSDCARD"
-			(at 249.682 125.73 90)
+			(at 249.936 133.35 90)
 			(effects
 				(font
@@
 		)
 		(property "Footprint" ""
-			(at 252.73 125.73 0)
+			(at 252.73 133.35 0)
 			(effects
 				(font
@@
 		)
 		(property "Datasheet" ""
-			(at 252.73 125.73 0)
+			(at 252.73 133.35 0)
 			(effects
 				(font
@@
 		)
 		(property "Description" "Power symbol creates a global label with name \"VSDCARD\""
-			(at 254.508 125.73 0)
+			(at 254.508 133.35 0)
 			(effects
 				(font

Commit message: Change TE resistor to 100k pull-down and export production files
Parts:
- J12, JP4: LCSC (none) -> -
