File: frontpanel/frontpanel.kicad_pcb (KiCad board)
At the start: 2 copper layers, 114.9 x 125.5 mm, 1 part

Commit message: Work in progress
Parts:
- added H1: ~, MountingHole:MountingHole_2.2mm_M2_Pad_Via, F.Cu at (-50.0, -88.2)
- added H2: ~, MountingHole:MountingHole_2.2mm_M2_Pad_Via, F.Cu at (50.0, -88.2)
- added H3: ~, MountingHole:MountingHole_2.2mm_M2_Pad_Via, F.Cu at (-36.0, 30.0)
- added H4: ~, MountingHole:MountingHole_2.2mm_M2_Pad_Via, F.Cu at (36.0, 30.0)
- added H5: ~, MountingHole:MountingHole_2.2mm_M2_Pad_Via, F.Cu at (-53.0, 3.00)
- added H6: ~, MountingHole:MountingHole_2.2mm_M2_Pad_Via, F.Cu at (53.0, 3.00)
- N1: footprint proto1_kicad_art:proto1_kicad_art -> design:proto1_kicad_art2
- moved N1 21.4 mm to (0.00, -21.4)
Routing:
- added copper zone on B.Cu, net GND
Other:
- board text added: "Badge.Team"
- board text added: "DOT MATRIX WITH STEREO SOUND"
- board text added: "Prototype 1"

Commit message: Frontpanel stuff
Parts:
- removed H5, H6: ~, MountingHole:MountingHole_2.2mm_M2_Pad_Via
- added C1: 100n, Capacitor_SMD:C_0603_1608Metric, F.Cu at (-4.21, -36.6)
- added C2: 1u, Capacitor_SMD:C_0402_1005Metric, F.Cu at (-29.0, -38.5)
- added C3: 100n, Capacitor_SMD:C_0402_1005Metric, F.Cu at (-29.0, -37.5)
- added C4: 100n, Capacitor_SMD:C_0402_1005Metric, F.Cu at (-29.0, -41.0)
- added C5: 1u, Capacitor_SMD:C_0402_1005Metric, F.Cu at (-29.0, -40.0)
- added D10: LL4148, Diode_SMD:D_SOD-323, F.Cu at (22.5, -48.0)
- added D11: LL4148, Diode_SMD:D_SOD-323, F.Cu at (19.0, -25.0)
- added D12: LL4148, Diode_SMD:D_SOD-323, F.Cu at (10.8, -32.0)
- added D13: LL4148, Diode_SMD:D_SOD-323, F.Cu at (-16.0, -34.0)
- added D14: LL4148, Diode_SMD:D_SOD-323, F.Cu at (-16.0, -32.0)
- added D15: LL4148, Diode_SMD:D_SOD-323, F.Cu at (-1.50, -33.0)
- added D16: LL4148, Diode_SMD:D_SOD-323, F.Cu at (1.00, -17.5)
- added D17: LL4148, Diode_SMD:D_SOD-323, F.Cu at (-16.0, -40.0)
- added D18: LL4148, Diode_SMD:D_SOD-323, F.Cu at (24.5, -48.0)
- added D19: LL4148, Diode_SMD:D_SOD-323, F.Cu at (7.50, -33.0)
- added D2: LL4148, Diode_SMD:D_SOD-323, F.Cu at (24.0, -32.0)
- added D20: LL4148, Diode_SMD:D_SOD-323, F.Cu at (4.00, -17.5)
- added D21: LL4148, Diode_SMD:D_SOD-323, F.Cu at (-16.0, -38.0)
- added D3: LL4148, Diode_SMD:D_SOD-323, F.Cu at (33.0, -38.0)
- added D4: LL4148, Diode_SMD:D_SOD-323, F.Cu at (26.5, -32.0)
- added D5: LL4148, Diode_SMD:D_SOD-323, F.Cu at (17.8, -39.0)
- added D6: LL4148, Diode_SMD:D_SOD-323, F.Cu at (-24.5, -48.0)
- added D7: LL4148, Diode_SMD:D_SOD-323, F.Cu at (11.0, -46.0)
- added D8: LL4148, Diode_SMD:D_SOD-323, F.Cu at (-22.5, -48.0)
- added D9: LL4148, Diode_SMD:D_SOD-323, F.Cu at (-16.0, -36.0)
- added J1: I2C, library:1X04_1MM_RA_GND, F.Cu at (-10.0, -47.0)
- added J2: USB device, Connector_USB:USB_C_Receptacle_HRO_TYPE-C-31-M-12, F.Cu at (0.00, -48.0)
- added JP1: A0, Jumper:SolderJumper-2_P1.3mm_Open_TrianglePad1.0x1.5mm, F.Cu at (1.00, -21.0)
- added JP2: A1, Jumper:SolderJumper-2_P1.3mm_Open_TrianglePad1.0x1.5mm, F.Cu at (4.00, -21.0)
- added R1: 5k1, Resistor_SMD:R_0402_1005Metric, F.Cu at (1.99, -41.4)
- added R11: 10k, Resistor_SMD:R_0402_1005Metric, F.Cu at (5.00, -35.5)
- added R2: 5k1, Resistor_SMD:R_0402_1005Metric, F.Cu at (-1.99, -41.4)
- added R3: 33, Resistor_SMD:R_0402_1005Metric, F.Cu at (0.00, -41.4)
- added R4: 33, Resistor_SMD:R_0402_1005Metric, F.Cu at (0.99, -41.4)
- added R5: 1.5k, Resistor_SMD:R_0402_1005Metric, F.Cu at (-0.99, -41.4)
- added R7: 10k, Resistor_SMD:R_0402_1005Metric, F.Cu at (30.0, -42.0)
- added R8: 10k, Resistor_SMD:R_0402_1005Metric, F.Cu at (36.0, -40.5)
- added R9: 10k, Resistor_SMD:R_0402_1005Metric, F.Cu at (30.0, -43.0)
- added S1: JS1400BFQ, joystick_footprint:SW_JS1400BFQ, F.Cu at (-25.8, -31.8)
- added SW1: X, button_footprint:KEY-SMD_2P-L6.0-W6.0-P6.00, F.Cu at (24.8, -39.4)
- added SW10: C, button_footprint:KEY-SMD_2P-L6.0-W6.0-P6.00, F.Cu at (18.9, -17.5)
- added SW11: Z, button_footprint:KEY-SMD_2P-L6.0-W6.0-P6.00, F.Cu at (10.8, -25.4)
- added SW12: K1-1539SA-01, analog_joystick:SW-SMD_K1-1539SA-01, F.Cu at (-9.27, -17.4)
- added SW14: SELECT, button_footprint:KEY-SMD_2P-L6.0-W6.0-P6.00, F.Cu at (-6.00, -28.8)
- added SW18: START, button_footprint:KEY-SMD_2P-L6.0-W6.0-P6.00, F.Cu at (3.00, -28.8)
- added SW2: A, button_footprint:KEY-SMD_2P-L6.0-W6.0-P6.00, F.Cu at (32.9, -31.5)
- added SW3: B, button_footprint:KEY-SMD_2P-L6.0-W6.0-P6.00, F.Cu at (25.9, -24.5)
- added SW4: Y, button_footprint:KEY-SMD_2P-L6.0-W6.0-P6.00, F.Cu at (17.8, -32.4)
- added SW5: R, shoulderbutton:KEY-TH_TC-1101V-C-A-W, F.Cu at (32.0, -48.0)
- added SW6: HOME, button_footprint:KEY-SMD_2P-L6.0-W6.0-P6.00, F.Cu at (10.8, -39.4)
- added SW7: -, button_footprint:KEY-SMD_2P-L6.0-W6.0-P6.00, F.Cu at (-17.8, -46.4)
- added SW8: L, shoulderbutton:KEY-TH_TC-1101V-C-A-W, F.Cu at (-32.0, -48.0)
- added SW9: +, button_footprint:KEY-SMD_2P-L6.0-W6.0-P6.00, F.Cu at (17.8, -46.4)
- added TP1: 3.3v, TestPoint:TestPoint_Pad_D1.5mm, F.Cu at (7.00, -51.0)
- added TP2: GND, TestPoint:TestPoint_Pad_D1.5mm, F.Cu at (9.54, -51.0)
- added TP3: SWIO, TestPoint:TestPoint_Pad_D1.5mm, F.Cu at (12.1, -51.0)
- added U1: CH32V003F4U6, Package_DFN_QFN:QFN-20-1EP_3x3mm_P0.4mm_EP1.65x1.65mm, F.Cu at (0.00, -38.0)
- added U2: LM1117MP-3.3, Package_TO_SOT_SMD:SOT-223-3_TabPin2, F.Cu at (-34.0, -40.0)
- H1, H2, H3, H4: value ~ -> Mounting hole; footprint MountingHole:MountingHole_2.2mm_M2_Pad_Via -> MountingHole:MountingHole_2.1mm
- N1: value Housing -> Board; footprint design:proto1_kicad_art2 -> design:proto1_kicad_frontpanel
- moved H3 32.0 mm to (-44.4, 60.9)
- moved H4 32.0 mm to (44.4, 60.9)
- moved H1 30.4 mm to (-50.4, -57.9)
- moved H2 30.4 mm to (50.4, -57.9)
- moved N1 21.4 mm to (0.00, 0.00)
Routing:
- net COL2: track 0.00 -> 139.9 mm, vias 0 -> 2
- net COL3: track 0.00 -> 113.8 mm, vias 0 -> 4
- net ROW5: track 0.00 -> 100.9 mm, vias 0 -> 2
- net +3.3V: track 0.00 -> 91.7 mm, vias 0 -> 4
- net ROW1: track 0.00 -> 84.9 mm, vias 0 -> 2
- net ROW2: track 0.00 -> 78.6 mm, vias 0 -> 2
- net ROW3: track 0.00 -> 65.6 mm, vias 0 -> 3
- net ROW4: track 0.00 -> 61.0 mm, vias 0 -> 3
- net COL1: track 0.00 -> 58.8 mm, vias 0 -> 2
- net JOY_E: track 0.00 -> 42.6 mm, vias 0 -> 2
- net VBUS: track 0.00 -> 41.7 mm, vias 0 -> 2
- net JOY_V: track 0.00 -> 36.7 mm, vias 0 -> 2
- net COL4: track 0.00 -> 33.7 mm, vias 0 -> 2
- net SCL: track 0.00 -> 24.2 mm
- net SDA: track 0.00 -> 23.3 mm
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- added copper zone on In1.Cu, net +3.3V
- added copper zone on F.Cu, net GND
- added copper zone on In2.Cu, net GND
Other:
- board size 114.9 x 125.5 mm -> 114.9 x 129.9 mm
- copper layers 2 -> 4
- board text removed: "Badge.Team"
- board text removed: "DOT MATRIX WITH STEREO SOUND"

Commit message: Frontpanel :D
Parts:
- added H1: Gamepad, mountinghole:mountinghole_1.6mm, F.Cu at (-40.0, -49.0)
- added H2: Gamepad, mountinghole:mountinghole_1.6mm, F.Cu at (40.0, -49.0)
- added H3: Gamepad, mountinghole:mountinghole_1.6mm, F.Cu at (-40.0, -4.30)
- added H4: Gamepad, mountinghole:mountinghole_1.6mm, F.Cu at (40.0, -4.30)
- added N2: Stamp, stamp:stamp, B.Cu at (0.00, -28.0)
- added U1: LM66100DCKR, ideal_diode:SC-70-6_L2.0-W1.3-P0.65-LS2.1-BL, F.Cu at (-7.54, -44.1)
- C1: footprint Capacitor_SMD:C_0603_1608Metric -> Capacitor_SMD:C_0402_1005Metric
- moved D19 5.49 mm to (4.40, -13.2)
- moved D20 5.49 mm to (7.40, -13.2)
- moved JP1 5.49 mm to (4.40, -16.7)
- moved JP2 5.49 mm to (7.40, -16.7)
- moved TP1 0.50 mm to (7.00, -50.5)
- moved TP2 0.50 mm to (9.54, -50.5)
- moved TP3 0.50 mm to (12.1, -50.5)
- renumbered D2 to D1, D19 to D10, D9 to D11, D17 to D12, D21 to D15, D10 to D16, D8 to D17, D12 to D18, D16 to D19, D3 to D2, D4 to D3, D5 to D4, D18 to D5, D11 to D8, D15 to D9, H1 to H5, H2 to H6, H3 to H7, H4 to H8, R5 to R3, R3 to R4, R4 to R5, R7 to R6, R8 to R7, R11 to R8, SW12 to SW1, SW14 to SW10, SW18 to SW11, SW9 to SW12, SW7 to SW13, SW11 to SW14, SW1 to SW2, SW2 to SW3, SW3 to SW4, SW4 to SW5, SW5 to SW6, SW8 to SW7, SW6 to SW8, SW10 to SW9, U1 to U2, U2 to U3
Connections:
- J1 pad 2: +3.3V -> Net-(J1-VCC)
Routing:
- net +3.3V: track 91.7 -> 77.4 mm
- net ROW5: track 100.9 -> 106.6 mm
- net COL3: track 113.8 -> 118.7 mm
- net ROW4: track 61.0 -> 65.2 mm
- net Net-(J1-VCC): track 0.00 -> 2.88 mm
- net GND: vias 10 -> 144
- removed copper zone on In1.Cu, net +3.3V
- removed copper zone on In2.Cu, net GND
Other:
- copper layers 4 -> 2
- board text added: "+"
- board text added: "+ - P"
- board text added: "-"
- board text added: "2 1"
- board text added: "A"
- board text added: "ANALOG"
- board text added: "B"
- board text added: "C"
- board text added: "H"
- board text added: "L"
- board text added: "QWIIC"
- board text added: "R"
- board text added: "SELECT"
- board text added: "START"
- board text added: "WHY2025 Prototype 1"
- board text added: "WHYpad"
- board text added: "X"
- board text added: "Y"
- board text added: "Z"
- board text removed: "Prototype 1"

Commit message: Frontpanel stuff
Parts:
- removed C1, C3, C4: 100n, Capacitor_SMD:C_0402_1005Metric
- removed C2, C5: 1u, Capacitor_SMD:C_0402_1005Metric
- removed D1, D10, D11, D12, D13, D14, D15, D16, D17, D18, D19, D2, D20, D3, D4, D5, D6, D7, D8, D9: LL4148, Diode_SMD:D_SOD-323
- removed H1, H2, H3, H4: Gamepad, mountinghole:mountinghole_1.6mm
- removed J1: I2C, library:1X04_1MM_RA_GND
- removed J2: USB device, Connector_USB:USB_C_Receptacle_HRO_TYPE-C-31-M-12
- removed JP1: A0, Jumper:SolderJumper-2_P1.3mm_Open_TrianglePad1.0x1.5mm
- removed JP2: A1, Jumper:SolderJumper-2_P1.3mm_Open_TrianglePad1.0x1.5mm
- removed N2: Stamp, stamp:stamp
- removed R1, R2: 5k1, Resistor_SMD:R_0402_1005Metric
- removed R3: 1.5k, Resistor_SMD:R_0402_1005Metric
- removed R4, R5: 33, Resistor_SMD:R_0402_1005Metric
- removed R6, R7, R8, R9: 10k, Resistor_SMD:R_0402_1005Metric
- removed S1: JS1400BFQ, joystick_footprint:SW_JS1400BFQ
- removed SW1: K1-1539SA-01, analog_joystick:SW-SMD_K1-1539SA-01
- removed SW10: SELECT, button_footprint:KEY-SMD_2P-L6.0-W6.0-P6.00
- removed SW11: START, button_footprint:KEY-SMD_2P-L6.0-W6.0-P6.00
- removed SW12: +, button_footprint:KEY-SMD_2P-L6.0-W6.0-P6.00
- removed SW13: -, button_footprint:KEY-SMD_2P-L6.0-W6.0-P6.00
- removed SW14: Z, button_footprint:KEY-SMD_2P-L6.0-W6.0-P6.00
- removed SW2: X, button_footprint:KEY-SMD_2P-L6.0-W6.0-P6.00
- removed SW3: A, button_footprint:KEY-SMD_2P-L6.0-W6.0-P6.00
- removed SW4: B, button_footprint:KEY-SMD_2P-L6.0-W6.0-P6.00
- removed SW5: Y, button_footprint:KEY-SMD_2P-L6.0-W6.0-P6.00
- removed SW6: R, shoulderbutton:KEY-TH_TC-1101V-C-A-W
- removed SW7: L, shoulderbutton:KEY-TH_TC-1101V-C-A-W
- removed SW8: HOME, button_footprint:KEY-SMD_2P-L6.0-W6.0-P6.00
- removed SW9: C, button_footprint:KEY-SMD_2P-L6.0-W6.0-P6.00
- removed TP1: 3.3v, TestPoint:TestPoint_Pad_D1.5mm
- removed TP2: GND, TestPoint:TestPoint_Pad_D1.5mm
- removed TP3: SWIO, TestPoint:TestPoint_Pad_D1.5mm
- removed U1: LM66100DCKR, ideal_diode:SC-70-6_L2.0-W1.3-P0.65-LS2.1-BL
- removed U2: CH32V003F4U6, Package_DFN_QFN:QFN-20-1EP_3x3mm_P0.4mm_EP1.65x1.65mm
- removed U3: LM1117MP-3.3, Package_TO_SOT_SMD:SOT-223-3_TabPin2
- N1: footprint design:proto1_kicad_frontpanel -> design:frontpanel_honeycomb
Routing:
- net COL2: track 139.9 -> 0.00 mm, vias 2 -> 0
- net COL3: track 118.7 -> 0.00 mm, vias 4 -> 0
- net ROW5: track 106.6 -> 0.00 mm, vias 2 -> 0
- net ROW1: track 84.9 -> 0.00 mm, vias 2 -> 0
- net ROW2: track 78.6 -> 0.00 mm, vias 2 -> 0
- net +3.3V: track 77.4 -> 0.00 mm, vias 4 -> 0
- net ROW3: track 65.6 -> 0.00 mm, vias 3 -> 0
- net ROW4: track 65.2 -> 0.00 mm, vias 3 -> 0
- net COL1: track 58.8 -> 0.00 mm, vias 2 -> 0
- net JOY_E: track 42.6 -> 0.00 mm, vias 2 -> 0
- net VBUS: track 41.7 -> 0.00 mm, vias 2 -> 0
- net JOY_V: track 36.7 -> 0.00 mm, vias 2 -> 0
- net COL4: track 33.7 -> 0.00 mm, vias 2 -> 0
- net SCL: track 24.2 -> 0.00 mm
- net SDA: track 23.3 -> 0.00 mm
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- added copper zone on B.Cu, net (none)
- removed copper zone on B.Cu, net GND
- removed copper zone on F.Cu, net GND
Other:
- outline, holes or cut-outs redrawn
- board text added: "WHY2025 Prototype 2"
- board text removed: "+"
- board text removed: "+ - P"
- board text removed: "-"
- board text removed: "2 1"
- board text removed: "A"
- board text removed: "ANALOG"
- board text removed: "B"
- board text removed: "C"
- board text removed: "H"
- board text removed: "L"
- board text removed: "QWIIC"
- board text removed: "R"
- board text removed: "SELECT"
- board text removed: "START"
- board text removed: "WHY2025 Prototype 1"
- board text removed: "WHYpad"
- board text removed: "X"
- board text removed: "Y"
- board text removed: "Z"
