File: frontpanel/frontpanel.kicad_sch (KiCad schematic)
At the start: 1 part

Commit message: Work in progress
Parts:
- added H1, H2, H3, H4, H5, H6: ~, MountingHole:MountingHole_2.2mm_M2_Pad_Via, symbol Mechanical:MountingHole_Pad
- N1: footprint proto1_kicad_art:proto1_kicad_art -> design:proto1_kicad_art2
Connections:
- new net GND: H1.1, H2.1, H3.1, H4.1, H5.1, H6.1
Other:
- company: (none) -> Badge.Team
- title: (none) -> WHY2025 badge

Commit message: Frontpanel stuff
Parts:
- removed H5, H6: ~, MountingHole:MountingHole_2.2mm_M2_Pad_Via, symbol Mechanical:MountingHole_Pad
- added C1: 100n, Capacitor_SMD:C_0603_1608Metric, symbol vfd:C_Small
- added C2, C5: 1u, Capacitor_SMD:C_0402_1005Metric, symbol mch2021-rescue:C-Device
- added C3, C4: 100n, Capacitor_SMD:C_0402_1005Metric, symbol mch2021-rescue:C-Device
- added D10, D11, D12, D13, D14, D15, D16, D17, D18, D19, D2, D20, D21, D3, D4, D5, D6, D7, D8, D9: LL4148, Diode_SMD:D_SOD-323, symbol button_matrix:D_Small
- added J1: I2C, library:1X04_1MM_RA_GND, symbol symbols:QWIIC_MCH
- added J2: USB device, Connector_USB:USB_C_Receptacle_HRO_TYPE-C-31-M-12, symbol mch2021-rescue:USB_C_Receptacle_USB2.0-Connector
- added JP1: A0, Jumper:SolderJumper-2_P1.3mm_Open_TrianglePad1.0x1.5mm, symbol vfd:Jumper_2_Open
- added JP2: A1, Jumper:SolderJumper-2_P1.3mm_Open_TrianglePad1.0x1.5mm, symbol vfd:Jumper_2_Open
- added R1, R2: 5k1, Resistor_SMD:R_0402_1005Metric, symbol mch2021-rescue:R_Small-Device
- added R11, R7, R8, R9: 10k, Resistor_SMD:R_0402_1005Metric, symbol button_matrix:R
- added R3, R4: 33, Resistor_SMD:R_0402_1005Metric, symbol mch2021-rescue:R-Device
- added R5: 1.5k, Resistor_SMD:R_0402_1005Metric, symbol mch2021-rescue:R-Device
- added S1: JS1400BFQ, joystick_footprint:SW_JS1400BFQ, symbol JS1400BFQ:JS1400BFQ
- added SW1: X, button_footprint:KEY-SMD_2P-L6.0-W6.0-P6.00, symbol Switch:SW_Push
- added SW10: C, button_footprint:KEY-SMD_2P-L6.0-W6.0-P6.00, symbol Switch:SW_Push
- added SW11: Z, button_footprint:KEY-SMD_2P-L6.0-W6.0-P6.00, symbol Switch:SW_Push
- added SW12: K1-1539SA-01, analog_joystick:SW-SMD_K1-1539SA-01, symbol SW-SMD_K1-1539SA-01:K1-1539SA-01
- added SW14: SELECT, button_footprint:KEY-SMD_2P-L6.0-W6.0-P6.00, symbol Switch:SW_Push
- added SW18: START, button_footprint:KEY-SMD_2P-L6.0-W6.0-P6.00, symbol Switch:SW_Push
- added SW2: A, button_footprint:KEY-SMD_2P-L6.0-W6.0-P6.00, symbol Switch:SW_Push
- added SW3: B, button_footprint:KEY-SMD_2P-L6.0-W6.0-P6.00, symbol Switch:SW_Push
- added SW4: Y, button_footprint:KEY-SMD_2P-L6.0-W6.0-P6.00, symbol Switch:SW_Push
- added SW5: R, shoulderbutton:KEY-TH_TC-1101V-C-A-W, symbol pushbutton_gnd:pushbutton_gnd
- added SW6: HOME, button_footprint:KEY-SMD_2P-L6.0-W6.0-P6.00, symbol Switch:SW_Push
- added SW7: -, button_footprint:KEY-SMD_2P-L6.0-W6.0-P6.00, symbol Switch:SW_Push
- added SW8: L, shoulderbutton:KEY-TH_TC-1101V-C-A-W, symbol pushbutton_gnd:pushbutton_gnd
- added SW9: +, button_footprint:KEY-SMD_2P-L6.0-W6.0-P6.00, symbol Switch:SW_Push
- added TP1: 3.3v, TestPoint:TestPoint_Pad_D1.5mm, symbol vfd:TestPoint
- added TP2: GND, TestPoint:TestPoint_Pad_D1.5mm, symbol vfd:TestPoint
- added TP3: SWIO, TestPoint:TestPoint_Pad_D1.5mm, symbol vfd:TestPoint
- added U1: CH32V003F4U6, Package_DFN_QFN:QFN-20-1EP_3x3mm_P0.4mm_EP1.65x1.65mm, symbol vfd:CH32V003F4U6
- added U2: LM1117MP-3.3, Package_TO_SOT_SMD:SOT-223-3_TabPin2, symbol Regulator_Linear:LM1117MP-3.3
- H1, H2, H3, H4: value ~ -> Mounting hole; footprint MountingHole:MountingHole_2.2mm_M2_Pad_Via -> MountingHole:MountingHole_2.1mm; symbol Mechanical:MountingHole_Pad -> Mechanical:MountingHole; LCSC C2928171 -> -; now left out of the parts list
- N1: value Housing -> Board; footprint design:proto1_kicad_art2 -> design:proto1_kicad_frontpanel; LCSC (none) -> -; now left out of the parts list
Connections:
- net GND: now also C1.1, C2.2, C3.2, C4.2, C5.2, J1.1 (GND), J1.5, J1.6, J2.A1 (GND), J2.A12 (GND), J2.B1 (GND), J2.B12 (GND), J2.S1 (SHIELD), R1.1, R11.1, R2.1, R7.2, R8.2, R9.2, S1.SH1 (SHIELD), S1.SH2 (SHIELD), SW12.3, SW12.4, SW5.3, SW5.4, SW8.3, SW8.4, TP2.1, U1.21 (VSS), U1.4 (VSS), U2.1 (GND); no longer H1.1, H2.1, H3.1, H4.1
- new net: J2.A6 (D+), J2.B6 (D+), R4.1
- new net: D20.2 (A), JP2.1 (A)
- new net: D6.2 (A), SW8.2
- new net: D7.2 (A), SW6.2
- new net: D2.2 (A), SW1.2
- new net: D9.1 (K), S1.1
- new net: D10.2 (A), SW9.2
- new net: D4.2 (A), SW3.2
- new net: D19.2 (A), SW18.2
- new net: D11.2 (A), SW10.2
- new net: D14.1 (K), S1.3
- new net: D8.2 (A), SW7.2
- new net: D3.2 (A), SW2.2
- new net: D5.2 (A), SW4.2
- new net: D18.2 (A), SW5.2
- new net: D16.2 (A), JP1.1 (A)
- new net: D15.2 (A), SW14.2
- new net: D13.1 (K), S1.2
- new net: D17.1 (K), S1.4
- new net: D21.1 (K), S1.6
- new net: D12.2 (A), SW11.2
- new net: J2.A7 (D-), J2.B7 (D-), R3.1
- new net +3.3V: C1.2, C4.1, C5.1, J1.2 (VCC), TP1.1, U1.6 (VDD), U2.2 (VO)
- new net CC1: J2.A5 (CC1), R1.2
- new net CC2: J2.B5 (CC2), R2.2
- new net COL1: D18.1 (K), D2.1 (K), D3.1 (K), D4.1 (K), D5.1 (K), R7.1, U1.14 (PC7)
- new net COL2: D11.1 (K), D15.1 (K), D19.1 (K), D6.1 (K), D7.1 (K), R8.1, U1.13 (PC6)
- new net COL3: D10.1 (K), D12.1 (K), D16.1 (K), D20.1 (K), D8.1 (K), R9.1, U1.12 (PC5)
- new net COL4: R11.2, S1.5, U1.11 (PC4)
- new net JOY_E: SW12.1, SW12.6, U1.1 (PD7)
- new net JOY_H: SW12.5, U1.2 (PA1)
- new net JOY_V: SW12.2, U1.3 (PA2)
- new net ROW1: D17.2 (A), SW1.1, SW8.1, SW9.1, U1.20 (PD6)
- new net ROW2: D21.2 (A), SW2.1, SW6.1, SW7.1, U1.16 (PD2)
- new net ROW3: D9.2 (A), SW10.1, SW11.1, SW3.1, U1.10 (PC3)
- new net ROW4: D13.2 (A), JP1.2 (B), SW14.1, SW4.1, U1.7 (PC0)
- new net ROW5: D14.2 (A), JP2.2 (B), SW18.1, SW5.1, U1.5 (PD0)
- new net SCL: J1.4 (SCL), U1.9 (PC2)
- new net SDA: J1.3 (SDA), U1.8 (PC1)
- new net SWIO: TP3.1, U1.15 (PD1)
- new net USB_N: R3.2, R5.2, U1.18 (PD4)
- new net USB_P: R4.2, U1.17 (PD3)
- new net USB_PU: R5.1, U1.19 (PD5)
- new net VBUS: C2.1, C3.1, J2.A4 (VBUS), J2.A9 (VBUS), J2.B4 (VBUS), J2.B9 (VBUS), U2.3 (VI)
- no-connect marks 0 -> 2

Commit message: Frontpanel :D
Parts:
- added H1, H2, H3, H4: Gamepad, mountinghole:mountinghole_1.6mm, symbol Mechanical:MountingHole_Pad
- added N2: Stamp, stamp:stamp, symbol Mechanical:Housing
- added U1: LM66100DCKR, ideal_diode:SC-70-6_L2.0-W1.3-P0.65-LS2.1-BL, symbol LM66100DCKR:LM66100DCKR
- C1: footprint Capacitor_SMD:C_0603_1608Metric -> Capacitor_SMD:C_0402_1005Metric; LCSC C282519 -> C1525
- C2, C5: LCSC C107372 -> C88945
- C3, C4: LCSC (none) -> C1525
- R3: renamed from R5; LCSC (none) -> C25867
- R4: renamed from R3; LCSC (none) -> C25105
- R5: renamed from R4; LCSC (none) -> C25105
- SW10: renamed from SW14; LCSC (none) -> C115348
- SW11: renamed from SW18; LCSC (none) -> C115348
- SW12: renamed from SW9; LCSC (none) -> C115348
- SW13: renamed from SW7; LCSC (none) -> C115348
- SW14: renamed from SW11; LCSC (none) -> C115348
- SW2: renamed from SW1; LCSC (none) -> C115348
- SW3: renamed from SW2; LCSC (none) -> C115348
- SW4: renamed from SW3; LCSC (none) -> C115348
- SW5: renamed from SW4; LCSC (none) -> C115348
- SW6: renamed from SW5; LCSC (none) -> C318992
- SW7: renamed from SW8; LCSC (none) -> C318992
- SW8: renamed from SW6; LCSC (none) -> C115348
- SW9: renamed from SW10; LCSC (none) -> C115348
- U3: renamed from U2; LCSC (none) -> C498153
- renumbered D2 to D1, D19 to D10, D9 to D11, D17 to D12, D21 to D15, D10 to D16, D8 to D17, D12 to D18, D16 to D19, D3 to D2, D4 to D3, D5 to D4, D18 to D5, D11 to D8, D15 to D9, H1 to H5, H2 to H6, H3 to H7, H4 to H8, R7 to R6, R8 to R7, R11 to R8, SW12 to SW1, U1 to U2
Connections:
- net +3.3V: now also U1.3 (~{CE}), U1.6 (VOUT); no longer J1.2 (VCC)
- net GND: now also H1.1, H2.1, H3.1, H4.1, U1.2 (GND), U1.4 (NC), U1.5 (ST)
- new net: J1.2 (VCC), U1.1 (VIN)
Other:
- moved on the sheet: J1

Commit message: Frontpanel stuff
Parts:
- removed C1: 100n, Capacitor_SMD:C_0402_1005Metric, symbol vfd:C_Small
- removed C2, C5: 1u, Capacitor_SMD:C_0402_1005Metric, symbol mch2021-rescue:C-Device
- removed C3, C4: 100n, Capacitor_SMD:C_0402_1005Metric, symbol mch2021-rescue:C-Device
- removed D1, D10, D11, D12, D13, D14, D15, D16, D17, D18, D19, D2, D20, D3, D4, D5, D6, D7, D8, D9: LL4148, Diode_SMD:D_SOD-323, symbol button_matrix:D_Small
- removed H1, H2, H3, H4: Gamepad, mountinghole:mountinghole_1.6mm, symbol Mechanical:MountingHole_Pad
- removed J1: I2C, library:1X04_1MM_RA_GND, symbol symbols:QWIIC_MCH
- removed J2: USB device, Connector_USB:USB_C_Receptacle_HRO_TYPE-C-31-M-12, symbol mch2021-rescue:USB_C_Receptacle_USB2.0-Connector
- removed JP1: A0, Jumper:SolderJumper-2_P1.3mm_Open_TrianglePad1.0x1.5mm, symbol vfd:Jumper_2_Open
- removed JP2: A1, Jumper:SolderJumper-2_P1.3mm_Open_TrianglePad1.0x1.5mm, symbol vfd:Jumper_2_Open
- removed N2: Stamp, stamp:stamp, symbol Mechanical:Housing
- removed R1, R2: 5k1, Resistor_SMD:R_0402_1005Metric, symbol mch2021-rescue:R_Small-Device
- removed R3: 1.5k, Resistor_SMD:R_0402_1005Metric, symbol mch2021-rescue:R-Device
- removed R4, R5: 33, Resistor_SMD:R_0402_1005Metric, symbol mch2021-rescue:R-Device
- removed R6, R7, R8, R9: 10k, Resistor_SMD:R_0402_1005Metric, symbol button_matrix:R
- removed S1: JS1400BFQ, joystick_footprint:SW_JS1400BFQ, symbol JS1400BFQ:JS1400BFQ
- removed SW1: K1-1539SA-01, analog_joystick:SW-SMD_K1-1539SA-01, symbol SW-SMD_K1-1539SA-01:K1-1539SA-01
- removed SW10: SELECT, button_footprint:KEY-SMD_2P-L6.0-W6.0-P6.00, symbol Switch:SW_Push
- removed SW11: START, button_footprint:KEY-SMD_2P-L6.0-W6.0-P6.00, symbol Switch:SW_Push
- removed SW12: +, button_footprint:KEY-SMD_2P-L6.0-W6.0-P6.00, symbol Switch:SW_Push
- removed SW13: -, button_footprint:KEY-SMD_2P-L6.0-W6.0-P6.00, symbol Switch:SW_Push
- removed SW14: Z, button_footprint:KEY-SMD_2P-L6.0-W6.0-P6.00, symbol Switch:SW_Push
- removed SW2: X, button_footprint:KEY-SMD_2P-L6.0-W6.0-P6.00, symbol Switch:SW_Push
- removed SW3: A, button_footprint:KEY-SMD_2P-L6.0-W6.0-P6.00, symbol Switch:SW_Push
- removed SW4: B, button_footprint:KEY-SMD_2P-L6.0-W6.0-P6.00, symbol Switch:SW_Push
- removed SW5: Y, button_footprint:KEY-SMD_2P-L6.0-W6.0-P6.00, symbol Switch:SW_Push
- removed SW6: R, shoulderbutton:KEY-TH_TC-1101V-C-A-W, symbol pushbutton_gnd:pushbutton_gnd
- removed SW7: L, shoulderbutton:KEY-TH_TC-1101V-C-A-W, symbol pushbutton_gnd:pushbutton_gnd
- removed SW8: HOME, button_footprint:KEY-SMD_2P-L6.0-W6.0-P6.00, symbol Switch:SW_Push
- removed SW9: C, button_footprint:KEY-SMD_2P-L6.0-W6.0-P6.00, symbol Switch:SW_Push
- removed TP1: 3.3v, TestPoint:TestPoint_Pad_D1.5mm, symbol vfd:TestPoint
- removed TP2: GND, TestPoint:TestPoint_Pad_D1.5mm, symbol vfd:TestPoint
- removed TP3: SWIO, TestPoint:TestPoint_Pad_D1.5mm, symbol vfd:TestPoint
- removed U1: LM66100DCKR, ideal_diode:SC-70-6_L2.0-W1.3-P0.65-LS2.1-BL, symbol LM66100DCKR:LM66100DCKR
- removed U2: CH32V003F4U6, Package_DFN_QFN:QFN-20-1EP_3x3mm_P0.4mm_EP1.65x1.65mm, symbol vfd:CH32V003F4U6
- removed U3: LM1117MP-3.3, Package_TO_SOT_SMD:SOT-223-3_TabPin2, symbol Regulator_Linear:LM1117MP-3.3
- N1: footprint design:proto1_kicad_frontpanel -> design:frontpanel_template
Connections:
- no-connect marks 2 -> 0
Other:
- moved on the sheet: H5, H6, H7, H8, N1
