File: backexpansion/expansion-template/expansion-template.kicad_pcb (KiCad board)
At the start: 4 copper layers, 86 x 68 mm, 44 parts, among them J1 Internal Add-On

Commit message: Make the board 2mm taller to reach 70mm hight, this allows production at JLCPCB without the need for panneling.
Other:
- board size 86 x 68 mm -> 86 x 70 mm
